Commit message: adjusted constants + sign for correct direction

File: reseq_gazebo/description/robot_core.xacro (robot description, xacro)
@@ -11,6 +11,6 @@
   <xacro:property name="JointDiameter" value="0.06"/>
   <xacro:property name="toll" value="0.005"/>
-  <xacro:property name="JointA" value="0.08"/>
-  <xacro:property name="JointB" value="0.2"/>
+  <xacro:property name="JointA" value="0.1"/>
+  <xacro:property name="JointB" value="0.15"/>
   <xacro:property name="JointABottomClearance" value="0.04"/>
   <!-- All values are in radiants -->

Commit message: more space in joint area, still miss feedback yaw

File: reseq_gazebo/description/robot_core.xacro (robot description, xacro)
@@ -11,6 +11,6 @@
   <xacro:property name="JointDiameter" value="0.06"/>
   <xacro:property name="toll" value="0.005"/>
-  <xacro:property name="JointA" value="0.1"/>
-  <xacro:property name="JointB" value="0.15"/>
+  <xacro:property name="JointA" value="0.15"/>
+  <xacro:property name="JointB" value="0.2"/>
   <xacro:property name="JointABottomClearance" value="0.04"/>
   <!-- All values are in radiants -->

Commit message: added mk1 arm, new inertia problem :(

File: reseq_gazebo/description/robot_core.xacro (robot description, xacro)
@@ -10,12 +10,16 @@
   <xacro:property name="ChassisTopAndBottomClearance" value="0.02"/>
   <xacro:property name="JointDiameter" value="0.06"/>
-  <xacro:property name="toll" value="0.005"/>
+  <xacro:property name="toll" value="0.01"/>
   <xacro:property name="JointA" value="0.15"/>
   <xacro:property name="JointB" value="0.2"/>
   <xacro:property name="JointABottomClearance" value="0.04"/>
+  <xacro:property name="ForkThickness" value="0.01"/>
+  <xacro:property name="ForkHeight" value="0.04"/>
+  <xacro:property name="JetsonHolderLength" value="0.2"/>
+  <xacro:property name="JetsonHolderWidth" value="0.1"/>
   <!-- All values are in radiants -->
-  <xacro:property name="pitch" value="2.0944"/>
-  <xacro:property name="roll" value="1.74533"/>
-  <xacro:property name="yaw" value="0.523599"/>
+  <xacro:property name="pitch" value="${pi/2}"/>
+  <xacro:property name="roll" value="${pi*3/4}"/>
+  <xacro:property name="yaw" value="${pi/4}"/>
   <!-- All values are in kg -->
   <xacro:property name="WheelMass" value="0.1"/>
@@ -833,3 +837,96 @@
     <material>Gazebo/Black</material>
   </gazebo>
+    <!-- Arm mK1 -->
+  <joint name="arm_mK1_joint" type="revolute">
+    <parent link="chassis1_link"/>
+    <child link="arm_mK1_link"/>
+    <!-- Effort in Nm, angle in radians -->
+    <limit effort="10.0" lower="-${pi/4}" upper="${pi/2}" velocity="0.5"/>
+    <origin xyz="${WheelBase/2} 0 0" rpy="${pi/2} 0 0" />
+    <axis xyz="0 0 -1"/>
+  </joint>
+  <link name="arm_mK1_link">
+    <!-- cylinder to the right -->
+    <visual>
+      <origin xyz="0 0 ${ForkThickness/2+toll+ModuleWidth/2}" />
+      <geometry>
+        <cylinder radius="${ForkHeight/2}" length="${ForkThickness}"/>
+      </geometry>
+      <material name="JointColor"/>
+    </visual>
+    <!-- cylinder to the left -->
+    <visual>
+      <origin xyz="0 0 -${ForkThickness/2+toll+ModuleWidth/2}" />
+      <geometry>
+        <cylinder radius="${ForkHeight/2}" length="${ForkThickness}"/>
+      </geometry>
+      <material name="JointColor"/>
+    </visual>
+    <!-- right side of the fork -->
+    <visual>
+      <origin xyz="0 -${(toll+EquivalentWheelDiameter/2)/2} ${ForkThickness/2+toll+ModuleWidth/2}" />
+      <geometry>
+        <box size="${ForkHeight} ${toll+EquivalentWheelDiameter/2} ${ForkThickness}"/>
+      </geometry>
+      <material name="JointColor"/>
+    </visual>
+    <!-- left side of the fork -->
+    <visual>
+      <origin xyz="0 -${(toll+EquivalentWheelDiameter/2)/2} -${ForkThickness/2+toll+ModuleWidth/2}" />
+      <geometry>
+        <box size="${ForkHeight} ${toll+EquivalentWheelDiameter/2} ${ForkThickness}"/>
+      </geometry>
+      <material name="JointColor"/>
+    </visual>
+    <!-- front side of the fork -->
+    <visual>
+      <origin xyz="0 -${ForkThickness/2+toll+EquivalentWheelDiameter/2} 0" />
+      <geometry>
+        <box size="${ForkHeight} ${ForkThickness} ${ModuleWidth+(toll+ForkThickness)*2}"/>
+      </geometry>
+      <material name="JointColor"/>
+    </visual>
+    <!-- Jetson holder -->
+    <visual>
+      <origin xyz="0 -${ForkThickness/2+toll+EquivalentWheelDiameter/2+JetsonHolderLength/2} 0" />
+      <geometry>
+        <box size="${ForkHeight} ${JetsonHolderLength} ${JetsonHolderWidth}"/>
+      </geometry>
+      <material name="JointColor"/>
+    </visual>
+    <!-- cylinder to the right -->
+    <collision>
+      <origin xyz="0 0 ${ForkThickness/2+toll+ModuleWidth/2}" />
+      <geometry>
+        <cylinder radius="${ForkHeight/2}" length="${ForkThickness}"/>
+      </geometry>
+    </collision>
+    <!-- cylinder to the left -->
+    <collision>
+      <origin xyz="0 0 -${ForkThickness/2+toll+ModuleWidth/2}" />
+      <geometry>
+        <cylinder radius="${ForkHeight/2}" length="${ForkThickness}"/>
+      </geometry>
+    </collision>
+    <!-- front side of the fork -->
+    <collision>
+      <origin xyz="0 -${ForkThickness/2+toll+EquivalentWheelDiameter/2} 0" />
+      <geometry>
+        <box size="${ForkHeight} ${ForkThickness} ${ModuleWidth+(toll+ForkThickness)*2}"/>
+      </geometry>
+    </collision>
+    <!-- Jetson holder -->
+    <collision>
+      <origin xyz="0 -${ForkThickness/2+toll+EquivalentWheelDiameter/2+JetsonHolderLength/2} 0" />
+      <geometry>
+        <box size="${ForkHeight} ${JetsonHolderLength} ${JetsonHolderWidth}"/>
+      </geometry>
+    </collision>
+    <xacro:inertial_box mass="${0.5}" x="${ForkHeight}" y="${JetsonHolderLength}" z="${JetsonHolderWidth}">
+      <origin xyz="0 -${ForkThickness/2+toll+EquivalentWheelDiameter/2+JetsonHolderLength/2} 0" rpy="0 0 0"/>
+    </xacro:inertial_box>
+  </link>
+  <gazebo reference="arm_mK1_link">
+    <material>Gazebo/Grey</material>
+  </gazebo>
 </robot>

File: reseq_gazebo/description/ros2_control.xacro (robot description, xacro)
@@ -146,4 +146,7 @@
             <state_interface name="position"/>
         </joint>
+        <joint name="arm_mK1_joint">
+            <state_interface name="position"/>
+        </joint>
     </ros2_control>
     <gazebo>

Commit message: robot_core better formatting and added comments

File: reseq_gazebo/description/robot_core.xacro (robot description, xacro)
@@ -37,4 +37,7 @@
     <color rgba="0.5 0.5 0.5 1" />
   </material>
+  <material name="ArmColor">
+    <color rgba="0.5 0.5 0.5 1" />
+  </material>
   <!-- BASE LINK (center of equivalent wheel of module 1)-->
   <link name="base_link" />
@@ -183,37 +186,37 @@
   </joint>
   <link name="joint_a_1_link">
-    <visual>
-      <geometry>
-        <!-- left "toll" from each Track for clearance  -->
+    <!-- gearbox cilinder -->
+    <visual>
+      <geometry>
         <cylinder radius="${JointDiameter/2}" length="${ModuleWidth-2*TrackWidth-toll*2}"/>
       </geometry>
       <material name="JointColor"/>
     </visual>
+    <!-- horizontal shaft -->
     <visual>
       <origin xyz="${-JointA/2} 0 0" />
       <geometry>
-        <!-- left "toll" from each Track for clearance  -->
         <box size="${JointA} ${EquivalentWheelDiameter-2*JointABottomClearance} ${ModuleWidth-2*TrackWidth-toll*2}"/>
       </geometry>
       <material name="JointColor"/>
     </visual>
+    <!-- to hide space wile rotating -->
     <visual>
       <origin xyz="${-JointA} 0 0" />
       <geometry>
-        <!-- left "toll" from each Track for clearance  -->
         <sphere radius="${(ModuleWidth-2*TrackWidth-toll*2)/2}"/>
       </geometry>
       <material name="JointColor"/>
     </visual>
-    <collision>
-      <geometry>
-        <!-- left "toll" from each Track for clearance  -->
+    <!-- gearbox cilinder -->
+    <collision>
+      <geometry>
         <cylinder radius="${JointDiameter/2}" length="${ModuleWidth-2*TrackWidth-toll*2}"/>
       </geometry>
     </collision>
+    <!-- horizontal shaft -->
     <collision>
       <origin xyz="${-JointA/2} 0 0" />
       <geometry>
-        <!-- left "toll" from each Track for clearance  -->
         <box size="${JointA} ${EquivalentWheelDiameter-2*JointABottomClearance} ${ModuleWidth-2*TrackWidth-toll*2}"/>
       </geometry>
@@ -239,5 +242,4 @@
       <origin xyz="0 0 ${-(JointB-WheelBase/2-EquivalentWheelDiameter/6)/2}" />
       <geometry>
-        <!-- left "toll" from each Track for clearance  -->
         <cylinder radius="${(ModuleWidth-2*TrackWidth-toll*2)/2}" length="${JointB-WheelBase/2-EquivalentWheelDiameter/6}"/>
       </geometry>
@@ -247,5 +249,4 @@
       <origin xyz="0 0 ${-(JointB-WheelBase/2-EquivalentWheelDiameter/6)/2}" />
       <geometry>
-        <!-- left "toll" from each Track for clearance  -->
         <cylinder radius="${(ModuleWidth-2*TrackWidth-toll*2)/2}" length="${JointB-WheelBase/2-EquivalentWheelDiameter/6}"/>
       </geometry>
@@ -405,37 +406,37 @@
   </joint>
   <link name="joint_a_2_link">
-    <visual>
-      <geometry>
-        <!-- left "toll" from each Track for clearance  -->
+    <!-- gearbox cilinder -->
+    <visual>
+      <geometry>
         <cylinder radius="${JointDiameter/2}" length="${ModuleWidth-2*TrackWidth-toll*2}"/>
       </geometry>
       <material name="JointColor"/>
     </visual>
+    <!-- horizontal shaft -->
     <visual>
       <origin xyz="${-JointA/2} 0 0" />
       <geometry>
-        <!-- left "toll" from each Track for clearance  -->
         <box size="${JointA} ${EquivalentWheelDiameter-2*JointABottomClearance} ${ModuleWidth-2*TrackWidth-toll*2}"/>
       </geometry>
       <material name="JointColor"/>
     </visual>
+    <!-- to hide space wile rotating -->
     <visual>
       <origin xyz="${-JointA} 0 0" />
       <geometry>
-        <!-- left "toll" from each Track for clearance  -->
         <sphere radius="${(ModuleWidth-2*TrackWidth-toll*2)/2}"/>
       </geometry>
       <material name="JointColor"/>
     </visual>
-    <collision>
-      <geometry>
-        <!-- left "toll" from each Track for clearance  -->
+    <!-- gearbox cilinder -->
+    <collision>
+      <geometry>
         <cylinder radius="${JointDiameter/2}" length="${ModuleWidth-2*TrackWidth-toll*2}"/>
       </geometry>
     </collision>
+    <!-- horizontal shaft -->
     <collision>
       <origin xyz="${-JointA/2} 0 0" />
       <geometry>
-        <!-- left "toll" from each Track for clearance  -->
         <box size="${JointA} ${EquivalentWheelDiameter-2*JointABottomClearance} ${ModuleWidth-2*TrackWidth-toll*2}"/>
       </geometry>
@@ -461,5 +462,4 @@
       <origin xyz="0 0 ${-(JointB-WheelBase/2-EquivalentWheelDiameter/6)/2}" />
       <geometry>
-        <!-- left "toll" from each Track for clearance  -->
         <cylinder radius="${(ModuleWidth-2*TrackWidth-toll*2)/2}" length="${JointB-WheelBase/2-EquivalentWheelDiameter/6}"/>
       </geometry>
@@ -469,5 +469,4 @@
       <origin xyz="0 0 ${-(JointB-WheelBase/2-EquivalentWheelDiameter/6)/2}" />
       <geometry>
-        <!-- left "toll" from each Track for clearance  -->
         <cylinder radius="${(ModuleWidth-2*TrackWidth-toll*2)/2}" length="${JointB-WheelBase/2-EquivalentWheelDiameter/6}"/>
       </geometry>
@@ -627,37 +626,37 @@
   </joint>
   <link name="joint_a_3_link">
-    <visual>
-      <geometry>
-        <!-- left "toll" from each Track for clearance  -->
+    <!-- gearbox cilinder -->
+    <visual>
+      <geometry>
         <cylinder radius="${JointDiameter/2}" length="${ModuleWidth-2*TrackWidth-toll*2}"/>
       </geometry>
       <material name="JointColor"/>
     </visual>
+    <!-- horizontal shaft -->
     <visual>
       <origin xyz="${-JointA/2} 0 0" />
       <geometry>
-        <!-- left "toll" from each Track for clearance  -->
         <box size="${JointA} ${EquivalentWheelDiameter-2*JointABottomClearance} ${ModuleWidth-2*TrackWidth-toll*2}"/>
       </geometry>
       <material name="JointColor"/>
     </visual>
+    <!-- to hide space wile rotating -->
     <visual>
       <origin xyz="${-JointA} 0 0" />
       <geometry>
-        <!-- left "toll" from each Track for clearance  -->
         <sphere radius="${(ModuleWidth-2*TrackWidth-toll*2)/2}"/>
       </geometry>
       <material name="JointColor"/>
     </visual>
-    <collision>
-      <geometry>
-        <!-- left "toll" from each Track for clearance  -->
+    <!-- gearbox cilinder -->
+    <collision>
+      <geometry>
         <cylinder radius="${JointDiameter/2}" length="${ModuleWidth-2*TrackWidth-toll*2}"/>
       </geometry>
     </collision>
+    <!-- horizontal shaft -->
     <collision>
       <origin xyz="${-JointA/2} 0 0" />
       <geometry>
-        <!-- left "toll" from each Track for clearance  -->
         <box size="${JointA} ${EquivalentWheelDiameter-2*JointABottomClearance} ${ModuleWidth-2*TrackWidth-toll*2}"/>
       </geometry>
@@ -683,5 +682,4 @@
       <origin xyz="0 0 ${-(JointB-WheelBase/2-EquivalentWheelDiameter/6)/2}" />
       <geometry>
-        <!-- left "toll" from each Track for clearance  -->
         <cylinder radius="${(ModuleWidth-2*TrackWidth-toll*2)/2}" length="${JointB-WheelBase/2-EquivalentWheelDiameter/6}"/>
       </geometry>
@@ -691,5 +689,4 @@
       <origin xyz="0 0 ${-(JointB-WheelBase/2-EquivalentWheelDiameter/6)/2}" />
       <geometry>
-        <!-- left "toll" from each Track for clearance  -->
         <cylinder radius="${(ModuleWidth-2*TrackWidth-toll*2)/2}" length="${JointB-WheelBase/2-EquivalentWheelDiameter/6}"/>
       </geometry>
@@ -837,5 +834,5 @@
     <material>Gazebo/Black</material>
   </gazebo>
-    <!-- Arm mK1 -->
+  <!-- Arm mK1 -->
   <joint name="arm_mK1_joint" type="revolute">
     <parent link="chassis1_link"/>

Commit message: fixed jump start, it was not related to inertia :)

File: reseq_gazebo/description/robot_core.xacro (robot description, xacro)
@@ -22,5 +22,5 @@
   <!-- All values are in radiants -->
   <xacro:property name="pitch" value="${pi/2}"/>
-  <xacro:property name="roll" value="${pi*3/4}"/>
+  <xacro:property name="roll" value="${pi*0.9}"/>
   <xacro:property name="yaw" value="${pi/4}"/>
   <!-- All values are in kg -->
@@ -248,10 +248,4 @@
       <material name="JointColor"/>
     </visual>
-    <collision>
-      <origin xyz="0 0 ${-(JointB-WheelBase/2-EquivalentWheelDiameter/6)/2}" />
-      <geometry>
-        <cylinder radius="${(ModuleWidth-2*TrackWidth-toll*2)/2}" length="${JointB-WheelBase/2-EquivalentWheelDiameter/6}"/>
-      </geometry>
-    </collision>
     <xacro:inertial_cylinder mass="${JointBMass}" length="${JointB-WheelBase/2-EquivalentWheelDiameter/6}" radius="${(ModuleWidth-2*TrackWidth-toll*2)/2}">
       <origin xyz="0 0 ${-(JointB-WheelBase/2-EquivalentWheelDiameter/6)/2}" rpy="0 0 0"/>
@@ -468,10 +462,4 @@
       <material name="JointColor"/>
     </visual>
-    <collision>
-      <origin xyz="0 0 ${-(JointB-WheelBase/2-EquivalentWheelDiameter/6)/2}" />
-      <geometry>
-        <cylinder radius="${(ModuleWidth-2*TrackWidth-toll*2)/2}" length="${JointB-WheelBase/2-EquivalentWheelDiameter/6}"/>
-      </geometry>
-    </collision>
     <xacro:inertial_cylinder mass="${JointBMass}" length="${JointB-WheelBase/2-EquivalentWheelDiameter/6}" radius="${(ModuleWidth-2*TrackWidth-toll*2)/2}">
       <origin xyz="0 0 ${-(JointB-WheelBase/2-EquivalentWheelDiameter/6)/2}" rpy="0 0 0"/>
@@ -688,10 +676,4 @@
       <material name="JointColor"/>
     </visual>
-    <collision>
-      <origin xyz="0 0 ${-(JointB-WheelBase/2-EquivalentWheelDiameter/6)/2}" />
-      <geometry>
-        <cylinder radius="${(ModuleWidth-2*TrackWidth-toll*2)/2}" length="${JointB-WheelBase/2-EquivalentWheelDiameter/6}"/>
-      </geometry>
-    </collision>
     <xacro:inertial_cylinder mass="${JointBMass}" length="${JointB-WheelBase/2-EquivalentWheelDiameter/6}" radius="${(ModuleWidth-2*TrackWidth-toll*2)/2}">
       <origin xyz="0 0 ${-(JointB-WheelBase/2-EquivalentWheelDiameter/6)/2}" rpy="0 0 0"/>
@@ -841,7 +823,7 @@
     <child link="arm_mK1_link"/>
     <!-- Effort in Nm, angle in radians -->
-    <limit effort="10.0" lower="-${pi/4}" upper="${pi/2}" velocity="0.5"/>
+    <limit effort="10.0" lower="-${pi*0.001}" upper="${pi/2}" velocity="0.5"/>
     <origin xyz="${WheelBase/2} 0 0" rpy="${pi/2} 0 0" />
-    <axis xyz="0 0 -1"/>
+    <axis xyz="0 0 1"/>
   </joint>
   <link name="arm_mK1_link">
@@ -852,5 +834,5 @@
         <cylinder radius="${ForkHeight/2}" length="${ForkThickness}"/>
       </geometry>
-      <material name="JointColor"/>
+      <material name="ArmColor"/>
     </visual>
     <!-- cylinder to the left -->
@@ -860,37 +842,37 @@
         <cylinder radius="${ForkHeight/2}" length="${ForkThickness}"/>
       </geometry>
-      <material name="JointColor"/>
+      <material name="ArmColor"/>
     </visual>
     <!-- right side of the fork -->
     <visual>
-      <origin xyz="0 -${(toll+EquivalentWheelDiameter/2)/2} ${ForkThickness/2+toll+ModuleWidth/2}" />
-      <geometry>
-        <box size="${ForkHeight} ${toll+EquivalentWheelDiameter/2} ${ForkThickness}"/>
-      </geometry>
-      <material name="JointColor"/>
+      <origin xyz="${(toll+EquivalentWheelDiameter/2)/2} 0 ${ForkThickness/2+toll+ModuleWidth/2}" />
+      <geometry>
+        <box size="${toll+EquivalentWheelDiameter/2} ${ForkHeight} ${ForkThickness}"/>
+      </geometry>
+      <material name="ArmColor"/>
     </visual>
     <!-- left side of the fork -->
     <visual>
-      <origin xyz="0 -${(toll+EquivalentWheelDiameter/2)/2} -${ForkThickness/2+toll+ModuleWidth/2}" />
-      <geometry>
-        <box size="${ForkHeight} ${toll+EquivalentWheelDiameter/2} ${ForkThickness}"/>
-      </geometry>
-      <material name="JointColor"/>
+      <origin xyz="${(toll+EquivalentWheelDiameter/2)/2} 0 -${ForkThickness/2+toll+ModuleWidth/2}" />
+      <geometry>
+        <box size="${toll+EquivalentWheelDiameter/2} ${ForkHeight} ${ForkThickness}"/>
+      </geometry>
+      <material name="ArmColor"/>
     </visual>
     <!-- front side of the fork -->
     <visual>
-      <origin xyz="0 -${ForkThickness/2+toll+EquivalentWheelDiameter/2} 0" />
-      <geometry>
-        <box size="${ForkHeight} ${ForkThickness} ${ModuleWidth+(toll+ForkThickness)*2}"/>
-      </geometry>
-      <material name="JointColor"/>
+      <origin xyz="${ForkThickness/2+toll+EquivalentWheelDiameter/2} 0 0" />
+      <geometry>
+        <box size="${ForkThickness} ${ForkHeight} ${ModuleWidth+(toll+ForkThickness)*2}"/>
+      </geometry>
+      <material name="ArmColor"/>
     </visual>
     <!-- Jetson holder -->
     <visual>
-      <origin xyz="0 -${ForkThickness/2+toll+EquivalentWheelDiameter/2+JetsonHolderLength/2} 0" />
-      <geometry>
-        <box size="${ForkHeight} ${JetsonHolderLength} ${JetsonHolderWidth}"/>
-      </geometry>
-      <material name="JointColor"/>
+      <origin xyz="${ForkThickness/2+toll+EquivalentWheelDiameter/2+JetsonHolderLength/2} 0 0" />
+      <geometry>
+        <box size="${JetsonHolderLength} ${ForkHeight} ${JetsonHolderWidth}"/>
+      </geometry>
+      <material name="ArmColor"/>
     </visual>
     <!-- cylinder to the right -->
@@ -910,18 +892,18 @@
     <!-- front side of the fork -->
     <collision>
-      <origin xyz="0 -${ForkThickness/2+toll+EquivalentWheelDiameter/2} 0" />
-      <geometry>
-        <box size="${ForkHeight} ${ForkThickness} ${ModuleWidth+(toll+ForkThickness)*2}"/>
+      <origin xyz="${ForkThickness/2+toll+EquivalentWheelDiameter/2} 0 0" />
+      <geometry>
+        <box size="${ForkThickness} ${ForkHeight} ${ModuleWidth+(toll+ForkThickness)*2}"/>
       </geometry>
     </collision>
     <!-- Jetson holder -->
     <collision>
-      <origin xyz="0 -${ForkThickness/2+toll+EquivalentWheelDiameter/2+JetsonHolderLength/2} 0" />
-      <geometry>
-        <box size="${ForkHeight} ${JetsonHolderLength} ${JetsonHolderWidth}"/>
+      <origin xyz="${ForkThickness/2+toll+EquivalentWheelDiameter/2+JetsonHolderLength/2} 0 0" />
+      <geometry>
+        <box size="${JetsonHolderLength} ${ForkHeight} ${JetsonHolderWidth}"/>
       </geometry>
     </collision>
     <xacro:inertial_box mass="${0.5}" x="${ForkHeight}" y="${JetsonHolderLength}" z="${JetsonHolderWidth}">
-      <origin xyz="0 -${ForkThickness/2+toll+EquivalentWheelDiameter/2+JetsonHolderLength/2} 0" rpy="0 0 0"/>
+      <origin xyz="${ForkThickness/2+toll+EquivalentWheelDiameter/2+JetsonHolderLength/2} 0 0" rpy="0 0 0"/>
     </xacro:inertial_box>
   </link>
