Commit message: - minor changes (package.xml, README, body.xacro) - added lidar (still not able too see data from ros) - fixed arm.xacro inertia box - fixed (not quite sure about that) agevar reverse direction

File: reseq_gazebo/description/reseq_arm_mk1.xacro (robot description, xacro)
@@ -87,5 +87,5 @@
       </geometry>
     </collision>
-    <xacro:inertial_box mass="${0.5}" x="${ForkHeight}" y="${JetsonHolderLength}" z="${JetsonHolderWidth}">
+    <xacro:inertial_box mass="${0.5}" x="${JetsonHolderLength}" y="${ForkHeight}" z="${JetsonHolderWidth}">
       <origin xyz="${ForkThickness/2+toll+EquivalentWheelDiameter/2+JetsonHolderLength/2} 0 0" rpy="0 0 0"/>
     </xacro:inertial_box>

File: reseq_gazebo/description/reseq_body.xacro (robot description, xacro)
@@ -1,4 +1,4 @@
 <?xml version="1.0"?>
-<robot xmlns:xacro="http://www.ros.org/wiki/xacro"  name="reseq_gazebo">
+<robot xmlns:xacro="http://www.ros.org/wiki/xacro">
   <!-- This is a parametric description of reseq with 4 modules -->
   <!-- BASE LINK (center of equivalent wheel of module 1)-->

File: reseq_gazebo/description/reseq_parameters.xacro (robot description, xacro)
@@ -40,3 +40,6 @@
     <color rgba="0.5 0.5 0.5 1" />
   </material>
+  <material name="LidarColor">
+    <color rgba="0.5 0.5 0.5 1" />
+  </material>
 </robot>

File: reseq_gazebo/description/robot.urdf.xacro (robot description, xacro)
@@ -1,4 +1,4 @@
 <?xml version="1.0"?>
-<robot xmlns:xacro="http://www.ros.org/wiki/xacro"  name="reseq_gazebo">
+<robot xmlns:xacro="http://www.ros.org/wiki/xacro"  name="reseq">
   <xacro:arg name="use_ros2_control" default="true"/>
   <xacro:arg name="sim_mode" default="false"/>
@@ -7,4 +7,5 @@
   <xacro:include filename="reseq_body.xacro" />
   <xacro:include filename="reseq_arm_mk1.xacro" />
+  <xacro:include filename="lidar.xacro" />
   <xacro:include filename="ros2_control.xacro" />
 </robot>

Commit message: Started implementing joint position control currently It does not work so: - they are commented in 'launch_sim' file - the limit of the arm is set to '-pi*0.01' in stead of '-pi/2' to not   hit the ground

File: reseq_gazebo/description/reseq_arm_mk1.xacro (robot description, xacro)
@@ -6,5 +6,5 @@
     <child link="arm_mK1_link"/>
     <!-- Effort in Nm, angle in radians -->
-    <limit effort="10.0" lower="-${pi*0.001}" upper="${pi/2}" velocity="0.5"/>
+    <limit effort="10.0" lower="-${pi*0.01}" upper="${pi/2}" velocity="0.5"/>
     <origin xyz="${WheelBase/2} 0 0" rpy="${pi/2} 0 0" />
     <axis xyz="0 0 1"/>

File: reseq_gazebo/description/ros2_control.xacro (robot description, xacro)
@@ -13,4 +13,5 @@
             </command_interface>
             <state_interface name="position"/>
+            <state_interface name="velocity"/>
         </joint>
         <joint name="right_front_wheel_1_joint">
@@ -20,4 +21,5 @@
             </command_interface>
             <state_interface name="position"/>
+            <state_interface name="velocity"/>
         </joint>
         <joint name="left_back_wheel_1_joint">
@@ -27,4 +29,5 @@
             </command_interface>
             <state_interface name="position"/>
+            <state_interface name="velocity"/>
         </joint>
         <joint name="right_back_wheel_1_joint">
@@ -34,13 +37,20 @@
             </command_interface>
             <state_interface name="position"/>
+            <state_interface name="velocity"/>
         </joint>
         <joint name="joint_a_1_joint">
+            <command_interface name="position"/>
             <state_interface name="position"/>
+            <state_interface name="effort"/>
         </joint>
         <joint name="joint_b_1_joint">
+            <command_interface name="position"/>
             <state_interface name="position"/>
+            <state_interface name="effort"/>
         </joint>
         <joint name="chassis2_joint">
+            <command_interface name="position"/>
             <state_interface name="position"/>
+            <state_interface name="effort"/>
         </joint>
         <joint name="left_front_wheel_2_joint">
@@ -50,4 +60,5 @@
             </command_interface>
             <state_interface name="position"/>
+            <state_interface name="velocity"/>
         </joint>
         <joint name="right_front_wheel_2_joint">
@@ -57,4 +68,5 @@
             </command_interface>
             <state_interface name="position"/>
+            <state_interface name="velocity"/>
         </joint>
         <joint name="left_back_wheel_2_joint">
@@ -64,4 +76,5 @@
             </command_interface>
             <state_interface name="position"/>
+            <state_interface name="velocity"/>
         </joint>
         <joint name="right_back_wheel_2_joint">
@@ -71,13 +84,20 @@
             </command_interface>
             <state_interface name="position"/>
+            <state_interface name="velocity"/>
         </joint>
         <joint name="joint_a_2_joint">
+            <command_interface name="position"/>
             <state_interface name="position"/>
+            <state_interface name="effort"/>
         </joint>
         <joint name="joint_b_2_joint">
+            <command_interface name="position"/>
             <state_interface name="position"/>
+            <state_interface name="effort"/>
         </joint>
         <joint name="chassis3_joint">
+            <command_interface name="position"/>
             <state_interface name="position"/>
+            <state_interface name="effort"/>
         </joint>
         <joint name="left_front_wheel_3_joint">
@@ -87,4 +107,5 @@
             </command_interface>
             <state_interface name="position"/>
+            <state_interface name="velocity"/>
         </joint>
         <joint name="right_front_wheel_3_joint">
@@ -94,4 +115,5 @@
             </command_interface>
             <state_interface name="position"/>
+            <state_interface name="velocity"/>
         </joint>
         <joint name="left_back_wheel_3_joint">
@@ -101,4 +123,5 @@
             </command_interface>
             <state_interface name="position"/>
+            <state_interface name="velocity"/>
         </joint>
         <joint name="right_back_wheel_3_joint">
@@ -108,13 +131,20 @@
             </command_interface>
             <state_interface name="position"/>
+            <state_interface name="velocity"/>
         </joint>
         <joint name="joint_a_3_joint">
+            <command_interface name="position"/>
             <state_interface name="position"/>
+            <state_interface name="effort"/>
         </joint>
         <joint name="joint_b_3_joint">
+            <command_interface name="position"/>
             <state_interface name="position"/>
+            <state_interface name="effort"/>
         </joint>
         <joint name="chassis4_joint">
+            <command_interface name="position"/>
             <state_interface name="position"/>
+            <state_interface name="effort"/>
         </joint>
         <joint name="left_front_wheel_4_joint">
@@ -124,4 +154,5 @@
             </command_interface>
             <state_interface name="position"/>
+            <state_interface name="velocity"/>
         </joint>
         <joint name="right_front_wheel_4_joint">
@@ -131,4 +162,5 @@
             </command_interface>
             <state_interface name="position"/>
+            <state_interface name="velocity"/>
         </joint>
         <joint name="left_back_wheel_4_joint">
@@ -138,4 +170,5 @@
             </command_interface>
             <state_interface name="position"/>
+            <state_interface name="velocity"/>
         </joint>
         <joint name="right_back_wheel_4_joint">
@@ -145,7 +178,10 @@
             </command_interface>
             <state_interface name="position"/>
+            <state_interface name="velocity"/>
         </joint>
         <joint name="arm_mK1_joint">
+            <command_interface name="position"/>
             <state_interface name="position"/>
+            <state_interface name="effort"/>
         </joint>
     </ros2_control>
