Commit message: better xacro structure

File: reseq_gazebo/description/reseq_body.xacro (robot description, xacro)
@@ -1,45 +1,5 @@
 <?xml version="1.0"?>
 <robot xmlns:xacro="http://www.ros.org/wiki/xacro"  name="reseq_gazebo">
-  <!--
-  This is a parametric description of reseq with 4 modules
-  See 'Parameters.pdf' pdf for parameters meaning (when it will exist ;) )
-  All values are in meters
-  -->
-  <xacro:property name="WheelBase" value="0.25"/>
-  <xacro:property name="EquivalentWheelDiameter" value="0.12"/>
-  <xacro:property name="ModuleWidth" value="0.2"/>
-  <xacro:property name="TrackWidth" value="0.075"/>
-  <xacro:property name="ChassisTopAndBottomClearance" value="0.02"/>
-  <xacro:property name="JointDiameter" value="0.06"/>
-  <xacro:property name="toll" value="0.01"/>
-  <xacro:property name="JointA" value="0.15"/>
-  <xacro:property name="JointB" value="0.2"/>
-  <xacro:property name="JointABottomClearance" value="0.04"/>
-  <xacro:property name="ForkThickness" value="0.01"/>
-  <xacro:property name="ForkHeight" value="0.04"/>
-  <xacro:property name="JetsonHolderLength" value="0.2"/>
-  <xacro:property name="JetsonHolderWidth" value="0.1"/>
-  <!-- All values are in radiants -->
-  <xacro:property name="pitch" value="${pi/2}"/>
-  <xacro:property name="roll" value="${pi*0.9}"/>
-  <xacro:property name="yaw" value="${pi/4}"/>
-  <!-- All values are in kg -->
-  <xacro:property name="WheelMass" value="0.1"/>
-  <xacro:property name="ChassisMass" value="2.5"/>
-  <xacro:property name="JointAMass" value="0.1"/>
-  <xacro:property name="JointBMass" value="0.05"/>
-  <!-- Colors (from 0 to 1) -->
-  <material name="ChassisColor">
-    <color rgba="1 1 1 1" />
-  </material>
-  <material name="WheelColor">
-    <color rgba="0 0 0 1" />
-  </material>
-  <material name="JointColor">
-    <color rgba="0.5 0.5 0.5 1" />
-  </material>
-  <material name="ArmColor">
-    <color rgba="0.5 0.5 0.5 1" />
-  </material>
+  <!-- This is a parametric description of reseq with 4 modules -->
   <!-- BASE LINK (center of equivalent wheel of module 1)-->
   <link name="base_link" />
@@ -818,96 +778,3 @@
     <material>Gazebo/Black</material>
   </gazebo>
-  <!-- Arm mK1 -->
-  <joint name="arm_mK1_joint" type="revolute">
-    <parent link="chassis1_link"/>
-    <child link="arm_mK1_link"/>
-    <!-- Effort in Nm, angle in radians -->
-    <limit effort="10.0" lower="-${pi*0.001}" upper="${pi/2}" velocity="0.5"/>
-    <origin xyz="${WheelBase/2} 0 0" rpy="${pi/2} 0 0" />
-    <axis xyz="0 0 1"/>
-  </joint>
-  <link name="arm_mK1_link">
-    <!-- cylinder to the right -->
-    <visual>
-      <origin xyz="0 0 ${ForkThickness/2+toll+ModuleWidth/2}" />
-      <geometry>
-        <cylinder radius="${ForkHeight/2}" length="${ForkThickness}"/>
-      </geometry>
-      <material name="ArmColor"/>
-    </visual>
-    <!-- cylinder to the left -->
-    <visual>
-      <origin xyz="0 0 -${ForkThickness/2+toll+ModuleWidth/2}" />
-      <geometry>
-        <cylinder radius="${ForkHeight/2}" length="${ForkThickness}"/>
-      </geometry>
-      <material name="ArmColor"/>
-    </visual>
-    <!-- right side of the fork -->
-    <visual>
-      <origin xyz="${(toll+EquivalentWheelDiameter/2)/2} 0 ${ForkThickness/2+toll+ModuleWidth/2}" />
-      <geometry>
-        <box size="${toll+EquivalentWheelDiameter/2} ${ForkHeight} ${ForkThickness}"/>
-      </geometry>
-      <material name="ArmColor"/>
-    </visual>
-    <!-- left side of the fork -->
-    <visual>
-      <origin xyz="${(toll+EquivalentWheelDiameter/2)/2} 0 -${ForkThickness/2+toll+ModuleWidth/2}" />
-      <geometry>
-        <box size="${toll+EquivalentWheelDiameter/2} ${ForkHeight} ${ForkThickness}"/>
-      </geometry>
-      <material name="ArmColor"/>
-    </visual>
-    <!-- front side of the fork -->
-    <visual>
-      <origin xyz="${ForkThickness/2+toll+EquivalentWheelDiameter/2} 0 0" />
-      <geometry>
-        <box size="${ForkThickness} ${ForkHeight} ${ModuleWidth+(toll+ForkThickness)*2}"/>
-      </geometry>
-      <material name="ArmColor"/>
-    </visual>
-    <!-- Jetson holder -->
-    <visual>
-      <origin xyz="${ForkThickness/2+toll+EquivalentWheelDiameter/2+JetsonHolderLength/2} 0 0" />
-      <geometry>
-        <box size="${JetsonHolderLength} ${ForkHeight} ${JetsonHolderWidth}"/>
-      </geometry>
-      <material name="ArmColor"/>
-    </visual>
-    <!-- cylinder to the right -->
-    <collision>
-      <origin xyz="0 0 ${ForkThickness/2+toll+ModuleWidth/2}" />
-      <geometry>
-        <cylinder radius="${ForkHeight/2}" length="${ForkThickness}"/>
-      </geometry>
-    </collision>
-    <!-- cylinder to the left -->
-    <collision>
-      <origin xyz="0 0 -${ForkThickness/2+toll+ModuleWidth/2}" />
-      <geometry>
-        <cylinder radius="${ForkHeight/2}" length="${ForkThickness}"/>
-      </geometry>
-    </collision>
-    <!-- front side of the fork -->
-    <collision>
-      <origin xyz="${ForkThickness/2+toll+EquivalentWheelDiameter/2} 0 0" />
-      <geometry>
-        <box size="${ForkThickness} ${ForkHeight} ${ModuleWidth+(toll+ForkThickness)*2}"/>
-      </geometry>
-    </collision>
-    <!-- Jetson holder -->
-    <collision>
-      <origin xyz="${ForkThickness/2+toll+EquivalentWheelDiameter/2+JetsonHolderLength/2} 0 0" />
-      <geometry>
-        <box size="${JetsonHolderLength} ${ForkHeight} ${JetsonHolderWidth}"/>
-      </geometry>
-    </collision>
-    <xacro:inertial_box mass="${0.5}" x="${ForkHeight}" y="${JetsonHolderLength}" z="${JetsonHolderWidth}">
-      <origin xyz="${ForkThickness/2+toll+EquivalentWheelDiameter/2+JetsonHolderLength/2} 0 0" rpy="0 0 0"/>
-    </xacro:inertial_box>
-  </link>
-  <gazebo reference="arm_mK1_link">
-    <material>Gazebo/Grey</material>
-  </gazebo>
 </robot>

File: reseq_gazebo/description/robot.urdf.xacro (robot description, xacro)
@@ -4,5 +4,7 @@
   <xacro:arg name="sim_mode" default="false"/>
   <xacro:include filename="inertial_macros.xacro" />
-  <xacro:include filename="robot_core.xacro" />
+  <xacro:include filename="reseq_parameters.xacro" />
+  <xacro:include filename="reseq_body.xacro" />
+  <xacro:include filename="reseq_arm_mk1.xacro" />
   <xacro:include filename="ros2_control.xacro" />
 </robot>

Commit message: Fixed design error in xacro

File: reseq_gazebo/description/reseq_body.xacro (robot description, xacro)
@@ -202,11 +202,11 @@
   <link name="joint_b_1_link">
     <visual>
-      <origin xyz="0 0 ${-(JointB-WheelBase/2-EquivalentWheelDiameter/6)/2}" />
-      <geometry>
-        <cylinder radius="${(ModuleWidth-2*TrackWidth-toll*2)/2}" length="${JointB-WheelBase/2-EquivalentWheelDiameter/6}"/>
-      </geometry>
-      <material name="JointColor"/>
-    </visual>
-    <xacro:inertial_cylinder mass="${JointBMass}" length="${JointB-WheelBase/2-EquivalentWheelDiameter/6}" radius="${(ModuleWidth-2*TrackWidth-toll*2)/2}">
+      <origin xyz="0 0 -${JointB/2}" />
+      <geometry>
+        <cylinder radius="${(ModuleWidth-2*TrackWidth-toll*2)/2}" length="${JointB}"/>
+      </geometry>
+      <material name="JointColor"/>
+    </visual>
+    <xacro:inertial_cylinder mass="${JointBMass}" length="${JointB}" radius="${(ModuleWidth-2*TrackWidth-toll*2)/2}">
       <origin xyz="0 0 ${-(JointB-WheelBase/2-EquivalentWheelDiameter/6)/2}" rpy="0 0 0"/>
     </xacro:inertial_cylinder>
@@ -221,6 +221,5 @@
     <!-- Effort in Nm -->
     <limit effort="2.0" lower="${-roll}" upper="${roll}" velocity="0.5"/>
-    <!-- leaving 1/3 of the EquivalentWheelDiameter from front (origin is in the center of eq wheel, at the bottom of the chassis) -->
-    <origin xyz="0 0 ${-JointB}" rpy="${-pi/2} ${-pi/2} 0"/>
+    <origin xyz="0 0 -${JointB+WheelBase/2}" rpy="${-pi/2} ${-pi/2} 0"/>
     <axis xyz="1 0 0"/>
   </joint>
@@ -416,11 +415,11 @@
   <link name="joint_b_2_link">
     <visual>
-      <origin xyz="0 0 ${-(JointB-WheelBase/2-EquivalentWheelDiameter/6)/2}" />
-      <geometry>
-        <cylinder radius="${(ModuleWidth-2*TrackWidth-toll*2)/2}" length="${JointB-WheelBase/2-EquivalentWheelDiameter/6}"/>
-      </geometry>
-      <material name="JointColor"/>
-    </visual>
-    <xacro:inertial_cylinder mass="${JointBMass}" length="${JointB-WheelBase/2-EquivalentWheelDiameter/6}" radius="${(ModuleWidth-2*TrackWidth-toll*2)/2}">
+      <origin xyz="0 0 -${JointB/2}" />
+      <geometry>
+        <cylinder radius="${(ModuleWidth-2*TrackWidth-toll*2)/2}" length="${JointB}"/>
+      </geometry>
+      <material name="JointColor"/>
+    </visual>
+    <xacro:inertial_cylinder mass="${JointBMass}" length="${JointB}" radius="${(ModuleWidth-2*TrackWidth-toll*2)/2}">
       <origin xyz="0 0 ${-(JointB-WheelBase/2-EquivalentWheelDiameter/6)/2}" rpy="0 0 0"/>
     </xacro:inertial_cylinder>
@@ -436,5 +435,5 @@
     <limit effort="2.0" lower="${-roll}" upper="${roll}" velocity="0.5"/>
     <!-- leaving 1/3 of the EquivalentWheelDiameter from front (origin is in the center of eq wheel, at the bottom of the chassis) -->
-    <origin xyz="0 0 ${-JointB}" rpy="${-pi/2} ${-pi/2} 0"/>
+    <origin xyz="0 0 -${JointB+WheelBase/2}" rpy="${-pi/2} ${-pi/2} 0"/>
     <axis xyz="1 0 0"/>
   </joint>
@@ -630,11 +629,11 @@
   <link name="joint_b_3_link">
     <visual>
-      <origin xyz="0 0 ${-(JointB-WheelBase/2-EquivalentWheelDiameter/6)/2}" />
-      <geometry>
-        <cylinder radius="${(ModuleWidth-2*TrackWidth-toll*2)/2}" length="${JointB-WheelBase/2-EquivalentWheelDiameter/6}"/>
-      </geometry>
-      <material name="JointColor"/>
-    </visual>
-    <xacro:inertial_cylinder mass="${JointBMass}" length="${JointB-WheelBase/2-EquivalentWheelDiameter/6}" radius="${(ModuleWidth-2*TrackWidth-toll*2)/2}">
+      <origin xyz="0 0 -${JointB/2}" />
+      <geometry>
+        <cylinder radius="${(ModuleWidth-2*TrackWidth-toll*2)/2}" length="${JointB}"/>
+      </geometry>
+      <material name="JointColor"/>
+    </visual>
+    <xacro:inertial_cylinder mass="${JointBMass}" length="${JointB}" radius="${(ModuleWidth-2*TrackWidth-toll*2)/2}">
       <origin xyz="0 0 ${-(JointB-WheelBase/2-EquivalentWheelDiameter/6)/2}" rpy="0 0 0"/>
     </xacro:inertial_cylinder>
@@ -650,5 +649,5 @@
     <limit effort="2.0" lower="${-roll}" upper="${roll}" velocity="0.5"/>
     <!-- leaving 1/3 of the EquivalentWheelDiameter from front (origin is in the center of eq wheel, at the bottom of the chassis) -->
-    <origin xyz="0 0 ${-JointB}" rpy="${-pi/2} ${-pi/2} 0"/>
+    <origin xyz="0 0 -${JointB+WheelBase/2}" rpy="${-pi/2} ${-pi/2} 0"/>
     <axis xyz="1 0 0"/>
   </joint>
