Commit message: fix: rotate chassis joint axis to same reference

File: reseq_ros2/description/components.xacro (robot description, xacro)
@@ -1,4 +1,6 @@
 <?xml version="1.0"?>
 <robot xmlns:xacro="http://www.ros.org/wiki/xacro">
+  <xacro:include filename="inertial_macros.xacro" />
+  <xacro:include filename="reseq_parameters.xacro" />
   <xacro:macro name="chassis_joint_factory" params="id">
     <joint name="chassis${id}_joint" type="revolute">
@@ -7,5 +9,5 @@
       <!-- Effort in Nm -->
       <limit effort="2.0" lower="${-roll}" upper="${roll}" velocity="0.5"/>
-      <origin xyz="0 0 -${JointB+WheelBase/2}" rpy="${-pi/2} ${-pi/2} 0"/>
+      <origin xyz="-${JointB+WheelBase/2} 0 0" rpy="0 0 0"/>
       <axis xyz="1 0 0"/>
     </joint>
@@ -130,10 +132,11 @@
       <!-- Effort in Nm -->
       <limit effort="20.0" lower="${-pitch}" upper="${pitch}" velocity="0.5"/>
-      <origin xyz="${-WheelBase/2} 0 0" rpy="${pi/2} 0 0" />
-      <axis xyz="0 0 -1"/>
+      <origin xyz="${-WheelBase/2} 0 0" rpy="0 0 0" />
+      <axis xyz="0 1 0"/>
     </joint>
     <link name="joint_a_${id}_link">
       <!-- gearbox cilinder -->
       <visual>
+        <origin rpy="${pi/2} 0 0"/>
         <geometry>
           <cylinder radius="${JointDiameter/2}" length="${ModuleWidth-2*TrackWidth-toll*2}"/>
@@ -143,5 +146,5 @@
       <!-- horizontal shaft -->
       <visual>
-        <origin xyz="${-JointA/2} 0 0" />
+        <origin xyz="${-JointA/2} 0 0" rpy="${pi/2} 0 0"/>
         <geometry>
           <box size="${JointA} ${EquivalentWheelDiameter-2*JointABottomClearance} ${ModuleWidth-2*TrackWidth-toll*2}"/>
@@ -180,10 +183,10 @@
       <!-- Effort in Nm -->
       <limit effort="20.0" lower="${-yaw}" upper="${yaw}" velocity="0.5"/>
-      <origin xyz="${-JointA} 0 0" rpy="0 ${pi/2} 0" />
-      <axis xyz="0 1 0"/>
+      <origin xyz="${-JointA} 0 0" rpy="0 0 0" />
+      <axis xyz="0 0 1"/>
     </joint>
     <link name="joint_b_${id}_link">
       <visual>
-        <origin xyz="0 0 -${JointB/2}" />
+        <origin xyz="-${JointB/2} 0 0" rpy="0 ${pi/2} 0"/>
         <geometry>
           <cylinder radius="${(ModuleWidth-2*TrackWidth-toll*2)/2}" length="${JointB}"/>
@@ -196,3 +199,13 @@
     </link>
   </xacro:macro>
+  <link name="base_link" />
+  <joint name="chassis1_joint" type="fixed">
+    <parent link="base_link"/>
+    <child link="chassis1_link"/>
+    <!-- leaving 1/3 of the EquivalentWheelDiameter from front (origin is in the center of eq wheel, at the bottom of the chassis) -->
+    <origin xyz="0 0 ${(EquivalentWheelDiameter-2*ChassisTopAndBottomClearance)/2+ChassisTopAndBottomClearance}"/>
+  </joint>
+  <xacro:chassis id="1"/>
+  <xacro:chassis_joint_factory id="2"/>
+  <xacro:chassis id="2"/>
 </robot>

File: reseq_ros2/description/robot.urdf.xacro (robot description, xacro)
@@ -5,7 +5,7 @@
   <xacro:include filename="inertial_macros.xacro" />
   <xacro:include filename="reseq_parameters.xacro" />
-  <xacro:include filename="components.xacro"/>
-  <xacro:include filename="module_body.xacro" />
-  <!-- <xacro:include filename="reseq_body.xacro" /> -->
+  <!-- <xacro:include filename="components.xacro"/>
+  <xacro:include filename="module_body.xacro" /> -->
+  <xacro:include filename="reseq_body.xacro" />
   <!-- <xacro:include filename="reseq_arm_mk1.xacro" /> -->
   <!-- <xacro:include filename="lidar.xacro" /> -->

Commit message: fix: replicate collision automatically (temp)

File: reseq_ros2/description/components.xacro (robot description, xacro)
@@ -3,197 +3,208 @@
   <xacro:include filename="inertial_macros.xacro" />
   <xacro:include filename="reseq_parameters.xacro" />
+  <xacro:macro name="replicate_collision" params="**block">
+    <visual>
+      <xacro:insert_block name="block" />
+    </visual>
+    <collision>
+      <xacro:insert_block name="block" />
+    </collision>
+  </xacro:macro>
   <xacro:macro name="chassis_joint_factory" params="id">
     <joint name="chassis${id}_joint" type="revolute">
-      <parent link="joint_b_${id-1}_link"/>
-      <child link="chassis${id}_link"/>
+      <parent link="joint_b_${id-1}_link" />
+      <child link="chassis${id}_link" />
       <!-- Effort in Nm -->
-      <limit effort="2.0" lower="${-roll}" upper="${roll}" velocity="0.5"/>
-      <origin xyz="-${JointB+WheelBase/2} 0 0" rpy="0 0 0"/>
-      <axis xyz="1 0 0"/>
+      <limit effort="2.0" lower="${-roll}" upper="${roll}" velocity="0.5" />
+      <origin xyz="-${JointB+WheelBase/2} 0 0" rpy="0 0 0" />
+      <axis xyz="1 0 0" />
     </joint>
   </xacro:macro>
   <xacro:macro name="chassis" params="id">
     <link name="chassis${id}_link">
-      <visual>
-        <origin xyz="${EquivalentWheelDiameter/12+(toll+JointDiameter/2)/2} 0 0"/>
-        <geometry>
-          <!-- leaving 1/3 of the EquivalentWheelDiameter from front and toll from Joint and Tracks (for clearance) -->
-          <box size="${WheelBase-JointDiameter/2-toll+EquivalentWheelDiameter*2/3-EquivalentWheelDiameter/2} ${ModuleWidth-2*TrackWidth-2*toll} ${EquivalentWheelDiameter-2*ChassisTopAndBottomClearance}"/>
-        </geometry>
-        <material name="ChassisColor"/>
-      </visual>
-      <collision>
-        <origin xyz="${EquivalentWheelDiameter/12+(toll+JointDiameter/2)/2} 0 0"/>
-        <geometry>
-          <!-- leaving 1/3 of the EquivalentWheelDiameter from front and toll from Joint and Tracks (for clearance) -->
-          <box size="${WheelBase-JointDiameter/2-toll+EquivalentWheelDiameter*2/3-EquivalentWheelDiameter/2} ${ModuleWidth-2*TrackWidth-2*toll} ${EquivalentWheelDiameter-2*ChassisTopAndBottomClearance}"/>
-        </geometry>
-      </collision>
-      <xacro:inertial_box mass="${ChassisMass}" x="${WheelBase-JointDiameter/2-toll+EquivalentWheelDiameter*2/3-EquivalentWheelDiameter/2}" y="${ModuleWidth-2*TrackWidth-2*toll}" z="${EquivalentWheelDiameter-2*ChassisTopAndBottomClearance}">
-        <origin xyz="${EquivalentWheelDiameter/12+(toll+JointDiameter/2)/2} 0 0" rpy="0 0 0"/>
+      <xacro:replicate_collision>
+        <visual>
+          <origin xyz="${EquivalentWheelDiameter/12+(toll+JointDiameter/2)/2} 0 0" />
+          <geometry>
+            <!-- leaving 1/3 of the EquivalentWheelDiameter from front and toll from Joint and
+            Tracks (for clearance) -->
+            <box
+              size="${WheelBase-JointDiameter/2-toll+EquivalentWheelDiameter*2/3-EquivalentWheelDiameter/2} ${ModuleWidth-2*TrackWidth-2*toll} ${EquivalentWheelDiameter-2*ChassisTopAndBottomClearance}" />
+          </geometry>
+          <material name="ChassisColor" />
+        </visual>
+      </xacro:replicate_collision>
+      <xacro:inertial_box mass="${ChassisMass}"
+        x="${WheelBase-JointDiameter/2-toll+EquivalentWheelDiameter*2/3-EquivalentWheelDiameter/2}"
+        y="${ModuleWidth-2*TrackWidth-2*toll}"
+        z="${EquivalentWheelDiameter-2*ChassisTopAndBottomClearance}">
+        <origin xyz="${EquivalentWheelDiameter/12+(toll+JointDiameter/2)/2} 0 0" rpy="0 0 0" />
       </xacro:inertial_box>
     </link>
     <!-- LEFT FRONT WHEEL 1-->
     <joint name="left_front_wheel_${id}_joint" type="continuous">
-      <parent link="chassis${id}_link"/>
-      <child link="left_front_wheel_${id}_link"/>
+      <parent link="chassis${id}_link" />
+      <child link="left_front_wheel_${id}_link" />
       <origin xyz="${WheelBase/2} ${ModuleWidth/2-TrackWidth/2} 0" rpy="-${pi/2} 0 0" />
-      <axis xyz="0 0 1"/>
+      <axis xyz="0 0 1" />
     </joint>
     <link name="left_front_wheel_${id}_link">
       <visual>
         <geometry>
-          <cylinder radius="${EquivalentWheelDiameter/2}" length="${TrackWidth}"/>
-        </geometry>
-        <material name="WheelColor"/>
-      </visual>
-      <collision>
-        <geometry>
-          <cylinder radius="${EquivalentWheelDiameter/2}" length="${TrackWidth}"/>
-        </geometry>
-      </collision>
-      <xacro:inertial_cylinder mass="${WheelMass}" length="${TrackWidth}" radius="${EquivalentWheelDiameter/2}">
-        <origin xyz="0 0 0" rpy="0 0 0"/>
+          <cylinder radius="${EquivalentWheelDiameter/2}" length="${TrackWidth}" />
+        </geometry>
+        <material name="WheelColor" />
+      </visual>
+      <collision>
+        <geometry>
+          <cylinder radius="${EquivalentWheelDiameter/2}" length="${TrackWidth}" />
+        </geometry>
+      </collision>
+      <xacro:inertial_cylinder mass="${WheelMass}" length="${TrackWidth}"
+        radius="${EquivalentWheelDiameter/2}">
+        <origin xyz="0 0 0" rpy="0 0 0" />
       </xacro:inertial_cylinder>
     </link>
     <!-- RIGHT FRONT WHEEL 1-->
     <joint name="right_front_wheel_${id}_joint" type="continuous">
-      <parent link="chassis${id}_link"/>
-      <child link="right_front_wheel_${id}_link"/>
+      <parent link="chassis${id}_link" />
+      <child link="right_front_wheel_${id}_link" />
       <origin xyz="${WheelBase/2} ${-ModuleWidth/2+TrackWidth/2} 0" rpy="${pi/2} 0 0" />
-      <axis xyz="0 0 -1"/>
+      <axis xyz="0 0 -1" />
     </joint>
     <link name="right_front_wheel_${id}_link">
       <visual>
         <geometry>
-          <cylinder radius="${EquivalentWheelDiameter/2}" length="${TrackWidth}"/>
-        </geometry>
-        <material name="WheelColor"/>
-      </visual>
-      <collision>
-        <geometry>
-          <cylinder radius="${EquivalentWheelDiameter/2}" length="${TrackWidth}"/>
-        </geometry>
-      </collision>
-      <xacro:inertial_cylinder mass="${WheelMass}" length="${TrackWidth}" radius="${EquivalentWheelDiameter/2}">
-        <origin xyz="0 0 0" rpy="0 0 0"/>
+          <cylinder radius="${EquivalentWheelDiameter/2}" length="${TrackWidth}" />
+        </geometry>
+        <material name="WheelColor" />
+      </visual>
+      <collision>
+        <geometry>
+          <cylinder radius="${EquivalentWheelDiameter/2}" length="${TrackWidth}" />
+        </geometry>
+      </collision>
+      <xacro:inertial_cylinder mass="${WheelMass}" length="${TrackWidth}"
+        radius="${EquivalentWheelDiameter/2}">
+        <origin xyz="0 0 0" rpy="0 0 0" />
       </xacro:inertial_cylinder>
     </link>
     <!-- LEFT BACK WHEEL 1-->
     <joint name="left_back_wheel_${id}_joint" type="continuous">
-      <parent link="chassis${id}_link"/>
-      <child link="left_back_wheel_${id}_link"/>
+      <parent link="chassis${id}_link" />
+      <child link="left_back_wheel_${id}_link" />
       <origin xyz="${-WheelBase/2} ${ModuleWidth/2-TrackWidth/2} 0" rpy="-${pi/2} 0 0" />
-      <axis xyz="0 0 1"/>
+      <axis xyz="0 0 1" />
     </joint>
     <link name="left_back_wheel_${id}_link">
       <visual>
         <geometry>
-          <cylinder radius="${EquivalentWheelDiameter/2}" length="${TrackWidth}"/>
-        </geometry>
-        <material name="WheelColor"/>
-      </visual>
-      <collision>
-        <geometry>
-          <cylinder radius="${EquivalentWheelDiameter/2}" length="${TrackWidth}"/>
-        </geometry>
-      </collision>
-      <xacro:inertial_cylinder mass="${WheelMass}" length="${TrackWidth}" radius="${EquivalentWheelDiameter/2}">
-        <origin xyz="0 0 0" rpy="0 0 0"/>
+          <cylinder radius="${EquivalentWheelDiameter/2}" length="${TrackWidth}" />
+        </geometry>
+        <material name="WheelColor" />
+      </visual>
+      <collision>
+        <geometry>
+          <cylinder radius="${EquivalentWheelDiameter/2}" length="${TrackWidth}" />
+        </geometry>
+      </collision>
+      <xacro:inertial_cylinder mass="${WheelMass}" length="${TrackWidth}"
+        radius="${EquivalentWheelDiameter/2}">
+        <origin xyz="0 0 0" rpy="0 0 0" />
       </xacro:inertial_cylinder>
     </link>
     <!-- RIGHT BACK WHEEL 1-->
     <joint name="right_back_wheel_${id}_joint" type="continuous">
-      <parent link="chassis${id}_link"/>
-      <child link="right_back_wheel_${id}_link"/>
+      <parent link="chassis${id}_link" />
+      <child link="right_back_wheel_${id}_link" />
       <origin xyz="${-WheelBase/2} ${-ModuleWidth/2+TrackWidth/2} 0" rpy="${pi/2} 0 0" />
-      <axis xyz="0 0 -1"/>
+      <axis xyz="0 0 -1" />
     </joint>
     <link name="right_back_wheel_${id}_link">
       <visual>
         <geometry>
-          <cylinder radius="${EquivalentWheelDiameter/2}" length="${TrackWidth}"/>
-        </geometry>
-        <material name="WheelColor"/>
-      </visual>
-      <collision>
-        <geometry>
-          <cylinder radius="${EquivalentWheelDiameter/2}" length="${TrackWidth}"/>
-        </geometry>
-      </collision>
-      <xacro:inertial_cylinder mass="${WheelMass}" length="${TrackWidth}" radius="${EquivalentWheelDiameter/2}">
-        <origin xyz="0 0 0" rpy="0 0 0"/>
+          <cylinder radius="${EquivalentWheelDiameter/2}" length="${TrackWidth}" />
+        </geometry>
+        <material name="WheelColor" />
+      </visual>
+      <collision>
+        <geometry>
+          <cylinder radius="${EquivalentWheelDiameter/2}" length="${TrackWidth}" />
+        </geometry>
+      </collision>
+      <xacro:inertial_cylinder mass="${WheelMass}" length="${TrackWidth}"
+        radius="${EquivalentWheelDiameter/2}">
+        <origin xyz="0 0 0" rpy="0 0 0" />
       </xacro:inertial_cylinder>
     </link>
     <!-- JointA 1-->
     <joint name="joint_a_${id}_joint" type="revolute">
-      <parent link="chassis${id}_link"/>
-      <child link="joint_a_${id}_link"/>
+      <parent link="chassis${id}_link" />
+      <child link="joint_a_${id}_link" />
       <!-- Effort in Nm -->
-      <limit effort="20.0" lower="${-pitch}" upper="${pitch}" velocity="0.5"/>
+      <limit effort="20.0" lower="${-pitch}" upper="${pitch}" velocity="0.5" />
       <origin xyz="${-WheelBase/2} 0 0" rpy="0 0 0" />
-      <axis xyz="0 1 0"/>
+      <axis xyz="0 1 0" />
     </joint>
     <link name="joint_a_${id}_link">
       <!-- gearbox cilinder -->
-      <visual>
-        <origin rpy="${pi/2} 0 0"/>
-        <geometry>
-          <cylinder radius="${JointDiameter/2}" length="${ModuleWidth-2*TrackWidth-toll*2}"/>
-        </geometry>
-        <material name="JointColor"/>
-      </visual>
+      <xacro:replicate_collision>
+        <visual>
+          <origin rpy="${pi/2} 0 0" />
+          <geometry>
+            <cylinder radius="${JointDiameter/2}" length="${ModuleWidth-2*TrackWidth-toll*2}" />
+          </geometry>
+          <material name="JointColor" />
+        </visual>
+      </xacro:replicate_collision>
       <!-- horizontal shaft -->
-      <visual>
-        <origin xyz="${-JointA/2} 0 0" rpy="${pi/2} 0 0"/>
-        <geometry>
-          <box size="${JointA} ${EquivalentWheelDiameter-2*JointABottomClearance} ${ModuleWidth-2*TrackWidth-toll*2}"/>
-        </geometry>
-        <material name="JointColor"/>
-      </visual>
+      <xacro:replicate_collision>
+        <visual>
+          <origin xyz="${-JointA/2} 0 0" rpy="${pi/2} 0 0" />
+          <geometry>
+            <box
+              size="${JointA} ${EquivalentWheelDiameter-2*JointABottomClearance} ${ModuleWidth-2*TrackWidth-toll*2}" />
+          </geometry>
+          <material name="JointColor" />
+        </visual>
+      </xacro:replicate_collision>
       <!-- to hide space wile rotating -->
-      <visual>
-        <origin xyz="${-JointA} 0 0" />
-        <geometry>
-          <sphere radius="${(ModuleWidth-2*TrackWidth-toll*2)/2}"/>
-        </geometry>
-        <material name="JointColor"/>
-      </visual>
-      <!-- gearbox cilinder -->
-      <collision>
-        <geometry>
-          <cylinder radius="${JointDiameter/2}" length="${ModuleWidth-2*TrackWidth-toll*2}"/>
-        </geometry>
-      </collision>
-      <!-- horizontal shaft -->
-      <collision>
-        <origin xyz="${-JointA/2} 0 0" />
-        <geometry>
-          <box size="${JointA} ${EquivalentWheelDiameter-2*JointABottomClearance} ${ModuleWidth-2*TrackWidth-toll*2}"/>
-        </geometry>
-      </collision>
-      <xacro:inertial_box mass="${JointAMass}" x="${JointA}" y="${EquivalentWheelDiameter-2*JointABottomClearance}" z="${ModuleWidth-2*TrackWidth-toll*2}">
-        <origin xyz="${-JointA/2} 0 0" rpy="0 0 0"/>
+      <xacro:replicate_collision>
+        <visual>
+          <origin xyz="${-JointA} 0 0" />
+          <geometry>
+            <sphere radius="${(ModuleWidth-2*TrackWidth-toll*2)/2}" />
+          </geometry>
+          <material name="JointColor" />
+        </visual>
+      </xacro:replicate_collision>
+      <xacro:inertial_box mass="${JointAMass}" x="${JointA}"
+        y="${EquivalentWheelDiameter-2*JointABottomClearance}"
+        z="${ModuleWidth-2*TrackWidth-toll*2}">
+        <origin xyz="${-JointA/2} 0 0" rpy="0 0 0" />
       </xacro:inertial_box>
     </link>
     <!-- JointB 1-->
     <joint name="joint_b_${id}_joint" type="revolute">
-      <parent link="joint_a_${id}_link"/>
-      <child link="joint_b_${id}_link"/>
+      <parent link="joint_a_${id}_link" />
+      <child link="joint_b_${id}_link" />
       <!-- Effort in Nm -->
-      <limit effort="20.0" lower="${-yaw}" upper="${yaw}" velocity="0.5"/>
+      <limit effort="20.0" lower="${-yaw}" upper="${yaw}" velocity="0.5" />
       <origin xyz="${-JointA} 0 0" rpy="0 0 0" />
-      <axis xyz="0 0 1"/>
+      <axis xyz="0 0 1" />
     </joint>
     <link name="joint_b_${id}_link">
-      <visual>
-        <origin xyz="-${JointB/2} 0 0" rpy="0 ${pi/2} 0"/>
-        <geometry>
-          <cylinder radius="${(ModuleWidth-2*TrackWidth-toll*2)/2}" length="${JointB}"/>
-        </geometry>
-        <material name="JointColor"/>
-      </visual>
-      <xacro:inertial_cylinder mass="${JointBMass}" length="${JointB}" radius="${(ModuleWidth-2*TrackWidth-toll*2)/2}">
-        <origin xyz="0 0 ${-(JointB-WheelBase/2-EquivalentWheelDiameter/6)/2}" rpy="0 0 0"/>
+      <xacro:replicate_collision>
+        <visual>
+          <origin xyz="-${JointB/2} 0 0" rpy="0 ${pi/2} 0" />
+          <geometry>
+            <cylinder radius="${(ModuleWidth-2*TrackWidth-toll*2)/2}" length="${JointB}" />
+          </geometry>
+          <material name="JointColor" />
+        </visual>
+      </xacro:replicate_collision>
+      <xacro:inertial_cylinder mass="${JointBMass}" length="${JointB}"
+        radius="${(ModuleWidth-2*TrackWidth-toll*2)/2}">
+        <origin xyz="0 0 ${-(JointB-WheelBase/2-EquivalentWheelDiameter/6)/2}" rpy="0 0 0" />
       </xacro:inertial_cylinder>
     </link>
@@ -201,11 +212,13 @@
   <link name="base_link" />
   <joint name="chassis1_joint" type="fixed">
-    <parent link="base_link"/>
-    <child link="chassis1_link"/>
-    <!-- leaving 1/3 of the EquivalentWheelDiameter from front (origin is in the center of eq wheel, at the bottom of the chassis) -->
-    <origin xyz="0 0 ${(EquivalentWheelDiameter-2*ChassisTopAndBottomClearance)/2+ChassisTopAndBottomClearance}"/>
+    <parent link="base_link" />
+    <child link="chassis1_link" />
+    <!-- leaving 1/3 of the EquivalentWheelDiameter from front (origin is in the center of eq wheel,
+    at the bottom of the chassis) -->
+    <origin
+      xyz="0 0 ${(EquivalentWheelDiameter-2*ChassisTopAndBottomClearance)/2+ChassisTopAndBottomClearance}" />
   </joint>
-  <xacro:chassis id="1"/>
-  <xacro:chassis_joint_factory id="2"/>
-  <xacro:chassis id="2"/>
+  <xacro:chassis id="1" />
+  <xacro:chassis_joint_factory id="2" />
+  <xacro:chassis id="2" />
 </robot>
