Commit message: feat: reverse joint between chassis (draft)

File: reseq_ros2/description/components.xacro (robot description, xacro)
@@ -12,11 +12,80 @@
   </xacro:macro>
   <xacro:macro name="chassis_joint_factory" params="id">
-    <joint name="chassis${id}_joint" type="revolute">
-      <parent link="joint_b_${id-1}_link" />
-      <child link="chassis${id}_link" />
+    <!-- JointR -->
+    <joint name="joint_r_${id}_joint" type="revolute">
+      <parent link="chassis${id-1}_link" />
+      <child link="joint_r_${id}_link" />
       <!-- Effort in Nm -->
       <limit effort="2.0" lower="${-roll}" upper="${roll}" velocity="0.5" />
-      <origin xyz="-${JointB+WheelBase/2} 0 0" rpy="0 0 0" />
+      <origin xyz="-${WheelBase/2} 0 0" rpy="0 0 0" />
       <axis xyz="1 0 0" />
+    </joint>
+    <link name="joint_r_${id}_link">
+      <xacro:replicate_collision>
+        <visual>
+          <origin xyz="-${JointB/2} 0 0" rpy="0 ${pi/2} 0" />
+          <geometry>
+            <cylinder radius="${(ModuleWidth-2*TrackWidth-toll*2)/2}" length="${JointB}" />
+          </geometry>
+          <material name="JointColor" />
+        </visual>
+      </xacro:replicate_collision>
+    </link>
+    <!-- JointY -->
+    <joint name="joint_y_${id}_joint" type="revolute">
+      <parent link="joint_r_${id}_link" />
+      <child link="joint_y_${id}_link" />
+      <!-- Effort in Nm -->
+      <limit effort="20.0" lower="${-yaw}" upper="${yaw}" velocity="0.5" />
+      <origin xyz="-${JointB} 0 0" rpy="0 0 0" />
+      <axis xyz="0 0 1" />
+    </joint>
+    <link name="joint_y_${id}_link">
+      <!-- to hide space wile rotating -->
+      <xacro:replicate_collision>
+        <visual>
+          <geometry>
+            <sphere radius="${(ModuleWidth-2*TrackWidth-toll*2)/2}" />
+          </geometry>
+          <material name="JointColor" />
+        </visual>
+      </xacro:replicate_collision>
+      <!-- horizontal shaft -->
+      <xacro:replicate_collision>
+        <visual>
+          <origin xyz="-${JointA/2} 0 0" rpy="${pi/2} 0 0" />
+          <geometry>
+            <box
+              size="${JointA} ${EquivalentWheelDiameter-2*JointABottomClearance} ${ModuleWidth-2*TrackWidth-toll*2}" />
+          </geometry>
+          <material name="JointColor" />
+        </visual>
+      </xacro:replicate_collision>
+    </link>
+    <!-- JointP -->
+    <joint name="joint_p_${id}_joint" type="revolute">
+      <parent link="joint_y_${id}_link" />
+      <child link="joint_p_${id}_link" />
+      <!-- Effort in Nm -->
+      <limit effort="20.0" lower="${-pitch}" upper="${pitch}" velocity="0.5" />
+      <origin xyz="${-JointA} 0 0" rpy="0 0 0" />
+      <axis xyz="0 1 0" />
+    </joint>
+    <link name="joint_p_${id}_link">
+      <!-- gearbox cilinder -->
+      <xacro:replicate_collision>
+        <visual>
+          <origin rpy="${pi/2} 0 0" />
+          <geometry>
+            <cylinder radius="${JointDiameter/2}" length="${ModuleWidth-2*TrackWidth-toll*2}" />
+          </geometry>
+          <material name="JointColor" />
+        </visual>
+      </xacro:replicate_collision>
+    </link>
+    <joint name="chassis${id}_joint" type="fixed">
+      <parent link="joint_p_${id}_link" />
+      <child link="chassis${id}_link" />
+      <origin xyz="${-WheelBase/2} 0 0" rpy="0 0 0" />
     </joint>
   </xacro:macro>
@@ -25,5 +94,5 @@
       <xacro:replicate_collision>
         <visual>
-          <origin xyz="${EquivalentWheelDiameter/12+(toll+JointDiameter/2)/2} 0 0" />
+          <origin xyz="-${EquivalentWheelDiameter/12+(toll+JointDiameter/2)/2} 0 0" />
           <geometry>
             <!-- leaving 1/3 of the EquivalentWheelDiameter from front and toll from Joint and
@@ -136,75 +205,4 @@
         radius="${EquivalentWheelDiameter/2}">
         <origin xyz="0 0 0" rpy="0 0 0" />
-      </xacro:inertial_cylinder>
-    </link>
-    <!-- JointA 1-->
-    <joint name="joint_a_${id}_joint" type="revolute">
-      <parent link="chassis${id}_link" />
-      <child link="joint_a_${id}_link" />
-      <!-- Effort in Nm -->
-      <limit effort="20.0" lower="${-pitch}" upper="${pitch}" velocity="0.5" />
-      <origin xyz="${-WheelBase/2} 0 0" rpy="0 0 0" />
-      <axis xyz="0 1 0" />
-    </joint>
-    <link name="joint_a_${id}_link">
-      <!-- gearbox cilinder -->
-      <xacro:replicate_collision>
-        <visual>
-          <origin rpy="${pi/2} 0 0" />
-          <geometry>
-            <cylinder radius="${JointDiameter/2}" length="${ModuleWidth-2*TrackWidth-toll*2}" />
-          </geometry>
-          <material name="JointColor" />
-        </visual>
-      </xacro:replicate_collision>
-      <!-- horizontal shaft -->
-      <xacro:replicate_collision>
-        <visual>
-          <origin xyz="${-JointA/2} 0 0" rpy="${pi/2} 0 0" />
-          <geometry>
-            <box
-              size="${JointA} ${EquivalentWheelDiameter-2*JointABottomClearance} ${ModuleWidth-2*TrackWidth-toll*2}" />
-          </geometry>
-          <material name="JointColor" />
-        </visual>
-      </xacro:replicate_collision>
-      <!-- to hide space wile rotating -->
-      <xacro:replicate_collision>
-        <visual>
-          <origin xyz="${-JointA} 0 0" />
-          <geometry>
-            <sphere radius="${(ModuleWidth-2*TrackWidth-toll*2)/2}" />
-          </geometry>
-          <material name="JointColor" />
-        </visual>
-      </xacro:replicate_collision>
-      <xacro:inertial_box mass="${JointAMass}" x="${JointA}"
-        y="${EquivalentWheelDiameter-2*JointABottomClearance}"
-        z="${ModuleWidth-2*TrackWidth-toll*2}">
-        <origin xyz="${-JointA/2} 0 0" rpy="0 0 0" />
-      </xacro:inertial_box>
-    </link>
-    <!-- JointB 1-->
-    <joint name="joint_b_${id}_joint" type="revolute">
-      <parent link="joint_a_${id}_link" />
-      <child link="joint_b_${id}_link" />
-      <!-- Effort in Nm -->
-      <limit effort="20.0" lower="${-yaw}" upper="${yaw}" velocity="0.5" />
-      <origin xyz="${-JointA} 0 0" rpy="0 0 0" />
-      <axis xyz="0 0 1" />
-    </joint>
-    <link name="joint_b_${id}_link">
-      <xacro:replicate_collision>
-        <visual>
-          <origin xyz="-${JointB/2} 0 0" rpy="0 ${pi/2} 0" />
-          <geometry>
-            <cylinder radius="${(ModuleWidth-2*TrackWidth-toll*2)/2}" length="${JointB}" />
-          </geometry>
-          <material name="JointColor" />
-        </visual>
-      </xacro:replicate_collision>
-      <xacro:inertial_cylinder mass="${JointBMass}" length="${JointB}"
-        radius="${(ModuleWidth-2*TrackWidth-toll*2)/2}">
-        <origin xyz="0 0 ${-(JointB-WheelBase/2-EquivalentWheelDiameter/6)/2}" rpy="0 0 0" />
       </xacro:inertial_cylinder>
     </link>

Commit message: docs: document the macros for the chassis creation

File: reseq_ros2/description/components.xacro (robot description, xacro)
@@ -3,4 +3,9 @@
   <xacro:include filename="inertial_macros.xacro" />
   <xacro:include filename="reseq_parameters.xacro" />
+  <!--
+    Replicates the visual block inside the collision block to avoid code
+    duplication until the use of 3D meshes for the visuals
+    @param **block: the <visual/> block to replicate
+   -->
   <xacro:macro name="replicate_collision" params="**block">
     <visual>
@@ -11,4 +16,10 @@
     </collision>
   </xacro:macro>
+  <!--
+    Creates the joint between two consecutive chassis. It assumes that two
+    consecutive chassis have a consecutive id. This macro must be called between
+    the definition of the two chassis
+    @param id: the id of the joint (which is assumed part of the chassis behind)
+   -->
   <xacro:macro name="chassis_joint_factory" params="id">
     <!-- JointR -->
@@ -90,4 +101,8 @@
     </joint>
   </xacro:macro>
+  <!--
+    Defines the current chassis
+    @param id: the id of the chassis (starting from 1)
+  -->
   <xacro:macro name="chassis" params="id">
     <link name="chassis${id}_link">
