Commit message: fix: fix include path

File: reseq_ros2/description/reseq_parameters.xacro (robot description, xacro)
@@ -2,5 +2,5 @@
 <robot xmlns:xacro="http://www.ros.org/wiki/xacro">
   <!-- import values from config.yaml file -->
-  <xacro:property name="config_yaml_path" value="../../../../../src/reseq_ros2/config/config_mk2.yaml" />
+  <xacro:property name="config_yaml_path" value="$(find reseq_ros2)/config/config_mk2.yaml" />
   <xacro:property name="config_yaml_file" value="${xacro.load_yaml(config_yaml_path)}"/>
   <xacro:property name="a_yaml" value="${config_yaml_file['dimensions']['a']}" />

File: reseq_ros2/description/robot.urdf.xacro (robot description, xacro)
@@ -8,4 +8,3 @@
   <xacro:include filename="reseq_arm_mk1.xacro" />
   <xacro:include filename="lidar.xacro" />
-  <xacro:include filename="ros2_control.xacro" />
 </robot>

Commit message: Update reseq_parameters with mk1 param

File: reseq_ros2/description/reseq_parameters.xacro (robot description, xacro)
@@ -9,18 +9,18 @@
   <!-- See 'Parameters.pdf' pdf for parameters meaning (when it will exist ;) ) -->
   <!-- All values are in meters, radiants, kg -->
-  <xacro:property name="toll" value="0.01"/>
+  <xacro:property name="toll" value="0.001"/>
   <!-- chassis related -->
-  <xacro:property name="WheelBase" value="0.25"/>
+  <xacro:property name="WheelBase" value="0.137"/>
   <xacro:property name="EquivalentWheelDiameter" value="${r_eq_yaml*2}"/>
-  <xacro:property name="ModuleWidth" value="0.2"/>
-  <xacro:property name="TrackWidth" value="0.08"/>
-  <xacro:property name="ChassisTopAndBottomClearance" value="0.02"/>
+  <xacro:property name="ModuleWidth" value="0.27"/>
+  <xacro:property name="TrackWidth" value="0.052"/>
+  <xacro:property name="ChassisTopAndBottomClearance" value="0.013"/>
   <xacro:property name="WheelMass" value="0.1"/>
   <xacro:property name="ChassisMass" value="2.5"/>
   <!-- joint related -->
-  <xacro:property name="JointDiameter" value="0.07"/>
+  <xacro:property name="JointDiameter" value="0.048"/>
   <xacro:property name="JointA" value="${a_yaml-WheelBase/2}"/>
   <xacro:property name="JointB" value="${b_yaml-WheelBase/2}"/>
-  <xacro:property name="JointABottomClearance" value="0.04"/>
+  <xacro:property name="JointABottomClearance" value="0.013"/>
   <xacro:property name="pitch" value="${pi/2}"/>
   <xacro:property name="roll" value="${pi/2}"/>
@@ -29,8 +29,8 @@
   <xacro:property name="JointBMass" value="0.05"/>
   <!-- arm related -->
-  <xacro:property name="ForkThickness" value="0.01"/>
-  <xacro:property name="ForkHeight" value="0.03"/>
+  <xacro:property name="ForkThickness" value="0.02"/>
+  <xacro:property name="ForkHeight" value="0.05"/>
   <xacro:property name="JetsonHolderLength" value="0.158"/>
-  <xacro:property name="JetsonHolderWidth" value="0.09"/>
+  <xacro:property name="JetsonHolderWidth" value="0.085"/>
   <!-- Rvitz colors (for Gazebo ones change in single files) (from 0 to 1) -->
   <material name="ChassisColor">

Commit message: fix: define parameters in config file

File: reseq_ros2/description/reseq_parameters.xacro (robot description, xacro)
@@ -2,35 +2,35 @@
 <robot xmlns:xacro="http://www.ros.org/wiki/xacro">
   <!-- import values from config.yaml file -->
-  <xacro:property name="config_yaml_path" value="$(find reseq_ros2)/config/config_mk2.yaml" />
-  <xacro:property name="config_yaml_file" value="${xacro.load_yaml(config_yaml_path)}"/>
-  <xacro:property name="a_yaml" value="${config_yaml_file['dimensions']['a']}" />
-  <xacro:property name="b_yaml" value="${config_yaml_file['dimensions']['b']}" />
-  <xacro:property name="r_eq_yaml" value="${config_yaml_file['dimensions']['r_eq']}" />
+  <xacro:property name="config_yaml_path" value="$(find reseq_ros2)/config/config_mk1.yaml" />
+  <xacro:property name="config" value="${xacro.load_yaml(config_yaml_path)}"/>
+  <xacro:property name="a" value="${config['dimensions']['a']}" />
+  <xacro:property name="b" value="${config['dimensions']['b']}" />
+  <xacro:property name="r_eq" value="${config['dimensions']['r_eq']}" />
   <!-- See 'Parameters.pdf' pdf for parameters meaning (when it will exist ;) ) -->
   <!-- All values are in meters, radiants, kg -->
   <xacro:property name="toll" value="0.001"/>
   <!-- chassis related -->
-  <xacro:property name="WheelBase" value="0.137"/>
-  <xacro:property name="EquivalentWheelDiameter" value="${r_eq_yaml*2}"/>
-  <xacro:property name="ModuleWidth" value="0.27"/>
-  <xacro:property name="TrackWidth" value="0.052"/>
-  <xacro:property name="ChassisTopAndBottomClearance" value="0.013"/>
-  <xacro:property name="WheelMass" value="0.1"/>
-  <xacro:property name="ChassisMass" value="2.5"/>
+  <xacro:property name="WheelBase" value="${config['xacro']['WheelBase']}"/>
+  <xacro:property name="EquivalentWheelDiameter" value="${r_eq*2}"/>
+  <xacro:property name="ModuleWidth" value="${config['xacro']['ModuleWidth']}"/>
+  <xacro:property name="TrackWidth" value="${config['xacro']['TrackWidth']}"/>
+  <xacro:property name="ChassisTopAndBottomClearance" value="${config['xacro']['ChassisTopAndBottomClearance']}"/>
+  <xacro:property name="WheelMass" value="${config['xacro']['WheelMass']}"/>
+  <xacro:property name="ChassisMass" value="${config['xacro']['ChassisMass']}"/>
   <!-- joint related -->
-  <xacro:property name="JointDiameter" value="0.048"/>
-  <xacro:property name="JointA" value="${a_yaml-WheelBase/2}"/>
-  <xacro:property name="JointB" value="${b_yaml-WheelBase/2}"/>
-  <xacro:property name="JointABottomClearance" value="0.013"/>
+  <xacro:property name="JointDiameter" value="${config['xacro']['JointDiameter']}"/>
+  <xacro:property name="JointA" value="${a-WheelBase/2}"/>
+  <xacro:property name="JointB" value="${b-WheelBase/2}"/>
+  <xacro:property name="JointABottomClearance" value="${config['xacro']['JointABottomClearance']}"/>
   <xacro:property name="pitch" value="${pi/2}"/>
   <xacro:property name="roll" value="${pi/2}"/>
   <xacro:property name="yaw" value="${pi/4}"/>
-  <xacro:property name="JointAMass" value="0.1"/>
-  <xacro:property name="JointBMass" value="0.05"/>
-  <!-- arm related -->
-  <xacro:property name="ForkThickness" value="0.02"/>
-  <xacro:property name="ForkHeight" value="0.05"/>
-  <xacro:property name="JetsonHolderLength" value="0.158"/>
-  <xacro:property name="JetsonHolderWidth" value="0.085"/>
+  <xacro:property name="JointAMass" value="${config['xacro']['JointAMass']}"/>
+  <xacro:property name="JointBMass" value="${config['xacro']['JointBMass']}"/>
+  <!-- arm related (only mk1) -->
+  <xacro:property name="ForkThickness" value="${config['xacro']['ForkThickness']}"/>
+  <xacro:property name="ForkHeight" value="${config['xacro']['ForkHeight']}"/>
+  <xacro:property name="JetsonHolderLength" value="${config['xacro']['JetsonHolderLength']}"/>
+  <xacro:property name="JetsonHolderWidth" value="${config['xacro']['JetsonHolderWidth']}"/>
   <!-- Rvitz colors (for Gazebo ones change in single files) (from 0 to 1) -->
   <material name="ChassisColor">

Commit message: fix: fix organizations of parameters in the config files

File: reseq_ros2/description/reseq_parameters.xacro (robot description, xacro)
@@ -2,9 +2,10 @@
 <robot xmlns:xacro="http://www.ros.org/wiki/xacro">
   <!-- import values from config.yaml file -->
-  <xacro:property name="config_yaml_path" value="$(find reseq_ros2)/config/config_mk1.yaml" />
-  <xacro:property name="config" value="${xacro.load_yaml(config_yaml_path)}"/>
-  <xacro:property name="a" value="${config['dimensions']['a']}" />
-  <xacro:property name="b" value="${config['dimensions']['b']}" />
-  <xacro:property name="r_eq" value="${config['dimensions']['r_eq']}" />
+  <xacro:arg name="config_path" default="$(find reseq_ros2)/config/reseq_mk1_can.yaml"/>
+  <xacro:property name="config_path_prop" value="$(arg config_path)"/>
+  <xacro:property name="config" value="${xacro.load_yaml(config_path_prop)}"/>
+  <xacro:property name="a" value="${config['agevar_consts']['a']}" />
+  <xacro:property name="b" value="${config['agevar_consts']['b']}" />
+  <xacro:property name="r_eq" value="${config['agevar_consts']['r_eq']}" />
   <!-- See 'Parameters.pdf' pdf for parameters meaning (when it will exist ;) ) -->
   <!-- All values are in meters, radiants, kg -->

Commit message: fix: move num_modules to main part of YAML file

File: reseq_ros2/description/reseq_parameters.xacro (robot description, xacro)
@@ -12,5 +12,5 @@
   <xacro:property name="toll" value="0.001"/>
   <!-- chassis related -->
-  <xacro:property name="NumModules" value="${config['xacro']['NumModules']}"/>
+  <xacro:property name="NumModules" value="${config['num_modules']}"/>
   <xacro:property name="WheelBase" value="${config['xacro']['WheelBase']}"/>
   <xacro:property name="EquivalentWheelDiameter" value="${r_eq*2}"/>

Commit message: feat: add new arm parameters

File: reseq_ros2/description/reseq_parameters.xacro (robot description, xacro)
@@ -36,4 +36,12 @@
   <xacro:property name="JetsonHolderLength" value="${config['xacro']['JetsonHolderLength']}"/>
   <xacro:property name="JetsonHolderWidth" value="${config['xacro']['JetsonHolderWidth']}"/>
+  <xacro:property name="CylinderOnJetsonLength" value="${config['xacro']['CylinderOnJetsonLength']}"/>
+  <xacro:property name="CylinderOnJetsonRadius" value="${config['xacro']['CylinderOnJetsonRadius']}"/>
+  <xacro:property name="CylinderOnJetsonShift" value="${config['xacro']['CylinderOnJetsonShift']}"/>
+  <xacro:property name="CylinderRealsenseLength" value="${config['xacro']['CylinderRealsenseLength']}"/>
+  <xacro:property name="CylinderRealsenseRadius" value="${config['xacro']['CylinderRealsenseRadius']}"/>
+  <xacro:property name="RealsenseLength" value="${config['xacro']['RealsenseLength']}"/>
+  <xacro:property name="RealsenseWidth" value="${config['xacro']['RealsenseWidth']}"/>
+  <xacro:property name="RealsenseOriginSystem" value="${config['xacro']['RealsenseOriginSystem']}"/>
   <!-- Rviz colors (for Gazebo ones change in single files) (from 0 to 1) -->
   <material name="ChassisColor">

Commit message: fix(description): Remove mk1 specific parameters from reseq_parameters.xacro

File: reseq_ros2/description/reseq_parameters.xacro (robot description, xacro)
@@ -31,20 +31,4 @@
   <xacro:property name="JointAMass" value="${config['xacro']['JointAMass']}"/>
   <xacro:property name="JointBMass" value="${config['xacro']['JointBMass']}"/>
-  <!-- arm related (only mk1) -->
-  <!--
-  <xacro:property name="ForkThickness" value="${config['xacro']['ForkThickness']}"/>
-  <xacro:property name="ForkHeight" value="${config['xacro']['ForkHeight']}"/>
-  <xacro:property name="JetsonHolderLength" value="${config['xacro']['JetsonHolderLength']}"/>
-  <xacro:property name="JetsonHolderWidth" value="${config['xacro']['JetsonHolderWidth']}"/>
-  <xacro:property name="CylinderOnJetsonLength" value="${config['xacro']['CylinderOnJetsonLength']}"/>
-  <xacro:property name="CylinderOnJetsonRadius" value="${config['xacro']['CylinderOnJetsonRadius']}"/>
-  <xacro:property name="CylinderOnJetsonShift" value="${config['xacro']['CylinderOnJetsonShift']}"/>
-  <xacro:property name="CylinderRealsenseLength" value="${config['xacro']['CylinderRealsenseLength']}"/>
-  <xacro:property name="CylinderRealsenseRadius" value="${config['xacro']['CylinderRealsenseRadius']}"/>
-  <xacro:property name="RealsenseLength" value="${config['xacro']['RealsenseLength']}"/>
-  <xacro:property name="RealsenseWidth" value="${config['xacro']['RealsenseWidth']}"/>
-  <xacro:property name="RealsenseHeight" value="${config['xacro']['RealsenseHeight']}"/>
-  <xacro:property name="RealsenseOriginSystem" value="${config['xacro']['RealsenseOriginSystem']}"/>
-  -->
   <!-- Rviz colors (for Gazebo ones change in single files) (from 0 to 1) -->
   <material name="ChassisColor">
@@ -57,9 +41,4 @@
     <color rgba="0.5 0.5 0.5 1" />
   </material>
-  <!--
-  <material name="ArmColor">
-    <color rgba="0.5 0.5 0.5 1" />
-  </material>
-  -->
   <material name="LidarColor">
     <color rgba="0.5 0.5 0.5 1" />

Commit message: Modify Parameters and Pipeline for MK2 (#69)
* fix(config): Update xacro file reference for mk1 configuration

* feat(config): Add mk2 digital twin parameters and update reference in vcan config

* fix(config): Update agevar_consts_mk2.yaml parameters

* feat(config): Add mk2 CAN configuration file

* fix(config): Update default CAN configuration filename to mk2

* fix(utils): Ensure get_end_effector returns 0 if no end effector is found

* fix(description): Update configuration to use mk2 CAN parameters and comment out mk1 references

* fix(description): Remove mk1 specific parameters from reseq_parameters.xacro

* fix(description): Conditional inclusion of mk1 arm xacro based on version

* feat(description): Add reseq_arm_parameters.xacro for mk1 arm configuration

* Update reseq_ros2/config/agevar_consts_mk2.yaml

Co-authored-by: Luca De Paola <60526200+luca-byte@users.noreply.github.com>

* Update reseq_ros2/config/digital_twin_params_mk2.yaml

Co-authored-by: Luca De Paola <60526200+luca-byte@users.noreply.github.com>

---------

Co-authored-by: Luca De Paola <60526200+luca-byte@users.noreply.github.com>

File: reseq_ros2/description/reseq_parameters.xacro (robot description, xacro)
@@ -2,5 +2,5 @@
 <robot xmlns:xacro="http://www.ros.org/wiki/xacro">
   <!-- import values from config.yaml file -->
-  <xacro:arg name="config_path" default="$(find reseq_ros2)/config/reseq_mk1_can.yaml"/>
+  <xacro:arg name="config_path" default="$(find reseq_ros2)/config/reseq_mk2_can.yaml"/>
   <xacro:property name="config_path_prop" value="$(arg config_path)"/>
   <xacro:property name="config" value="${xacro.load_yaml(config_path_prop)}"/>
@@ -31,18 +31,4 @@
   <xacro:property name="JointAMass" value="${config['xacro']['JointAMass']}"/>
   <xacro:property name="JointBMass" value="${config['xacro']['JointBMass']}"/>
-  <!-- arm related (only mk1) -->
-  <xacro:property name="ForkThickness" value="${config['xacro']['ForkThickness']}"/>
-  <xacro:property name="ForkHeight" value="${config['xacro']['ForkHeight']}"/>
-  <xacro:property name="JetsonHolderLength" value="${config['xacro']['JetsonHolderLength']}"/>
-  <xacro:property name="JetsonHolderWidth" value="${config['xacro']['JetsonHolderWidth']}"/>
-  <xacro:property name="CylinderOnJetsonLength" value="${config['xacro']['CylinderOnJetsonLength']}"/>
-  <xacro:property name="CylinderOnJetsonRadius" value="${config['xacro']['CylinderOnJetsonRadius']}"/>
-  <xacro:property name="CylinderOnJetsonShift" value="${config['xacro']['CylinderOnJetsonShift']}"/>
-  <xacro:property name="CylinderRealsenseLength" value="${config['xacro']['CylinderRealsenseLength']}"/>
-  <xacro:property name="CylinderRealsenseRadius" value="${config['xacro']['CylinderRealsenseRadius']}"/>
-  <xacro:property name="RealsenseLength" value="${config['xacro']['RealsenseLength']}"/>
-  <xacro:property name="RealsenseWidth" value="${config['xacro']['RealsenseWidth']}"/>
-  <xacro:property name="RealsenseHeight" value="${config['xacro']['RealsenseHeight']}"/>
-  <xacro:property name="RealsenseOriginSystem" value="${config['xacro']['RealsenseOriginSystem']}"/>
   <!-- Rviz colors (for Gazebo ones change in single files) (from 0 to 1) -->
   <material name="ChassisColor">
@@ -55,7 +41,4 @@
     <color rgba="0.5 0.5 0.5 1" />
   </material>
-  <material name="ArmColor">
-    <color rgba="0.5 0.5 0.5 1" />
-  </material>
   <material name="LidarColor">
     <color rgba="0.5 0.5 0.5 1" />

File: reseq_ros2/description/robot.urdf.xacro (robot description, xacro)
@@ -5,4 +5,5 @@
   <xacro:include filename="inertial_macros.xacro" />
   <xacro:include filename="reseq_parameters.xacro" />
+  <xacro:include filename="reseq_arm_parameters.xacro" />
   <xacro:include filename="macros/utils.xacro" />
   <xacro:include filename="macros/joint.xacro" />
@@ -11,5 +12,12 @@
   <xacro:include filename="macros/control_wheel.xacro" />
   <xacro:include filename="reseq_body.xacro" />
-  <xacro:include filename="reseq_arm_mk1.xacro" />
+  <xacro:if value="${config['version'] == 'mk1'}">
+    <xacro:include filename="reseq_arm_mk1.xacro" />
+  </xacro:if>
+  <!--
+  <xacro:if value="${config['version'] == 'mk2'}">
+    <xacro:include filename="reseq_arm_mk2.xacro" />
+  </xacro:if>
+  -->
   <xacro:include filename="lidar.xacro" />
   <xacro:include filename="ros2_control.xacro" />
