Commit message: feat(gz): Urdf wheels and passive joints for gz

File: reseq_ros2/description/robot.urdf.xacro (robot description, xacro)
@@ -11,4 +11,5 @@
   <xacro:include filename="macros/wheel.xacro" />
   <xacro:include filename="macros/control_wheel.xacro" />
+  <xacro:include filename="macros/control_chassis_joint.xacro" />
   <xacro:include filename="reseq_body.xacro" />
   <xacro:if value="${config['version'] == 'mk1'}">

File: reseq_ros2/description/ros2_control.xacro (robot description, xacro)
@@ -20,3 +20,33 @@
         <xacro:loop module="1" n_modules="${NumModules}"/>
     </ros2_control>
+    <ros2_control name="GazeboSimSystem" type="system">
+        <hardware>
+            <plugin>gz_ros2_control/GazeboSimSystem</plugin>
+        </hardware>
+        <!-- Create n_modules modules by recursively calling the loop macro -->
+        <xacro:macro name="loop" params="module n_modules">
+            <xacro:if value="${module &lt;= n_modules}">
+                <!-- Wheels -->
+                <xacro:control_wheel_factory id="${module}" pos="front" side="left" />
+                <xacro:control_wheel_factory id="${module}" pos="front" side="right" />
+                <xacro:control_wheel_factory id="${module}" pos="back" side="left" />
+                <xacro:control_wheel_factory id="${module}" pos="back" side="right" />
+                <xacro:loop module="${module + 1}" n_modules="${n_modules}"/>
+            </xacro:if>
+        </xacro:macro>
+        <xacro:loop module="1" n_modules="${NumModules}"/>
+        <!-- Create n_modules modules by recursively calling the loop macro -->
+        <xacro:macro name="loop2" params="module n_modules">
+            <xacro:if value="${module &lt; n_modules}">
+                <xacro:control_chassis_joint_factory id="${module + 1}"/>
+                <xacro:loop2 module="${module + 1}" n_modules="${n_modules}"/>
+            </xacro:if>
+        </xacro:macro>
+        <xacro:loop2 module="1" n_modules="${NumModules}"/>
+    </ros2_control>
+    <gazebo>
+        <plugin name="gz_ros2_control::GazeboSimROS2ControlPlugin" filename="libgz_ros2_control-system.so">
+            <parameters>$(find reseq_ros2)/config/temp/reseq_controllers.yaml</parameters>
+        </plugin>
+    </gazebo>
 </robot>
