Commit message: feat: add missing inertial properties

File: reseq_ros2/description/lidar.xacro (robot description, xacro)
@@ -27,7 +27,7 @@
       </geometry>
     </collision>
-    <xacro:inertial_cylinder mass="0.1" length="0.04" radius="0.05">
-      <origin xyz="0 0 0" rpy="0 0 0"/>
-    </xacro:inertial_cylinder>
+    <xacro:inertial_cylinder_z mass="0.1" length="0.04" radius="0.05">
+      <origin xyz="0 0 0" rpy="0 0 ${pi/2}"/>
+    </xacro:inertial_cylinder_z>
   </link>
   <gazebo reference="laser_frame">

File: reseq_ros2/description/macros/joint.xacro (robot description, xacro)
@@ -27,4 +27,9 @@
         </visual>
       </xacro:replicate_collision>
+      <xacro:inertial_cylinder_x mass = "${JointBMass}"
+        length = "${JointB}"
+        radius = "${JointWidth/2}">
+        <origin xyz="-${JointB/2} 0 0" rpy="0 ${pi/2} 0" />
+      </xacro:inertial_cylinder_x>
     </link>
     <gazebo reference="joint_r_${id}_link">
@@ -61,4 +66,7 @@
         </visual>
       </xacro:replicate_collision>
+      <xacro:inertial_box mass="${JointAMass}" x="${JointA}" y="${EquivalentWheelDiameter-2*JointABottomClearance}" z="${JointWidth}">
+        <origin xyz="-${JointA/2} 0 0" rpy="0 0 0" />
+      </xacro:inertial_box>
     </link>
     <gazebo reference="joint_y_${id}_link">

File: reseq_ros2/description/macros/wheel.xacro (robot description, xacro)
@@ -36,8 +36,8 @@
             </geometry>
         </collision>
-        <xacro:inertial_cylinder mass="${WheelMass}" length="${TrackWidth}"
+        <xacro:inertial_cylinder_y mass="${WheelMass}" length="${TrackWidth}"
             radius="${EquivalentWheelDiameter/2}">
-            <origin xyz="0 0 0" rpy="${pi/2} 0 0" />
-        </xacro:inertial_cylinder>
+            <origin xyz="0 0 0" rpy="-${pi/2} 0 0" />
+        </xacro:inertial_cylinder_y>
         </link>
         <gazebo reference="${side}_${pos}_wheel_${id}_link">

File: reseq_ros2/description/reseq_arm_mk1.xacro (robot description, xacro)
@@ -71,4 +71,7 @@
       </visual>
     </xacro:replicate_collision>
+    <xacro:inertial_box mass="${0.5}" x="${JetsonHolderLength}" z="${ForkHeight}" y="${JetsonHolderWidth}">
+      <origin xyz="${ForkThickness/2+toll+EquivalentWheelDiameter/2+JetsonHolderLength/2} 0 0" rpy="0 0 0"/>
+    </xacro:inertial_box>
     <!-- cylinder on the jetson holder-->
     <xacro:replicate_collision>
@@ -81,8 +84,8 @@
       </visual>
     </xacro:replicate_collision>
-    <xacro:inertial_box mass="${0.5}" x="${JetsonHolderLength}" y="${ForkHeight}" z="${JetsonHolderWidth}">
-      <origin xyz="${ForkThickness/2+toll+EquivalentWheelDiameter/2+JetsonHolderLength/2} 0 0" rpy="0 0 0"/>
-    </xacro:inertial_box>
   </link>
+  <gazebo reference="arm_mk1_link">
+    <material>Gazebo/Grey</material>
+  </gazebo>
   <!-- head pitch joint-->
   <joint name="arm_head_pitch_1_joint" type="revolute">
@@ -139,4 +142,7 @@
       </visual>
     </xacro:replicate_collision>
+    <xacro:inertial_box mass="0.5" x="${RealsenseLength}" y="${RealsenseWidth}" z="${RealsenseHeight}">
+      <origin xyz ="0 0 -${CylinderRealsenseLength + RealsenseLength/2}" rpy="0 ${pi/2} 0"/>
+    </xacro:inertial_box>
   </link>
   <gazebo reference="arm_camera_holder">

Commit message: fix: change lidar position

File: reseq_ros2/description/lidar.xacro (robot description, xacro)
@@ -4,5 +4,5 @@
     <parent link="chassis2_link"/>
     <child link="laser_frame"/>
-    <origin xyz="0 0 0.1" rpy="0 0 0"/>
+    <origin xyz="-0.07 0 0.1" rpy="0 0 0"/>
   </joint>
   <link name="laser_frame">
