Commit message: feat: display modules depending on number

File: reseq_ros2/description/reseq_body.xacro (robot description, xacro)
@@ -8,6 +8,14 @@
     <origin xyz="0 0 ${(EquivalentWheelDiameter-2*ChassisTopAndBottomClearance)/2+ChassisTopAndBottomClearance}"/>
   </joint>
-  <xacro:chassis id="1"/>
-  <xacro:chassis_joint_factory id="2"/>
-  <xacro:chassis id="2"/>
+  <xacro:macro name="loop" params="module n_modules">
+    <xacro:if value="${module &lt; n_modules}">
+      <xacro:chassis id="${module}"/>
+      <xacro:chassis_joint_factory id="${module + 1}"/>
+      <xacro:loop module="${module + 1}" n_modules="${n_modules}"/>
+    </xacro:if>
+    <xacro:if value="${module == n_modules}">
+      <xacro:chassis id="${module}"/>
+    </xacro:if>
+  </xacro:macro>
+  <xacro:loop module="1" n_modules="${NumModules}"/>
 </robot>

File: reseq_ros2/description/reseq_parameters.xacro (robot description, xacro)
@@ -11,4 +11,5 @@
   <xacro:property name="toll" value="0.001"/>
   <!-- chassis related -->
+  <xacro:property name="NumModules" value="${config['xacro']['NumModules']}"/>
   <xacro:property name="WheelBase" value="${config['xacro']['WheelBase']}"/>
   <xacro:property name="EquivalentWheelDiameter" value="${r_eq*2}"/>

Commit message: feat: Add base footprint link

File: reseq_ros2/description/reseq_body.xacro (robot description, xacro)
@@ -2,4 +2,10 @@
 <robot xmlns:xacro="http://www.ros.org/wiki/xacro">
   <link name="base_link" />
+  <link name="base_footprint" />
+  <joint name="base_footprint_joint" type="fixed">
+    <parent link="base_link"/>
+    <child link="base_footprint"/>
+    <origin xyz="0 0 0" />
+  </joint>
   <joint name="chassis1_joint" type="fixed">
     <parent link="base_link"/>
