Commit message: fix: fix arm pitch joint name

File: reseq_ros2/description/reseq_arm_mk1.xacro (robot description, xacro)
@@ -2,5 +2,5 @@
 <robot xmlns:xacro="http://www.ros.org/wiki/xacro">
   <!-- This is a parametric description of reseq mK1 arm -->
-  <joint name="arm_mK1_joint" type="revolute">
+  <joint name="arm_pitch_1_joint" type="revolute">
     <parent link="chassis1_link"/>
     <child link="arm_mK1_link"/>

Commit message: feat: complete arm with camera holder and head joints

File: reseq_ros2/description/reseq_arm_mk1.xacro (robot description, xacro)
@@ -91,4 +91,65 @@
     </xacro:inertial_box>
   </link>
+  <!-- head pitch joint-->
+  <joint name="arm_mK1_head_pitch" type="revolute">
+    <parent link="arm_mK1_link"/>
+    <child link="camera_holder_intermediate"/>
+    <!-- Effort in Nm, angle in radians -->
+    <limit effort="10.0" lower="0" upper="-${pi}" velocity="0.5"/>
+    <origin xyz ="${ForkThickness/2+toll+EquivalentWheelDiameter/2+JetsonHolderLength + CylinderOnJetsonLength - CylinderOnJetsonRadius} -${CylinderOnJetsonShift} 0"/>
+    <axis xyz="0 1 0"/>
+  </joint>
+  <link name="camera_holder_intermediate">
+  </link>
+  <!-- head roll joint -->
+  <joint name="arm_mK1_head_roll" type="revolute">
+    <parent link="camera_holder_intermediate"/>
+    <child link="camera_holder"/>
+    <!-- Effort in Nm, angle in radians -->
+    <limit effort="10.0" lower="${-5*(pi/6)}" upper="${5*(pi/6)}" velocity="0.5"/>
+    <origin xyz ="0 0 0"/>
+    <axis xyz="1 0 0"/>
+  </joint>
+  <link name="camera_holder">
+    <!-- cylinder between realsense and rotation axis -->
+    <xacro:replicate_collision>
+      <visual>
+        <origin xyz ="0 0 -${CylinderRealsenseRadius + CylinderRealsenseLength/2}" rpy="0 0 0"/>
+        <geometry>
+          <cylinder radius="${CylinderRealsenseRadius}" length="${CylinderRealsenseLength}"/>
+        </geometry>
+        <material name="ArmColor"/>
+      </visual>
+    </xacro:replicate_collision>
+    <!-- sphere -->
+    <xacro:replicate_collision>
+      <visual>
+        <origin xyz ="0 0 0" rpy="${pi/2} ${pi} ${pi}"/>
+        <geometry>
+          <sphere radius="0.037"/>  <!-- this value? -->
+        </geometry>
+        <material name="ArmColor"/>
+      </visual>
+    </xacro:replicate_collision>
+    <!-- realsense holder -->
+    <xacro:replicate_collision>
+      <visual>
+        <origin xyz ="0 0 -${RealsenseLength + 2*CylinderRealsenseRadius + RealsenseLength/2}" rpy="0 ${pi/2} 0"/>
+        <geometry>
+          <box size="${RealsenseLength} ${RealsenseWidth} ${2*CylinderRealsenseRadius}"/>
+        </geometry>
+        <material name="ArmColor"/>
+      </visual>
+    </xacro:replicate_collision>
+  </link>
+  <joint name="camera_joint" type="fixed">
+    <parent link="camera_holder"/>
+    <child link="camera_link_copy"/>
+    <!-- Effort in Nm, angle in radians -->
+    <origin xyz ="0 ${RealsenseOriginSystem} -${RealsenseLength + 2*CylinderRealsenseRadius + RealsenseLength/2}" rpy="0 ${pi/2} 0"/>
+    <axis xyz="1 0 0"/>
+  </joint>
+  <link name="camera_link_copy">
+  </link>
   <gazebo reference="arm_mK1_link">
     <material>Gazebo/Grey</material>

Commit message: feat: create automatically collisions from visuals

File: reseq_ros2/description/reseq_arm_mk1.xacro (robot description, xacro)
@@ -12,4 +12,5 @@
   <link name="arm_mK1_link">
     <!-- cylinder to the right -->
+    <xacro:replicate_collision>
     <visual>
       <origin xyz="0 0 ${ForkThickness/2+toll+ModuleWidth/2}" />
@@ -19,5 +20,7 @@
       <material name="ArmColor"/>
     </visual>
+    </xacro:replicate_collision>
     <!-- cylinder to the left -->
+    <xacro:replicate_collision>
     <visual>
       <origin xyz="0 0 -${ForkThickness/2+toll+ModuleWidth/2}" />
@@ -27,5 +30,7 @@
       <material name="ArmColor"/>
     </visual>
+    </xacro:replicate_collision>
     <!-- right side of the fork -->
+    <xacro:replicate_collision>
     <visual>
       <origin xyz="${(toll+EquivalentWheelDiameter/2)/2} 0 ${ForkThickness/2+toll+ModuleWidth/2}" />
@@ -35,5 +40,7 @@
       <material name="ArmColor"/>
     </visual>
+    </xacro:replicate_collision>
     <!-- left side of the fork -->
+    <xacro:replicate_collision>
     <visual>
       <origin xyz="${(toll+EquivalentWheelDiameter/2)/2} 0 -${ForkThickness/2+toll+ModuleWidth/2}" />
@@ -43,5 +50,7 @@
       <material name="ArmColor"/>
     </visual>
+    </xacro:replicate_collision>
     <!-- front side of the fork -->
+    <xacro:replicate_collision>
     <visual>
       <origin xyz="${ForkThickness/2+toll+EquivalentWheelDiameter/2} 0 0" />
@@ -51,5 +60,7 @@
       <material name="ArmColor"/>
     </visual>
+    </xacro:replicate_collision>
     <!-- Jetson holder -->
+    <xacro:replicate_collision>
     <visual>
       <origin xyz="${ForkThickness/2+toll+EquivalentWheelDiameter/2+JetsonHolderLength/2} 0 0" />
@@ -59,4 +70,5 @@
       <material name="ArmColor"/>
     </visual>
+    </xacro:replicate_collision>
     <!-- cylinder to the right -->
     <collision>
@@ -65,26 +77,7 @@
         <cylinder radius="${ForkHeight/2}" length="${ForkThickness}"/>
       </geometry>
-    </collision>
-    <!-- cylinder to the left -->
-    <collision>
-      <origin xyz="0 0 -${ForkThickness/2+toll+ModuleWidth/2}" />
-      <geometry>
-        <cylinder radius="${ForkHeight/2}" length="${ForkThickness}"/>
-      </geometry>
-    </collision>
-    <!-- front side of the fork -->
-    <collision>
-      <origin xyz="${ForkThickness/2+toll+EquivalentWheelDiameter/2} 0 0" />
-      <geometry>
-        <box size="${ForkThickness} ${ForkHeight} ${ModuleWidth+(toll+ForkThickness)*2}"/>
-      </geometry>
-    </collision>
-    <!-- Jetson holder -->
-    <collision>
-      <origin xyz="${ForkThickness/2+toll+EquivalentWheelDiameter/2+JetsonHolderLength/2} 0 0" />
-      <geometry>
-        <box size="${JetsonHolderLength} ${ForkHeight} ${JetsonHolderWidth}"/>
-      </geometry>
-    </collision>
+        <material name="ArmColor"/>
+      </visual>
+    </xacro:replicate_collision>
     <xacro:inertial_box mass="${0.5}" x="${JetsonHolderLength}" y="${ForkHeight}" z="${JetsonHolderWidth}">
       <origin xyz="${ForkThickness/2+toll+EquivalentWheelDiameter/2+JetsonHolderLength/2} 0 0" rpy="0 0 0"/>

Commit message: fix: rotate arm joint

File: reseq_ros2/description/reseq_arm_mk1.xacro (robot description, xacro)
@@ -6,75 +6,76 @@
     <child link="arm_mK1_link"/>
     <!-- Effort in Nm, angle in radians -->
-    <limit effort="10.0" lower="-${pi*0.01}" upper="${pi/2}" velocity="0.5"/>
-    <origin xyz="${WheelBase/2} 0 0" rpy="${pi/2} 0 0" />
-    <axis xyz="0 0 1"/>
+    <limit effort="10.0" lower="${pi*0.01}" upper="-${pi/2}" velocity="0.5"/>
+    <origin xyz="${WheelBase/2} 0 0" />
+    <axis xyz="0 1 0"/>
   </joint>
   <link name="arm_mK1_link">
     <!-- cylinder to the right -->
     <xacro:replicate_collision>
-    <visual>
-      <origin xyz="0 0 ${ForkThickness/2+toll+ModuleWidth/2}" />
-      <geometry>
-        <cylinder radius="${ForkHeight/2}" length="${ForkThickness}"/>
-      </geometry>
-      <material name="ArmColor"/>
-    </visual>
+      <visual>
+        <origin xyz="0 ${-(ForkThickness/2+toll+ModuleWidth/2)} 0" rpy = "${pi/2} 0 0"/>
+        <geometry>
+          <cylinder radius="${ForkHeight/2}" length="${ForkThickness}"/>
+        </geometry>
+        <material name="ArmColor"/>
+      </visual>
     </xacro:replicate_collision>
     <!-- cylinder to the left -->
     <xacro:replicate_collision>
-    <visual>
-      <origin xyz="0 0 -${ForkThickness/2+toll+ModuleWidth/2}" />
-      <geometry>
-        <cylinder radius="${ForkHeight/2}" length="${ForkThickness}"/>
-      </geometry>
-      <material name="ArmColor"/>
-    </visual>
+      <visual>
+        <origin xyz="0 ${(ForkThickness/2+toll+ModuleWidth/2)} 0" rpy = "${pi/2} 0 0"/>
+        <geometry>
+          <cylinder radius="${ForkHeight/2}" length="${ForkThickness}"/>
+        </geometry>
+        <material name="ArmColor"/>
+      </visual>
     </xacro:replicate_collision>
     <!-- right side of the fork -->
     <xacro:replicate_collision>
-    <visual>
-      <origin xyz="${(toll+EquivalentWheelDiameter/2)/2} 0 ${ForkThickness/2+toll+ModuleWidth/2}" />
-      <geometry>
-        <box size="${toll+EquivalentWheelDiameter/2} ${ForkHeight} ${ForkThickness}"/>
-      </geometry>
-      <material name="ArmColor"/>
-    </visual>
+      <visual>
+        <origin xyz="${(toll+EquivalentWheelDiameter/2)/2} -${ForkThickness/2+toll+ModuleWidth/2} 0" rpy = "${pi/2} 0 0"/>
+        <geometry>
+          <box size="${toll+EquivalentWheelDiameter/2} ${ForkHeight} ${ForkThickness}"/>
+        </geometry>
+        <material name="ArmColor"/>
+      </visual>
     </xacro:replicate_collision>
     <!-- left side of the fork -->
     <xacro:replicate_collision>
-    <visual>
-      <origin xyz="${(toll+EquivalentWheelDiameter/2)/2} 0 -${ForkThickness/2+toll+ModuleWidth/2}" />
-      <geometry>
-        <box size="${toll+EquivalentWheelDiameter/2} ${ForkHeight} ${ForkThickness}"/>
-      </geometry>
-      <material name="ArmColor"/>
-    </visual>
+      <visual>
+        <origin xyz="${(toll+EquivalentWheelDiameter/2)/2} ${ForkThickness/2+toll+ModuleWidth/2} 0" rpy = "${pi/2} 0 0"/>
+        <geometry>
+          <box size="${toll+EquivalentWheelDiameter/2} ${ForkHeight} ${ForkThickness}"/>
+        </geometry>
+        <material name="ArmColor"/>
+      </visual>
     </xacro:replicate_collision>
     <!-- front side of the fork -->
     <xacro:replicate_collision>
-    <visual>
-      <origin xyz="${ForkThickness/2+toll+EquivalentWheelDiameter/2} 0 0" />
-      <geometry>
-        <box size="${ForkThickness} ${ForkHeight} ${ModuleWidth+(toll+ForkThickness)*2}"/>
-      </geometry>
-      <material name="ArmColor"/>
-    </visual>
+      <visual>
+        <origin xyz="${ForkThickness/2+toll+EquivalentWheelDiameter/2} 0 0" rpy = "${pi/2} 0 0"/>
+        <geometry>
+          <box size="${ForkThickness} ${ForkHeight} ${ModuleWidth+(toll+ForkThickness)*2}"/>
+        </geometry>
+        <material name="ArmColor"/>
+      </visual>
     </xacro:replicate_collision>
     <!-- Jetson holder -->
     <xacro:replicate_collision>
-    <visual>
-      <origin xyz="${ForkThickness/2+toll+EquivalentWheelDiameter/2+JetsonHolderLength/2} 0 0" />
-      <geometry>
-        <box size="${JetsonHolderLength} ${ForkHeight} ${JetsonHolderWidth}"/>
-      </geometry>
-      <material name="ArmColor"/>
-    </visual>
+      <visual>
+        <origin xyz="${ForkThickness/2+toll+EquivalentWheelDiameter/2+JetsonHolderLength/2} 0 0" rpy = "${pi/2} 0 0"/>
+        <geometry>
+          <box size="${JetsonHolderLength} ${ForkHeight} ${JetsonHolderWidth}"/>
+        </geometry>
+        <material name="ArmColor"/>
+      </visual>
     </xacro:replicate_collision>
-    <!-- cylinder to the right -->
-    <collision>
-      <origin xyz="0 0 ${ForkThickness/2+toll+ModuleWidth/2}" />
-      <geometry>
-        <cylinder radius="${ForkHeight/2}" length="${ForkThickness}"/>
-      </geometry>
+    <!-- cylinder on the jetson holder-->
+    <xacro:replicate_collision>
+      <visual>
+        <origin xyz ="${ForkThickness/2+toll+EquivalentWheelDiameter/2+JetsonHolderLength + CylinderOnJetsonLength/2} -${CylinderOnJetsonShift} 0" rpy="0 ${pi/2} 0"/>
+        <geometry>
+          <cylinder radius="${CylinderOnJetsonRadius}" length="${CylinderOnJetsonLength}"/>
+        </geometry>
         <material name="ArmColor"/>
       </visual>

Commit message: fix: revert realsense camera link

File: reseq_ros2/description/reseq_arm_mk1.xacro (robot description, xacro)
@@ -139,10 +139,10 @@
   <joint name="camera_joint" type="fixed">
     <parent link="camera_holder"/>
-    <child link="camera_link_copy"/>
+    <child link="camera_link"/>
     <!-- Effort in Nm, angle in radians -->
     <origin xyz ="0 ${RealsenseOriginSystem} -${RealsenseLength + 2*CylinderRealsenseRadius + RealsenseLength/2}" rpy="0 ${pi/2} 0"/>
     <axis xyz="1 0 0"/>
   </joint>
-  <link name="camera_link_copy">
+  <link name="camera_link">
   </link>
   <gazebo reference="arm_mK1_link">

Commit message: fix: rename joints according to joint_publisher

File: reseq_ros2/description/reseq_arm_mk1.xacro (robot description, xacro)
@@ -2,5 +2,5 @@
 <robot xmlns:xacro="http://www.ros.org/wiki/xacro">
   <!-- This is a parametric description of reseq mK1 arm -->
-  <joint name="arm_mK1_joint" type="revolute">
+  <joint name="arm_pitch_1_joint" type="revolute">
     <parent link="chassis1_link"/>
     <child link="arm_mK1_link"/>
@@ -86,5 +86,5 @@
   </link>
   <!-- head pitch joint-->
-  <joint name="arm_mK1_head_pitch" type="revolute">
+  <joint name="arm_head_pitch_1_joint" type="revolute">
     <parent link="arm_mK1_link"/>
     <child link="camera_holder_intermediate"/>
@@ -97,5 +97,5 @@
   </link>
   <!-- head roll joint -->
-  <joint name="arm_mK1_head_roll" type="revolute">
+  <joint name="arm_head_roll_1_joint" type="revolute">
     <parent link="camera_holder_intermediate"/>
     <child link="camera_holder"/>

Commit message: fix: rename links for clarity
The names were similar to the ones published by the realsense

File: reseq_ros2/description/reseq_arm_mk1.xacro (robot description, xacro)
@@ -4,5 +4,5 @@
   <joint name="arm_pitch_1_joint" type="revolute">
     <parent link="chassis1_link"/>
-    <child link="arm_mK1_link"/>
+    <child link="arm_mk1_link"/>
     <!-- Effort in Nm, angle in radians -->
     <limit effort="10.0" lower="${pi*0.01}" upper="-${pi/2}" velocity="0.5"/>
@@ -10,5 +10,5 @@
     <axis xyz="0 1 0"/>
   </joint>
-  <link name="arm_mK1_link">
+  <link name="arm_mk1_link">
     <!-- cylinder to the right -->
     <xacro:replicate_collision>
@@ -87,6 +87,6 @@
   <!-- head pitch joint-->
   <joint name="arm_head_pitch_1_joint" type="revolute">
-    <parent link="arm_mK1_link"/>
-    <child link="camera_holder_intermediate"/>
+    <parent link="arm_mk1_link"/>
+    <child link="arm_camera_holder_intermediate"/>
     <!-- Effort in Nm, angle in radians -->
     <limit effort="10.0" lower="0" upper="-${pi}" velocity="0.5"/>
@@ -94,10 +94,10 @@
     <axis xyz="0 1 0"/>
   </joint>
-  <link name="camera_holder_intermediate">
+  <link name="arm_camera_holder_intermediate">
   </link>
   <!-- head roll joint -->
   <joint name="arm_head_roll_1_joint" type="revolute">
-    <parent link="camera_holder_intermediate"/>
-    <child link="camera_holder"/>
+    <parent link="arm_camera_holder_intermediate"/>
+    <child link="arm_camera_holder"/>
     <!-- Effort in Nm, angle in radians -->
     <limit effort="10.0" lower="${-5*(pi/6)}" upper="${5*(pi/6)}" velocity="0.5"/>
@@ -105,5 +105,5 @@
     <axis xyz="1 0 0"/>
   </joint>
-  <link name="camera_holder">
+  <link name="arm_camera_holder">
     <!-- cylinder between realsense and rotation axis -->
     <xacro:replicate_collision>
@@ -137,6 +137,6 @@
     </xacro:replicate_collision>
   </link>
-  <joint name="camera_joint" type="fixed">
-    <parent link="camera_holder"/>
+  <joint name="arm_camera_joint" type="fixed">
+    <parent link="arm_camera_holder"/>
     <child link="camera_link"/>
     <!-- Effort in Nm, angle in radians -->

Commit message: fix: fix arm dimensions

File: reseq_ros2/description/reseq_arm_mk1.xacro (robot description, xacro)
@@ -74,5 +74,5 @@
     <xacro:replicate_collision>
       <visual>
-        <origin xyz ="${ForkThickness/2+toll+EquivalentWheelDiameter/2+JetsonHolderLength + CylinderOnJetsonLength/2} -${CylinderOnJetsonShift} 0" rpy="0 ${pi/2} 0"/>
+        <origin xyz ="${ForkThickness/2+toll+EquivalentWheelDiameter/2+JetsonHolderLength + CylinderOnJetsonLength/2} 0 ${CylinderOnJetsonShift}" rpy="0 ${pi/2} 0"/>
         <geometry>
           <cylinder radius="${CylinderOnJetsonRadius}" length="${CylinderOnJetsonLength}"/>
@@ -91,5 +91,5 @@
     <!-- Effort in Nm, angle in radians -->
     <limit effort="10.0" lower="0" upper="-${pi}" velocity="0.5"/>
-    <origin xyz ="${ForkThickness/2+toll+EquivalentWheelDiameter/2+JetsonHolderLength + CylinderOnJetsonLength - CylinderOnJetsonRadius} -${CylinderOnJetsonShift} 0"/>
+    <origin xyz ="${ForkThickness/2+toll+EquivalentWheelDiameter/2+JetsonHolderLength + CylinderOnJetsonLength} 0 ${CylinderOnJetsonShift}"/>
     <axis xyz="0 1 0"/>
   </joint>
@@ -109,5 +109,5 @@
     <xacro:replicate_collision>
       <visual>
-        <origin xyz ="0 0 -${CylinderRealsenseRadius + CylinderRealsenseLength/2}" rpy="0 0 0"/>
+        <origin xyz ="0 0 -${CylinderRealsenseLength/2}" rpy="0 0 0"/>
         <geometry>
           <cylinder radius="${CylinderRealsenseRadius}" length="${CylinderRealsenseLength}"/>
@@ -121,5 +121,5 @@
         <origin xyz ="0 0 0" rpy="${pi/2} ${pi} ${pi}"/>
         <geometry>
-          <sphere radius="0.037"/>  <!-- this value? -->
+          <sphere radius="${CylinderRealsenseRadius}"/>
         </geometry>
         <material name="ArmColor"/>
@@ -129,7 +129,7 @@
     <xacro:replicate_collision>
       <visual>
-        <origin xyz ="0 0 -${RealsenseLength + 2*CylinderRealsenseRadius + RealsenseLength/2}" rpy="0 ${pi/2} 0"/>
+        <origin xyz ="0 0 -${CylinderRealsenseLength + RealsenseLength/2}" rpy="0 ${pi/2} 0"/>
         <geometry>
-          <box size="${RealsenseLength} ${RealsenseWidth} ${2*CylinderRealsenseRadius}"/>
+          <box size="${RealsenseLength} ${RealsenseWidth} ${RealsenseHeight}"/>
         </geometry>
         <material name="ArmColor"/>
@@ -141,5 +141,5 @@
     <child link="camera_link"/>
     <!-- Effort in Nm, angle in radians -->
-    <origin xyz ="0 ${RealsenseOriginSystem} -${RealsenseLength + 2*CylinderRealsenseRadius + RealsenseLength/2}" rpy="0 ${pi/2} 0"/>
+    <origin xyz ="0 ${RealsenseOriginSystem} -${CylinderRealsenseLength}" rpy="0 ${pi/2} 0"/>
     <axis xyz="1 0 0"/>
   </joint>

File: reseq_ros2/description/reseq_parameters.xacro (robot description, xacro)
@@ -43,4 +43,5 @@
   <xacro:property name="RealsenseLength" value="${config['xacro']['RealsenseLength']}"/>
   <xacro:property name="RealsenseWidth" value="${config['xacro']['RealsenseWidth']}"/>
+  <xacro:property name="RealsenseHeight" value="${config['xacro']['RealsenseHeight']}"/>
   <xacro:property name="RealsenseOriginSystem" value="${config['xacro']['RealsenseOriginSystem']}"/>
   <!-- Rviz colors (for Gazebo ones change in single files) (from 0 to 1) -->

Commit message: feat(gazebo): Modify gazebo launch file to use GZ Fortress
Co-Authored-By: Lorenzo Ciocca <103076648+lorixhack@users.noreply.github.com>

File: reseq_ros2/description/reseq_arm_mk1.xacro (robot description, xacro)
@@ -149,8 +149,8 @@
     <material>Gazebo/Grey</material>
   </gazebo>
-  <joint name="arm_camera_joint" type="fixed">
+  <!-- <joint name="arm_camera_joint" type="fixed">
     <parent link="arm_camera_holder"/>
     <child link="camera_link"/>
-    <!-- Effort in Nm, angle in radians -->
+    Effort in Nm, angle in radians
     <origin xyz ="0 ${RealsenseOriginSystem} -${CylinderRealsenseLength}" rpy="0 ${pi/2} 0"/>
     <axis xyz="1 0 0"/>
@@ -161,3 +161,4 @@
     <material>Gazebo/Grey</material>
   </gazebo>
+   -->
 </robot>

Commit message: fix: Add inertial attribut to arm camera holder intermediate

File: reseq_ros2/description/reseq_arm_mk1.xacro (robot description, xacro)
@@ -99,4 +99,10 @@
   </joint>
   <link name="arm_camera_holder_intermediate">
+    <inertial>
+      <mass value="0.05"/> <!-- 50 grams -->
+      <inertia ixx="1e-4" ixy="0" ixz="0"
+             iyy="1e-4" iyz="0"
+             izz="1e-4"/>
+    </inertial>
   </link>
   <gazebo reference="arm_camera_holder_intermediate">
