Commit message: feat: Add differential controllers

File: reseq_ros2/description/ros2_control.xacro (robot description, xacro)
@@ -1,20 +1,22 @@
 <?xml version="1.0"?>
 <robot xmlns:xacro="http://www.ros.org/wiki/xacro">
-    <ros2_control name="GazeboSystem" type="system">
+    <ros2_control name="Rviz" type="system">
+        <!-- Mirror commands to their states -->
         <hardware>
-            <plugin>gazebo_ros2_control/GazeboSystem</plugin>
+            <plugin>mock_components/GenericSystem</plugin>
+            <param name="calculate_dynamics">true</param>
         </hardware>
-    <!-- Create n_modules modules by recursively calling the loop macro -->
-    <xacro:macro name="loop" params="module n_modules">
-        <xacro:if value="${module &lt; n_modules}">
-            <!-- Wheels -->
-            <xacro:control_wheel_factory id="${module}" pos="front" side="left" />
-            <xacro:control_wheel_factory id="${module}" pos="front" side="right" />
-            <xacro:control_wheel_factory id="${module}" pos="back" side="left" />
-            <xacro:control_wheel_factory id="${module}" pos="back" side="right" />
-            <xacro:loop module="${module + 1}" n_modules="${n_modules}"/>
-        </xacro:if>
-    </xacro:macro>
-    <xacro:loop module="1" n_modules="${NumModules}"/>
+        <!-- Create n_modules modules by recursively calling the loop macro -->
+        <xacro:macro name="loop" params="module n_modules">
+            <xacro:if value="${module &lt;= n_modules}">
+                <!-- Wheels -->
+                <xacro:control_wheel_factory id="${module}" pos="front" side="left" />
+                <xacro:control_wheel_factory id="${module}" pos="front" side="right" />
+                <xacro:control_wheel_factory id="${module}" pos="back" side="left" />
+                <xacro:control_wheel_factory id="${module}" pos="back" side="right" />
+                <xacro:loop module="${module + 1}" n_modules="${n_modules}"/>
+            </xacro:if>
+        </xacro:macro>
+        <xacro:loop module="1" n_modules="${NumModules}"/>
     </ros2_control>
 </robot>

Commit message: feat: mk1 arm joints in gazebo

File: reseq_ros2/description/ros2_control.xacro (robot description, xacro)
@@ -28,4 +28,20 @@
         </xacro:macro>
         <xacro:loop module="1" n_modules="${NumModules}" />
+        <!-- ARM CONTROLLER INTERFACES -->
+        <joint name="arm_pitch_1_joint">
+            <command_interface name="position" />
+            <state_interface name="position" />
+            <state_interface name="velocity"/>
+        </joint>
+        <joint name="arm_head_pitch_1_joint">
+            <command_interface name="position" />
+            <state_interface name="position" />
+            <state_interface name="velocity"/>
+        </joint>
+        <joint name="arm_head_roll_1_joint">
+            <command_interface name="position" />
+            <state_interface name="position" />
+            <state_interface name="velocity" />
+        </joint>
     </ros2_control>
     <xacro:if value="$(arg sim_mode)">
