Commit message: fix: add JointWidth property

File: reseq_ros2/description/macros/joint.xacro (robot description, xacro)
@@ -22,5 +22,5 @@
           <origin xyz="-${JointB/2} 0 0" rpy="0 ${pi/2} 0" />
           <geometry>
-            <cylinder radius="${(ModuleWidth-2*TrackWidth-toll*2)/2}" length="${JointB}" />
+            <cylinder radius="${JointWidth/2}" length="${JointB}" />
           </geometry>
           <material name="JointColor" />
@@ -42,5 +42,5 @@
         <visual>
           <geometry>
-            <sphere radius="${(ModuleWidth-2*TrackWidth-toll*2)/2}" />
+            <sphere radius="${JointWidth/2}" />
           </geometry>
           <material name="JointColor" />
@@ -53,5 +53,5 @@
           <geometry>
             <box
-              size="${JointA} ${EquivalentWheelDiameter-2*JointABottomClearance} ${ModuleWidth-2*TrackWidth-toll*2}" />
+              size="${JointA} ${EquivalentWheelDiameter-2*JointABottomClearance} ${JointWidth}" />
           </geometry>
           <material name="JointColor" />

File: reseq_ros2/description/reseq_parameters.xacro (robot description, xacro)
@@ -23,4 +23,5 @@
   <xacro:property name="JointB" value="${b-WheelBase/2}"/>
   <xacro:property name="JointABottomClearance" value="${config['xacro']['JointABottomClearance']}"/>
+  <xacro:property name="JointWidth" value="${config['xacro']['JointWidth']}"/>
   <xacro:property name="pitch" value="${pi/2}"/>
   <xacro:property name="roll" value="${pi/2}"/>
