Commit message: feat: split macros into multiple files

File: reseq_ros2/description/macros/chassis.xacro (robot description, xacro)
@@ -1,104 +1,4 @@
 <?xml version="1.0"?>
 <robot xmlns:xacro="http://www.ros.org/wiki/xacro">
-  <xacro:include filename="inertial_macros.xacro" />
-  <xacro:include filename="reseq_parameters.xacro" />
-  <!--
-    Replicates the visual block inside the collision block to avoid code
-    duplication until the use of 3D meshes for the visuals
-    @param **block: the <visual/> block to replicate
-   -->
-  <xacro:macro name="replicate_collision" params="**block">
-    <visual>
-      <xacro:insert_block name="block" />
-    </visual>
-    <collision>
-      <xacro:insert_block name="block" />
-    </collision>
-  </xacro:macro>
-  <!--
-    Creates the joint between two consecutive chassis. It assumes that two
-    consecutive chassis have a consecutive id. This macro must be called between
-    the definition of the two chassis
-    @param id: the id of the joint (which is assumed part of the chassis behind)
-   -->
-  <xacro:macro name="chassis_joint_factory" params="id">
-    <!-- JointR -->
-    <joint name="joint_r_${id}_joint" type="revolute">
-      <parent link="chassis${id-1}_link" />
-      <child link="joint_r_${id}_link" />
-      <!-- Effort in Nm -->
-      <limit effort="2.0" lower="${-roll}" upper="${roll}" velocity="0.5" />
-      <origin xyz="-${WheelBase/2} 0 0" rpy="0 0 0" />
-      <axis xyz="1 0 0" />
-    </joint>
-    <link name="joint_r_${id}_link">
-      <xacro:replicate_collision>
-        <visual>
-          <origin xyz="-${JointB/2} 0 0" rpy="0 ${pi/2} 0" />
-          <geometry>
-            <cylinder radius="${(ModuleWidth-2*TrackWidth-toll*2)/2}" length="${JointB}" />
-          </geometry>
-          <material name="JointColor" />
-        </visual>
-      </xacro:replicate_collision>
-    </link>
-    <!-- JointY -->
-    <joint name="joint_y_${id}_joint" type="revolute">
-      <parent link="joint_r_${id}_link" />
-      <child link="joint_y_${id}_link" />
-      <!-- Effort in Nm -->
-      <limit effort="20.0" lower="${-yaw}" upper="${yaw}" velocity="0.5" />
-      <origin xyz="-${JointB} 0 0" rpy="0 0 0" />
-      <axis xyz="0 0 1" />
-    </joint>
-    <link name="joint_y_${id}_link">
-      <!-- to hide space wile rotating -->
-      <xacro:replicate_collision>
-        <visual>
-          <geometry>
-            <sphere radius="${(ModuleWidth-2*TrackWidth-toll*2)/2}" />
-          </geometry>
-          <material name="JointColor" />
-        </visual>
-      </xacro:replicate_collision>
-      <!-- horizontal shaft -->
-      <xacro:replicate_collision>
-        <visual>
-          <origin xyz="-${JointA/2} 0 0" rpy="${pi/2} 0 0" />
-          <geometry>
-            <box
-              size="${JointA} ${EquivalentWheelDiameter-2*JointABottomClearance} ${ModuleWidth-2*TrackWidth-toll*2}" />
-          </geometry>
-          <material name="JointColor" />
-        </visual>
-      </xacro:replicate_collision>
-    </link>
-    <!-- JointP -->
-    <joint name="joint_p_${id}_joint" type="revolute">
-      <parent link="joint_y_${id}_link" />
-      <child link="joint_p_${id}_link" />
-      <!-- Effort in Nm -->
-      <limit effort="20.0" lower="${-pitch}" upper="${pitch}" velocity="0.5" />
-      <origin xyz="${-JointA} 0 0" rpy="0 0 0" />
-      <axis xyz="0 1 0" />
-    </joint>
-    <link name="joint_p_${id}_link">
-      <!-- gearbox cilinder -->
-      <xacro:replicate_collision>
-        <visual>
-          <origin rpy="${pi/2} 0 0" />
-          <geometry>
-            <cylinder radius="${JointDiameter/2}" length="${ModuleWidth-2*TrackWidth-toll*2}" />
-          </geometry>
-          <material name="JointColor" />
-        </visual>
-      </xacro:replicate_collision>
-    </link>
-    <joint name="chassis${id}_joint" type="fixed">
-      <parent link="joint_p_${id}_link" />
-      <child link="chassis${id}_link" />
-      <origin xyz="${-WheelBase/2} 0 0" rpy="0 0 0" />
-    </joint>
-  </xacro:macro>
   <!--
     Defines the current chassis
@@ -223,15 +123,3 @@
     </link>
   </xacro:macro>
-  <link name="base_link" />
-  <joint name="chassis1_joint" type="fixed">
-    <parent link="base_link" />
-    <child link="chassis1_link" />
-    <!-- leaving 1/3 of the EquivalentWheelDiameter from front (origin is in the center of eq wheel,
-    at the bottom of the chassis) -->
-    <origin
-      xyz="0 0 ${(EquivalentWheelDiameter-2*ChassisTopAndBottomClearance)/2+ChassisTopAndBottomClearance}" />
-  </joint>
-  <xacro:chassis id="1" />
-  <xacro:chassis_joint_factory id="2" />
-  <xacro:chassis id="2" />
 </robot>

File: reseq_ros2/description/reseq_body.xacro (robot description, xacro)
@@ -1,8 +1,5 @@
 <?xml version="1.0"?>
 <robot xmlns:xacro="http://www.ros.org/wiki/xacro">
-  <!-- This is a parametric description of reseq with 4 modules -->
-  <!-- BASE LINK (center of equivalent wheel of module 1)-->
   <link name="base_link" />
-  <!-- CHASSIS1 -->
   <joint name="chassis1_joint" type="fixed">
     <parent link="base_link"/>
@@ -11,769 +8,6 @@
     <origin xyz="0 0 ${(EquivalentWheelDiameter-2*ChassisTopAndBottomClearance)/2+ChassisTopAndBottomClearance}"/>
   </joint>
-  <link name="chassis1_link">
-    <visual>
-      <origin xyz="${EquivalentWheelDiameter/12+(toll+JointDiameter/2)/2} 0 0"/>
-      <geometry>
-        <!-- leaving 1/3 of the EquivalentWheelDiameter from front and toll from Joint and Tracks (for clearance) -->
-        <box size="${WheelBase-JointDiameter/2-toll+EquivalentWheelDiameter*2/3-EquivalentWheelDiameter/2} ${ModuleWidth-2*TrackWidth-2*toll} ${EquivalentWheelDiameter-2*ChassisTopAndBottomClearance}"/>
-      </geometry>
-      <material name="ChassisColor"/>
-    </visual>
-    <collision>
-      <origin xyz="${EquivalentWheelDiameter/12+(toll+JointDiameter/2)/2} 0 0"/>
-      <geometry>
-        <!-- leaving 1/3 of the EquivalentWheelDiameter from front and toll from Joint and Tracks (for clearance) -->
-        <box size="${WheelBase-JointDiameter/2-toll+EquivalentWheelDiameter*2/3-EquivalentWheelDiameter/2} ${ModuleWidth-2*TrackWidth-2*toll} ${EquivalentWheelDiameter-2*ChassisTopAndBottomClearance}"/>
-      </geometry>
-    </collision>
-    <xacro:inertial_box mass="${ChassisMass}" x="${WheelBase-JointDiameter/2-toll+EquivalentWheelDiameter*2/3-EquivalentWheelDiameter/2}" y="${ModuleWidth-2*TrackWidth-2*toll}" z="${EquivalentWheelDiameter-2*ChassisTopAndBottomClearance}">
-      <origin xyz="${EquivalentWheelDiameter/12+(toll+JointDiameter/2)/2} 0 0" rpy="0 0 0"/>
-    </xacro:inertial_box>
-  </link>
-  <gazebo reference="chassis1_link">
-    <material>Gazebo/White</material>
-  </gazebo>
-  <!-- LEFT FRONT WHEEL 1-->
-  <joint name="left_front_wheel_1_joint" type="continuous">
-    <parent link="chassis1_link"/>
-    <child link="left_front_wheel_1_link"/>
-    <origin xyz="${WheelBase/2} ${ModuleWidth/2-TrackWidth/2} 0" rpy="-${pi/2} 0 0" />
-    <axis xyz="0 0 1"/>
-  </joint>
-  <link name="left_front_wheel_1_link">
-    <visual>
-      <geometry>
-        <cylinder radius="${EquivalentWheelDiameter/2}" length="${TrackWidth}"/>
-      </geometry>
-      <material name="WheelColor"/>
-    </visual>
-    <collision>
-      <geometry>
-        <cylinder radius="${EquivalentWheelDiameter/2}" length="${TrackWidth}"/>
-      </geometry>
-    </collision>
-    <xacro:inertial_cylinder mass="${WheelMass}" length="${TrackWidth}" radius="${EquivalentWheelDiameter/2}">
-      <origin xyz="0 0 0" rpy="0 0 0"/>
-    </xacro:inertial_cylinder>
-  </link>
-  <gazebo reference="left_front_wheel_1_link">
-    <material>Gazebo/Black</material>
-  </gazebo>
-  <!-- RIGHT FRONT WHEEL 1-->
-  <joint name="right_front_wheel_1_joint" type="continuous">
-    <parent link="chassis1_link"/>
-    <child link="right_front_wheel_1_link"/>
-    <origin xyz="${WheelBase/2} ${-ModuleWidth/2+TrackWidth/2} 0" rpy="${pi/2} 0 0" />
-    <axis xyz="0 0 -1"/>
-  </joint>
-  <link name="right_front_wheel_1_link">
-    <visual>
-      <geometry>
-        <cylinder radius="${EquivalentWheelDiameter/2}" length="${TrackWidth}"/>
-      </geometry>
-      <material name="WheelColor"/>
-    </visual>
-    <collision>
-      <geometry>
-        <cylinder radius="${EquivalentWheelDiameter/2}" length="${TrackWidth}"/>
-      </geometry>
-    </collision>
-    <xacro:inertial_cylinder mass="${WheelMass}" length="${TrackWidth}" radius="${EquivalentWheelDiameter/2}">
-      <origin xyz="0 0 0" rpy="0 0 0"/>
-    </xacro:inertial_cylinder>
-  </link>
-  <gazebo reference="right_front_wheel_1_link">
-    <material>Gazebo/Black</material>
-  </gazebo>
-  <!-- LEFT BACK WHEEL 1-->
-  <joint name="left_back_wheel_1_joint" type="continuous">
-    <parent link="chassis1_link"/>
-    <child link="left_back_wheel_1_link"/>
-    <origin xyz="${-WheelBase/2} ${ModuleWidth/2-TrackWidth/2} 0" rpy="-${pi/2} 0 0" />
-    <axis xyz="0 0 1"/>
-  </joint>
-  <link name="left_back_wheel_1_link">
-    <visual>
-      <geometry>
-        <cylinder radius="${EquivalentWheelDiameter/2}" length="${TrackWidth}"/>
-      </geometry>
-      <material name="WheelColor"/>
-    </visual>
-    <collision>
-      <geometry>
-        <cylinder radius="${EquivalentWheelDiameter/2}" length="${TrackWidth}"/>
-      </geometry>
-    </collision>
-    <xacro:inertial_cylinder mass="${WheelMass}" length="${TrackWidth}" radius="${EquivalentWheelDiameter/2}">
-      <origin xyz="0 0 0" rpy="0 0 0"/>
-    </xacro:inertial_cylinder>
-  </link>
-  <gazebo reference="left_back_wheel_1_link">
-    <material>Gazebo/Black</material>
-  </gazebo>
-  <!-- RIGHT BACK WHEEL 1-->
-  <joint name="right_back_wheel_1_joint" type="continuous">
-    <parent link="chassis1_link"/>
-    <child link="right_back_wheel_1_link"/>
-    <origin xyz="${-WheelBase/2} ${-ModuleWidth/2+TrackWidth/2} 0" rpy="${pi/2} 0 0" />
-    <axis xyz="0 0 -1"/>
-  </joint>
-  <link name="right_back_wheel_1_link">
-    <visual>
-      <geometry>
-        <cylinder radius="${EquivalentWheelDiameter/2}" length="${TrackWidth}"/>
-      </geometry>
-      <material name="WheelColor"/>
-    </visual>
-    <collision>
-      <geometry>
-        <cylinder radius="${EquivalentWheelDiameter/2}" length="${TrackWidth}"/>
-      </geometry>
-    </collision>
-    <xacro:inertial_cylinder mass="${WheelMass}" length="${TrackWidth}" radius="${EquivalentWheelDiameter/2}">
-      <origin xyz="0 0 0" rpy="0 0 0"/>
-    </xacro:inertial_cylinder>
-  </link>
-  <gazebo reference="right_back_wheel_1_link">
-    <material>Gazebo/Black</material>
-  </gazebo>
-  <!-- JointA 1-->
-  <joint name="joint_a_1_joint" type="revolute">
-    <parent link="chassis1_link"/>
-    <child link="joint_a_1_link"/>
-    <!-- Effort in Nm -->
-    <limit effort="20.0" lower="${-pitch}" upper="${pitch}" velocity="0.5"/>
-    <origin xyz="${-WheelBase/2} 0 0" rpy="${pi/2} 0 0" />
-    <axis xyz="0 0 -1"/>
-  </joint>
-  <link name="joint_a_1_link">
-    <!-- gearbox cilinder -->
-    <visual>
-      <geometry>
-        <cylinder radius="${JointDiameter/2}" length="${ModuleWidth-2*TrackWidth-toll*2}"/>
-      </geometry>
-      <material name="JointColor"/>
-    </visual>
-    <!-- horizontal shaft -->
-    <visual>
-      <origin xyz="${-JointA/2} 0 0" />
-      <geometry>
-        <box size="${JointA} ${EquivalentWheelDiameter-2*JointABottomClearance} ${ModuleWidth-2*TrackWidth-toll*2}"/>
-      </geometry>
-      <material name="JointColor"/>
-    </visual>
-    <!-- to hide space wile rotating -->
-    <visual>
-      <origin xyz="${-JointA} 0 0" />
-      <geometry>
-        <sphere radius="${(ModuleWidth-2*TrackWidth-toll*2)/2}"/>
-      </geometry>
-      <material name="JointColor"/>
-    </visual>
-    <!-- gearbox cilinder -->
-    <collision>
-      <geometry>
-        <cylinder radius="${JointDiameter/2}" length="${ModuleWidth-2*TrackWidth-toll*2}"/>
-      </geometry>
-    </collision>
-    <!-- horizontal shaft -->
-    <collision>
-      <origin xyz="${-JointA/2} 0 0" />
-      <geometry>
-        <box size="${JointA} ${EquivalentWheelDiameter-2*JointABottomClearance} ${ModuleWidth-2*TrackWidth-toll*2}"/>
-      </geometry>
-    </collision>
-    <xacro:inertial_box mass="${JointAMass}" x="${JointA}" y="${EquivalentWheelDiameter-2*JointABottomClearance}" z="${ModuleWidth-2*TrackWidth-toll*2}">
-      <origin xyz="${-JointA/2} 0 0" rpy="0 0 0"/>
-    </xacro:inertial_box>
-  </link>
-  <gazebo reference="joint_a_1_link">
-    <material>Gazebo/Grey</material>
-  </gazebo>
-  <!-- JointB 1-->
-  <joint name="joint_b_1_joint" type="revolute">
-    <parent link="joint_a_1_link"/>
-    <child link="joint_b_1_link"/>
-    <!-- Effort in Nm -->
-    <limit effort="20.0" lower="${-yaw}" upper="${yaw}" velocity="0.5"/>
-    <origin xyz="${-JointA} 0 0" rpy="0 ${pi/2} 0" />
-    <axis xyz="0 1 0"/>
-  </joint>
-  <link name="joint_b_1_link">
-    <visual>
-      <origin xyz="0 0 -${JointB/2}" />
-      <geometry>
-        <cylinder radius="${(ModuleWidth-2*TrackWidth-toll*2)/2}" length="${JointB}"/>
-      </geometry>
-      <material name="JointColor"/>
-    </visual>
-    <xacro:inertial_cylinder mass="${JointBMass}" length="${JointB}" radius="${(ModuleWidth-2*TrackWidth-toll*2)/2}">
-      <origin xyz="0 0 ${-(JointB-WheelBase/2-EquivalentWheelDiameter/6)/2}" rpy="0 0 0"/>
-    </xacro:inertial_cylinder>
-  </link>
-  <gazebo reference="joint_b_1_link">
-    <material>Gazebo/Grey</material>
-  </gazebo>
-  <!-- CHASSIS2 -->
-  <joint name="chassis2_joint" type="revolute">
-    <parent link="joint_b_1_link"/>
-    <child link="chassis2_link"/>
-    <!-- Effort in Nm -->
-    <limit effort="2.0" lower="${-roll}" upper="${roll}" velocity="0.5"/>
-    <origin xyz="0 0 -${JointB+WheelBase/2}" rpy="${-pi/2} ${-pi/2} 0"/>
-    <axis xyz="1 0 0"/>
-  </joint>
-  <link name="chassis2_link">
-    <visual>
-      <origin xyz="${EquivalentWheelDiameter/12+(toll+JointDiameter/2)/2} 0 0"/>
-      <geometry>
-        <!-- leaving 1/3 of the EquivalentWheelDiameter from front and toll from Joint and Tracks (for clearance) -->
-        <box size="${WheelBase-JointDiameter/2-toll+EquivalentWheelDiameter*2/3-EquivalentWheelDiameter/2} ${ModuleWidth-2*TrackWidth-2*toll} ${EquivalentWheelDiameter-2*ChassisTopAndBottomClearance}"/>
-      </geometry>
-      <material name="ChassisColor"/>
-    </visual>
-    <collision>
-      <origin xyz="${EquivalentWheelDiameter/12+(toll+JointDiameter/2)/2} 0 0"/>
-      <geometry>
-        <!-- leaving 1/3 of the EquivalentWheelDiameter from front and toll from Joint and Tracks (for clearance) -->
-        <box size="${WheelBase-JointDiameter/2-toll+EquivalentWheelDiameter*2/3-EquivalentWheelDiameter/2} ${ModuleWidth-2*TrackWidth-2*toll} ${EquivalentWheelDiameter-2*ChassisTopAndBottomClearance}"/>
-      </geometry>
-    </collision>
-    <xacro:inertial_box mass="${ChassisMass}" x="${WheelBase-JointDiameter/2-toll+EquivalentWheelDiameter*2/3-EquivalentWheelDiameter/2}" y="${ModuleWidth-2*TrackWidth-2*toll}" z="${EquivalentWheelDiameter-2*ChassisTopAndBottomClearance}">
-      <origin xyz="${EquivalentWheelDiameter/12+(toll+JointDiameter/2)/2} 0 0" rpy="0 0 0"/>
-    </xacro:inertial_box>
-  </link>
-  <gazebo reference="chassis2_link">
-    <material>Gazebo/White</material>
-  </gazebo>
-  <!-- LEFT FRONT WHEEL 2-->
-  <joint name="left_front_wheel_2_joint" type="continuous">
-    <parent link="chassis2_link"/>
-    <child link="left_front_wheel_2_link"/>
-    <origin xyz="${WheelBase/2} ${ModuleWidth/2-TrackWidth/2} 0" rpy="-${pi/2} 0 0" />
-    <axis xyz="0 0 1"/>
-  </joint>
-  <link name="left_front_wheel_2_link">
-    <visual>
-      <geometry>
-        <cylinder radius="${EquivalentWheelDiameter/2}" length="${TrackWidth}"/>
-      </geometry>
-      <material name="WheelColor"/>
-    </visual>
-    <collision>
-      <geometry>
-        <cylinder radius="${EquivalentWheelDiameter/2}" length="${TrackWidth}"/>
-      </geometry>
-    </collision>
-    <xacro:inertial_cylinder mass="${WheelMass}" length="${TrackWidth}" radius="${EquivalentWheelDiameter/2}">
-      <origin xyz="0 0 0" rpy="0 0 0"/>
-    </xacro:inertial_cylinder>
-  </link>
-  <gazebo reference="left_front_wheel_2_link">
-    <material>Gazebo/Black</material>
-  </gazebo>
-  <!-- RIGHT FRONT WHEEL 2-->
-  <joint name="right_front_wheel_2_joint" type="continuous">
-    <parent link="chassis2_link"/>
-    <child link="right_front_wheel_2_link"/>
-    <origin xyz="${WheelBase/2} ${-ModuleWidth/2+TrackWidth/2} 0" rpy="${pi/2} 0 0" />
-    <axis xyz="0 0 -1"/>
-  </joint>
-  <link name="right_front_wheel_2_link">
-    <visual>
-      <geometry>
-        <cylinder radius="${EquivalentWheelDiameter/2}" length="${TrackWidth}"/>
-      </geometry>
-      <material name="WheelColor"/>
-    </visual>
-    <collision>
-      <geometry>
-        <cylinder radius="${EquivalentWheelDiameter/2}" length="${TrackWidth}"/>
-      </geometry>
-    </collision>
-    <xacro:inertial_cylinder mass="${WheelMass}" length="${TrackWidth}" radius="${EquivalentWheelDiameter/2}">
-      <origin xyz="0 0 0" rpy="0 0 0"/>
-    </xacro:inertial_cylinder>
-  </link>
-  <gazebo reference="right_front_wheel_2_link">
-    <material>Gazebo/Black</material>
-  </gazebo>
-  <!-- LEFT BACK WHEEL 2-->
-  <joint name="left_back_wheel_2_joint" type="continuous">
-    <parent link="chassis2_link"/>
-    <child link="left_back_wheel_2_link"/>
-    <origin xyz="${-WheelBase/2} ${ModuleWidth/2-TrackWidth/2} 0" rpy="-${pi/2} 0 0" />
-    <axis xyz="0 0 1"/>
-  </joint>
-  <link name="left_back_wheel_2_link">
-    <visual>
-      <geometry>
-        <cylinder radius="${EquivalentWheelDiameter/2}" length="${TrackWidth}"/>
-      </geometry>
-      <material name="WheelColor"/>
-    </visual>
-    <collision>
-      <geometry>
-        <cylinder radius="${EquivalentWheelDiameter/2}" length="${TrackWidth}"/>
-      </geometry>
-    </collision>
-    <xacro:inertial_cylinder mass="${WheelMass}" length="${TrackWidth}" radius="${EquivalentWheelDiameter/2}">
-      <origin xyz="0 0 0" rpy="0 0 0"/>
-    </xacro:inertial_cylinder>
-  </link>
-  <gazebo reference="left_back_wheel_2_link">
-    <material>Gazebo/Black</material>
-  </gazebo>
-  <!-- RIGHT BACK WHEEL 2-->
-  <joint name="right_back_wheel_2_joint" type="continuous">
-    <parent link="chassis2_link"/>
-    <child link="right_back_wheel_2_link"/>
-    <origin xyz="${-WheelBase/2} ${-ModuleWidth/2+TrackWidth/2} 0" rpy="${pi/2} 0 0" />
-    <axis xyz="0 0 -1"/>
-  </joint>
-  <link name="right_back_wheel_2_link">
-    <visual>
-      <geometry>
-        <cylinder radius="${EquivalentWheelDiameter/2}" length="${TrackWidth}"/>
-      </geometry>
-      <material name="WheelColor"/>
-    </visual>
-    <collision>
-      <geometry>
-        <cylinder radius="${EquivalentWheelDiameter/2}" length="${TrackWidth}"/>
-      </geometry>
-    </collision>
-    <xacro:inertial_cylinder mass="${WheelMass}" length="${TrackWidth}" radius="${EquivalentWheelDiameter/2}">
-      <origin xyz="0 0 0" rpy="0 0 0"/>
-    </xacro:inertial_cylinder>
-  </link>
-  <gazebo reference="right_back_wheel_2_link">
-    <material>Gazebo/Black</material>
-  </gazebo>
-  <!-- JointA 2-->
-  <joint name="joint_a_2_joint" type="revolute">
-    <parent link="chassis2_link"/>
-    <child link="joint_a_2_link"/>
-    <!-- Effort in Nm -->
-    <limit effort="20.0" lower="${-pitch}" upper="${pitch}" velocity="0.5"/>
-    <origin xyz="${-WheelBase/2} 0 0" rpy="${pi/2} 0 0" />
-    <axis xyz="0 0 -1"/>
-  </joint>
-  <link name="joint_a_2_link">
-    <!-- gearbox cilinder -->
-    <visual>
-      <geometry>
-        <cylinder radius="${JointDiameter/2}" length="${ModuleWidth-2*TrackWidth-toll*2}"/>
-      </geometry>
-      <material name="JointColor"/>
-    </visual>
-    <!-- horizontal shaft -->
-    <visual>
-      <origin xyz="${-JointA/2} 0 0" />
-      <geometry>
-        <box size="${JointA} ${EquivalentWheelDiameter-2*JointABottomClearance} ${ModuleWidth-2*TrackWidth-toll*2}"/>
-      </geometry>
-      <material name="JointColor"/>
-    </visual>
-    <!-- to hide space wile rotating -->
-    <visual>
-      <origin xyz="${-JointA} 0 0" />
-      <geometry>
-        <sphere radius="${(ModuleWidth-2*TrackWidth-toll*2)/2}"/>
-      </geometry>
-      <material name="JointColor"/>
-    </visual>
-    <!-- gearbox cilinder -->
-    <collision>
-      <geometry>
-        <cylinder radius="${JointDiameter/2}" length="${ModuleWidth-2*TrackWidth-toll*2}"/>
-      </geometry>
-    </collision>
-    <!-- horizontal shaft -->
-    <collision>
-      <origin xyz="${-JointA/2} 0 0" />
-      <geometry>
-        <box size="${JointA} ${EquivalentWheelDiameter-2*JointABottomClearance} ${ModuleWidth-2*TrackWidth-toll*2}"/>
-      </geometry>
-    </collision>
-    <xacro:inertial_box mass="${JointAMass}" x="${JointA}" y="${EquivalentWheelDiameter-2*JointABottomClearance}" z="${ModuleWidth-2*TrackWidth-toll*2}">
-      <origin xyz="${-JointA/2} 0 0" rpy="0 0 0"/>
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
File: reseq_ros2/description/robot.urdf.xacro (robot description, xacro)
@@ -5,8 +5,9 @@
   <xacro:include filename="inertial_macros.xacro" />
   <xacro:include filename="reseq_parameters.xacro" />
-  <!-- <xacro:include filename="components.xacro"/>
-  <xacro:include filename="module_body.xacro" /> -->
+  <xacro:include filename="macros/utils.xacro" />
+  <xacro:include filename="macros/joint.xacro" />
+  <xacro:include filename="macros/chassis.xacro" />
   <xacro:include filename="reseq_body.xacro" />
-  <!-- <xacro:include filename="reseq_arm_mk1.xacro" /> -->
-  <!-- <xacro:include filename="lidar.xacro" /> -->
+  <xacro:include filename="reseq_arm_mk1.xacro" />
+  <xacro:include filename="lidar.xacro" />
 </robot>
