Commit message: feat: Implement macro for wheels

File: reseq_ros2/description/macros/chassis.xacro (robot description, xacro)
@@ -26,100 +26,9 @@
       </xacro:inertial_box>
     </link>
-    <!-- LEFT FRONT WHEEL 1-->
-    <joint name="left_front_wheel_${id}_joint" type="continuous">
-      <parent link="chassis${id}_link" />
-      <child link="left_front_wheel_${id}_link" />
-      <origin xyz="${WheelBase/2} ${ModuleWidth/2-TrackWidth/2} 0" rpy="-${pi/2} 0 0" />
-      <axis xyz="0 0 1" />
-    </joint>
-    <link name="left_front_wheel_${id}_link">
-      <visual>
-        <geometry>
-          <cylinder radius="${EquivalentWheelDiameter/2}" length="${TrackWidth}" />
-        </geometry>
-        <material name="WheelColor" />
-      </visual>
-      <collision>
-        <geometry>
-          <cylinder radius="${EquivalentWheelDiameter/2}" length="${TrackWidth}" />
-        </geometry>
-      </collision>
-      <xacro:inertial_cylinder mass="${WheelMass}" length="${TrackWidth}"
-        radius="${EquivalentWheelDiameter/2}">
-        <origin xyz="0 0 0" rpy="0 0 0" />
-      </xacro:inertial_cylinder>
-    </link>
-    <!-- RIGHT FRONT WHEEL 1-->
-    <joint name="right_front_wheel_${id}_joint" type="continuous">
-      <parent link="chassis${id}_link" />
-      <child link="right_front_wheel_${id}_link" />
-      <origin xyz="${WheelBase/2} ${-ModuleWidth/2+TrackWidth/2} 0" rpy="${pi/2} 0 0" />
-      <axis xyz="0 0 -1" />
-    </joint>
-    <link name="right_front_wheel_${id}_link">
-      <visual>
-        <geometry>
-          <cylinder radius="${EquivalentWheelDiameter/2}" length="${TrackWidth}" />
-        </geometry>
-        <material name="WheelColor" />
-      </visual>
-      <collision>
-        <geometry>
-          <cylinder radius="${EquivalentWheelDiameter/2}" length="${TrackWidth}" />
-        </geometry>
-      </collision>
-      <xacro:inertial_cylinder mass="${WheelMass}" length="${TrackWidth}"
-        radius="${EquivalentWheelDiameter/2}">
-        <origin xyz="0 0 0" rpy="0 0 0" />
-      </xacro:inertial_cylinder>
-    </link>
-    <!-- LEFT BACK WHEEL 1-->
-    <joint name="left_back_wheel_${id}_joint" type="continuous">
-      <parent link="chassis${id}_link" />
-      <child link="left_back_wheel_${id}_link" />
-      <origin xyz="${-WheelBase/2} ${ModuleWidth/2-TrackWidth/2} 0" rpy="-${pi/2} 0 0" />
-      <axis xyz="0 0 1" />
-    </joint>
-    <link name="left_back_wheel_${id}_link">
-      <visual>
-        <geometry>
-          <cylinder radius="${EquivalentWheelDiameter/2}" length="${TrackWidth}" />
-        </geometry>
-        <material name="WheelColor" />
-      </visual>
-      <collision>
-        <geometry>
-          <cylinder radius="${EquivalentWheelDiameter/2}" length="${TrackWidth}" />
-        </geometry>
-      </collision>
-      <xacro:inertial_cylinder mass="${WheelMass}" length="${TrackWidth}"
-        radius="${EquivalentWheelDiameter/2}">
-        <origin xyz="0 0 0" rpy="0 0 0" />
-      </xacro:inertial_cylinder>
-    </link>
-    <!-- RIGHT BACK WHEEL 1-->
-    <joint name="right_back_wheel_${id}_joint" type="continuous">
-      <parent link="chassis${id}_link" />
-      <child link="right_back_wheel_${id}_link" />
-      <origin xyz="${-WheelBase/2} ${-ModuleWidth/2+TrackWidth/2} 0" rpy="${pi/2} 0 0" />
-      <axis xyz="0 0 -1" />
-    </joint>
-    <link name="right_back_wheel_${id}_link">
-      <visual>
-        <geometry>
-          <cylinder radius="${EquivalentWheelDiameter/2}" length="${TrackWidth}" />
-        </geometry>
-        <material name="WheelColor" />
-      </visual>
-      <collision>
-        <geometry>
-          <cylinder radius="${EquivalentWheelDiameter/2}" length="${TrackWidth}" />
-        </geometry>
-      </collision>
-      <xacro:inertial_cylinder mass="${WheelMass}" length="${TrackWidth}"
-        radius="${EquivalentWheelDiameter/2}">
-        <origin xyz="0 0 0" rpy="0 0 0" />
-      </xacro:inertial_cylinder>
-    </link>
+    <!-- Wheels -->
+    <xacro:wheel_factory id="${id}" pos="front" side="left" />
+    <xacro:wheel_factory id="${id}" pos="front" side="right" />
+    <xacro:wheel_factory id="${id}" pos="back" side="left" />
+    <xacro:wheel_factory id="${id}" pos="back" side="right" />
   </xacro:macro>
 </robot>

File: reseq_ros2/description/robot.urdf.xacro (robot description, xacro)
@@ -8,4 +8,5 @@
   <xacro:include filename="macros/joint.xacro" />
   <xacro:include filename="macros/chassis.xacro" />
+  <xacro:include filename="macros/wheel.xacro" />
   <xacro:include filename="reseq_body.xacro" />
   <xacro:include filename="reseq_arm_mk1.xacro" />

Commit message: feat: add missing gazebo reference

File: reseq_ros2/description/macros/chassis.xacro (robot description, xacro)
@@ -26,4 +26,7 @@
       </xacro:inertial_box>
     </link>
+    <gazebo reference="chassis${id}_link">
+      <material>Gazebo/White</material>
+    </gazebo>
     <!-- Wheels -->
     <xacro:wheel_factory id="${id}" pos="front" side="left" />

File: reseq_ros2/description/macros/joint.xacro (robot description, xacro)
@@ -28,4 +28,7 @@
       </xacro:replicate_collision>
     </link>
+    <gazebo reference="joint_r_${id}_link">
+      <material>Gazebo/Grey</material>
+    </gazebo>
     <!-- JointY -->
     <joint name="joint_y_${id}_joint" type="revolute">
@@ -59,4 +62,7 @@
       </xacro:replicate_collision>
     </link>
+    <gazebo reference="joint_y_${id}_link">
+      <material>Gazebo/Grey</material>
+    </gazebo>
     <!-- JointP -->
     <joint name="joint_p_${id}_joint" type="revolute">
@@ -80,4 +86,7 @@
       </xacro:replicate_collision>
     </link>
+    <gazebo reference="joint_p_${id}_link">
+      <material>Gazebo/Grey</material>
+    </gazebo>
     <joint name="chassis${id}_joint" type="fixed">
       <parent link="joint_p_${id}_link" />

File: reseq_ros2/description/macros/wheel.xacro (robot description, xacro)
@@ -41,4 +41,7 @@
         </xacro:inertial_cylinder>
         </link>
+        <gazebo reference="${side}_${pos}_wheel_${id}_link">
+            <material>Gazebo/Black</material>
+        </gazebo>
     </xacro:macro>
 </robot>

File: reseq_ros2/description/reseq_arm_mk1.xacro (robot description, xacro)
@@ -96,4 +96,7 @@
   <link name="arm_camera_holder_intermediate">
   </link>
+  <gazebo reference="arm_camera_holder_intermediate">
+    <material>Gazebo/Grey</material>
+  </gazebo>
   <!-- head roll joint -->
   <joint name="arm_head_roll_1_joint" type="revolute">
@@ -137,4 +140,7 @@
     </xacro:replicate_collision>
   </link>
+  <gazebo reference="arm_camera_holder">
+    <material>Gazebo/Grey</material>
+  </gazebo>
   <joint name="arm_camera_joint" type="fixed">
     <parent link="arm_camera_holder"/>
@@ -146,5 +152,5 @@
   <link name="camera_link">
   </link>
-  <gazebo reference="arm_mK1_link">
+  <gazebo reference="camera_link">
     <material>Gazebo/Grey</material>
   </gazebo>
