Commit message: fix: Rotate also collision and inertial cylinder

File: reseq_ros2/description/macros/wheel.xacro (robot description, xacro)
@@ -24,5 +24,5 @@
         <link name="${side}_${pos}_wheel_${id}_link">
         <visual>
-            <origin xyz="0 0 0"  rpy="${-side_sign*pi/2} 0 0"/>
+            <origin xyz="0 0 0" rpy="${-side_sign*pi/2} 0 0"/>
             <geometry>
             <cylinder radius="${EquivalentWheelDiameter/2}" length="${TrackWidth}" />
@@ -31,4 +31,5 @@
         </visual>
         <collision>
+            <origin xyz="0 0 0" rpy="${-side_sign*pi/2} 0 0"/>
             <geometry>
             <cylinder radius="${EquivalentWheelDiameter/2}" length="${TrackWidth}" />
@@ -37,5 +38,5 @@
         <xacro:inertial_cylinder mass="${WheelMass}" length="${TrackWidth}"
             radius="${EquivalentWheelDiameter/2}">
-            <origin xyz="0 0 0" rpy="0 0 0" />
+            <origin xyz="0 0 0" rpy="${-side_sign*pi/2} 0 0"/>
         </xacro:inertial_cylinder>
         </link>

Commit message: fix: Rotate wheel around Y axis
Co-authored-by: Luca De Paola <60526200+luca-byte@users.noreply.github.com>

File: reseq_ros2/description/macros/wheel.xacro (robot description, xacro)
@@ -20,5 +20,5 @@
         <child link="${side}_${pos}_wheel_${id}_link" />
         <origin xyz="${pos_sign*WheelBase/2} ${side_sign*(ModuleWidth/2-TrackWidth/2)} 0" rpy="0 0 0" />
-        <axis xyz="0 0 ${side_sign}" />
+        <axis xyz="0 1 0" />
         </joint>
         <link name="${side}_${pos}_wheel_${id}_link">

Commit message: fix: Rotate all wheels in the same direction
Rotating the link depending on the side was correct but also useless.
For simplicity, we've decided to avoid it.

File: reseq_ros2/description/macros/wheel.xacro (robot description, xacro)
@@ -24,5 +24,5 @@
         <link name="${side}_${pos}_wheel_${id}_link">
         <visual>
-            <origin xyz="0 0 0" rpy="${-side_sign*pi/2} 0 0"/>
+            <origin xyz="0 0 0" rpy="${pi/2} 0 0" />
             <geometry>
             <cylinder radius="${EquivalentWheelDiameter/2}" length="${TrackWidth}" />
@@ -31,5 +31,5 @@
         </visual>
         <collision>
-            <origin xyz="0 0 0" rpy="${-side_sign*pi/2} 0 0"/>
+            <origin xyz="0 0 0" rpy="${pi/2} 0 0" />
             <geometry>
             <cylinder radius="${EquivalentWheelDiameter/2}" length="${TrackWidth}" />
@@ -38,5 +38,5 @@
         <xacro:inertial_cylinder mass="${WheelMass}" length="${TrackWidth}"
             radius="${EquivalentWheelDiameter/2}">
-            <origin xyz="0 0 0" rpy="${-side_sign*pi/2} 0 0"/>
+            <origin xyz="0 0 0" rpy="${pi/2} 0 0" />
         </xacro:inertial_cylinder>
         </link>

Commit message: feat(gz): added friction coefficients to wheels

File: reseq_ros2/description/macros/wheel.xacro (robot description, xacro)
@@ -43,4 +43,10 @@
         <gazebo reference="${side}_${pos}_wheel_${id}_link">
             <material>Gazebo/Black</material>
+            <!-- mu1 and mu2 are two respectively friction coefficients for respectively primary
+                 direction and the secondary direction. the secondary direction is perpendicular to
+                 the primary direction. mu1 is important for forward/backward grip, while mu2 is
+                 critical for sideways grip (you dont want the model to slip when it turns)  -->
+            <mu1 value="${WheelMu1}"/>
+            <mu2 value="${WheelMu2}"/>
         </gazebo>
     </xacro:macro>

File: reseq_ros2/description/reseq_parameters.xacro (robot description, xacro)
@@ -14,4 +14,6 @@
   <xacro:property name="NumModules" value="${config['num_modules']}"/>
   <xacro:property name="WheelBase" value="${config['xacro']['WheelBase']}"/>
+  <xacro:property name="WheelMu1" value="${config['xacro']['WheelMu1']}"/>
+  <xacro:property name="WheelMu2" value="${config['xacro']['WheelMu2']}"/>
   <xacro:property name="EquivalentWheelDiameter" value="${r_eq*2}"/>
   <xacro:property name="ModuleWidth" value="${config['xacro']['ModuleWidth']}"/>

Commit message: fix(gz): No need for friction coefficients

File: reseq_ros2/description/macros/wheel.xacro (robot description, xacro)
@@ -43,10 +43,4 @@
         <gazebo reference="${side}_${pos}_wheel_${id}_link">
             <material>Gazebo/Black</material>
-            <!-- mu1 and mu2 are two respectively friction coefficients for respectively primary
-                 direction and the secondary direction. the secondary direction is perpendicular to
-                 the primary direction. mu1 is important for forward/backward grip, while mu2 is
-                 critical for sideways grip (you dont want the model to slip when it turns)  -->
-            <mu1 value="${WheelMu1}"/>
-            <mu2 value="${WheelMu2}"/>
         </gazebo>
     </xacro:macro>

File: reseq_ros2/description/reseq_parameters.xacro (robot description, xacro)
@@ -14,6 +14,4 @@
   <xacro:property name="NumModules" value="${config['num_modules']}"/>
   <xacro:property name="WheelBase" value="${config['xacro']['WheelBase']}"/>
-  <xacro:property name="WheelMu1" value="${config['xacro']['WheelMu1']}"/>
-  <xacro:property name="WheelMu2" value="${config['xacro']['WheelMu2']}"/>
   <xacro:property name="EquivalentWheelDiameter" value="${r_eq*2}"/>
   <xacro:property name="ModuleWidth" value="${config['xacro']['ModuleWidth']}"/>
