Commit message: fix(gz): Rename of modules control joint

File: reseq_ros2/description/macros/control_chassis_joint.xacro (robot description, xacro)
@@ -6,11 +6,11 @@
     -->
     <xacro:macro name="control_chassis_joint_factory" params="id">
-        <joint name="joint_y_${id}_joint">
+        <joint name="mod${id}__yaw_joint">
             <state_interface name="position" />
         </joint>
-        <joint name="joint_r_${id}_joint">
+        <joint name="mod${id}__roll_joint">
             <state_interface name="position" />
         </joint>
-        <joint name="joint_p_${id}_joint">
+        <joint name="mod${id}__pitch_joint">
             <state_interface name="position" />
         </joint>
