Commit message: feat(HW): Update names of ROS2C nodes for consistency and identifiability

File: reseq_ros2/description/macros/control_macros.xacro (robot description, xacro)
@@ -8,5 +8,5 @@
     -->
     <xacro:macro name="control_wheel_factory" params="id pos side">
-        <joint name="${side}_${pos}_wheel_${id}_joint">
+        <joint name="mod${id}__${side}_${pos}_wheel">
             <command_interface name="velocity" />
             <state_interface name="velocity" />
@@ -18,11 +18,11 @@
     -->
     <xacro:macro name="control_joint_factory" params="id">
-        <joint name="joint_r_${id}_joint">
+        <joint name="mod${id}__roll_joint">
             <state_interface name="position" />
         </joint>
-        <joint name="joint_p_${id}_joint">
+        <joint name="mod${id}__pitch_joint">
             <state_interface name="position" />
         </joint>
-        <joint name="joint_y_${id}_joint">
+        <joint name="mod${id}__yaw_joint">
             <state_interface name="position" />
         </joint>

File: reseq_ros2/description/macros/joint.xacro (robot description, xacro)
@@ -9,5 +9,5 @@
   <xacro:macro name="chassis_joint_factory" params="id">
     <!-- JointR -->
-    <joint name="joint_r_${id}_joint" type="revolute">
+    <joint name="mod${id}__roll_joint" type="revolute">
       <parent link="chassis${id-1}_link" />
       <child link="joint_r_${id}_link" />
@@ -29,5 +29,5 @@
     </link>
     <!-- JointY -->
-    <joint name="joint_y_${id}_joint" type="revolute">
+    <joint name="mod${id}__yaw_joint" type="revolute">
       <parent link="joint_r_${id}_link" />
       <child link="joint_y_${id}_link" />
@@ -60,5 +60,5 @@
     </link>
     <!-- JointP -->
-    <joint name="joint_p_${id}_joint" type="revolute">
+    <joint name="mod${id}__pitch_joint" type="revolute">
       <parent link="joint_y_${id}_link" />
       <child link="joint_p_${id}_link" />

File: reseq_ros2/description/macros/wheel.xacro (robot description, xacro)
@@ -16,5 +16,5 @@
             <xacro:property name="side_sign" value="-1" />
         </xacro:if>
-        <joint name="${side}_${pos}_wheel_${id}_joint" type="continuous">
+        <joint name="mod${id}__${side}_${pos}_wheel" type="continuous">
         <parent link="chassis${id}_link" />
         <child link="${side}_${pos}_wheel_${id}_link" />

Commit message: fix: Control chassis joint useless

File: reseq_ros2/description/macros/control_macros.xacro (robot description, xacro)
@@ -9,4 +9,6 @@
     <xacro:macro name="control_wheel_factory" params="id pos side">
         <joint name="mod${id}__${side}_${pos}_wheel">
+            <command_interface name="position" />
+            <state_interface name="position" />
             <command_interface name="velocity" />
             <state_interface name="velocity" />

File: reseq_ros2/description/robot.urdf.xacro (robot description, xacro)
@@ -11,5 +11,4 @@
   <xacro:include filename="macros/wheel.xacro" />
   <xacro:include filename="macros/control_macros.xacro" />
-  <xacro:include filename="macros/control_chassis_joint.xacro"/>
   <xacro:include filename="reseq_body.xacro" />
   <xacro:if value="${config['version'] == 'mk1'}">

File: reseq_ros2/description/ros2_control.xacro (robot description, xacro)
@@ -3,5 +3,6 @@
     <ros2_control name="ReseqHardwareSystem" type="system">
         <hardware>
-            <plugin>reseq_hardware/ReseqHardware</plugin>
+            <!-- <plugin>reseq_hardware/ReseqHardware</plugin> -->
+            <plugin>gz_ros2_control/GazeboSimSystem</plugin>
             <param name="num_modules">${NumModules}</param>
             <!-- TODO: vcan, and gazebo alternatives -->
@@ -24,29 +25,4 @@
         <xacro:loop module="1" n_modules="${NumModules}" />
     </ros2_control>
-    <ros2_control name="GazeboSimSystem" type="system">
-        <hardware>
-            <plugin>gz_ros2_control/GazeboSimSystem</plugin>
-        </hardware>
-        <!-- Create n_modules modules by recursively calling the loop macro -->
-        <xacro:macro name="loop" params="module n_modules">
-            <xacro:if value="${module &lt;= n_modules}">
-                <!-- Wheels -->
-                <xacro:control_wheel_factory id="${module}" pos="front" side="left" />
-                <xacro:control_wheel_factory id="${module}" pos="front" side="right" />
-                <xacro:control_wheel_factory id="${module}" pos="back" side="left" />
-                <xacro:control_wheel_factory id="${module}" pos="back" side="right" />
-                <xacro:loop module="${module + 1}" n_modules="${n_modules}"/>
-            </xacro:if>
-        </xacro:macro>
-        <xacro:loop module="1" n_modules="${NumModules}"/>
-        <!-- Create n_modules modules by recursively calling the loop macro -->
-        <xacro:macro name="loop2" params="module n_modules">
-            <xacro:if value="${module &lt; n_modules}">
-                <xacro:control_chassis_joint_factory id="${module + 1}"/>
-                <xacro:loop2 module="${module + 1}" n_modules="${n_modules}"/>
-            </xacro:if>
-        </xacro:macro>
-        <xacro:loop2 module="1" n_modules="${NumModules}"/>
-    </ros2_control>
     <gazebo>
         <plugin name="gz_ros2_control::GazeboSimROS2ControlPlugin" filename="libgz_ros2_control-system.so">
