Commit message: chore: modify URDF ranges to improve arm maneuverability

File: reseq_ros2/config/reseq_mk2_arm/simplified_arm_assembly.urdf (robot description, URDF)
Before this commit: robot simplified_arm_assembly, 8 links, 7 joints
Joints:
- joint pitch_joint_1: limit lower=-1.309 upper=1.309 effort=6 velocity=2 -> lower=-3.14 upper=1.309 effort=6 velocity=2
- joint roll_joint_2: limit lower=0 upper=6.28 effort=6 velocity=2 -> lower=-6.28 upper=6.28 effort=6 velocity=2
- joint roll_joint_4: limit lower=0 upper=6.28 effort=3 velocity=1 -> lower=-6.28 upper=6.28 effort=3 velocity=1

Commit message: fix: fix URDF meshes directory

File: reseq_ros2/config/reseq_mk2_arm/simplified_arm_assembly.urdf (robot description, URDF)
Before this commit: robot simplified_arm_assembly, 8 links, 7 joints
Links:
- link module_joint: geometry collision mesh filename=package://reseq_ros2/description/meshes/module_joint.STL; visual mesh filename=package://reseq_ros2/description/meshes/module_joint.STL
- link pitch_1: geometry collision mesh filename=package://reseq_ros2/description/meshes/pitch_1.STL; visual mesh filename=package://reseq_ros2/description/meshes/pitch_1.STL
- link pitch_3: geometry collision mesh filename=package://reseq_ros2/description/meshes/pitch_3.STL; visual mesh filename=package://reseq_ros2/description/meshes/pitch_3.STL
- link pitch_5: geometry collision mesh filename=package://reseq_ros2/description/meshes/pitch_5.STL; visual mesh filename=package://reseq_ros2/description/meshes/pitch_5.STL
- link roll_2: geometry collision mesh filename=package://reseq_ros2/description/meshes/roll_2.STL; visual mesh filename=package://reseq_ros2/description/meshes/roll_2.STL
- link roll_4: geometry collision mesh filename=package://reseq_ros2/description/meshes/roll_4.STL; visual mesh filename=package://reseq_ros2/description/meshes/roll_4.STL
- link roll_6: geometry collision mesh filename=package://reseq_ros2/description/meshes/roll_6.STL; visual mesh filename=package://reseq_ros2/description/meshes/roll_6.STL
