Commit message: chore(description): Refactor of robot description

File: reseq_description/description/arm_mk1/reseq_arm_mk1.xacro (robot description, xacro)
@@ -3,4 +3,24 @@
   <!-- This is a parametric description of reseq mK1 arm -->
   <!-- TODO: Add arm joints to the HW Interface -->
+  <!-- PARAMETERS -->
+  <xacro:property name="ForkThickness" value="0.02"/>
+  <xacro:property name="ForkHeight" value="0.05"/>
+  <xacro:property name="JetsonHolderWidth" value="0.085"/>
+  <xacro:property name="JetsonHolderLength" value="0.158"/>
+  <xacro:property name="CylinderOnJetsonLength" value="0.085"/>
+  <xacro:property name="CylinderOnJetsonRadius" value="0.026"/>
+  <xacro:property name="CylinderOnJetsonShift" value="0.012"/>
+  <xacro:property name="CylinderRealsenseLength" value="0.055"/>
+  <xacro:property name="CylinderRealsenseRadius" value="0.026"/>
+  <xacro:property name="RealsenseHeight" value="0.02"/>
+  <xacro:property name="RealsenseLength" value="0.026"/>
+  <xacro:property name="RealsenseWidth" value="0.09"/>
+  <xacro:property name="RealsenseOriginSystem" value="0.0162"/>
+  <!-- XACRO INCLUDES -->
+  <xacro:include filename="../sensors/rgbd_camera.xacro" />
+  <!-- Rviz colors (for Gazebo ones change in single files) (from 0 to 1) -->
+  <material name="ArmColor">
+    <color rgba="0.5 0.5 0.5 1" />
+  </material>
   <joint name="arm_pitch_1_joint" type="revolute">
     <parent link="chassis1_link"/>

File: reseq_description/description/reseq_body.xacro (robot description, xacro)
@@ -1,4 +1,10 @@
 <?xml version="1.0"?>
 <robot xmlns:xacro="http://www.ros.org/wiki/xacro">
+  <!-- INCLUDE MACROS FOR THE BODY -->
+  <xacro:include filename="macros/joint.xacro" />
+  <xacro:include filename="macros/chassis.xacro" />
+  <xacro:include filename="macros/wheel.xacro" />
+  <xacro:include filename="macros/control_macros.xacro" />
+  <xacro:include filename="sensors/lidar.xacro" />
   <link name="base_link" />
   <link name="base_footprint" />
