Commit message: Add MoveIt coordinate controller node

File: reseq_arm_mk2/config/simplified_arm_assembly.urdf (robot description, URDF)
Before this commit: robot reseq_arm_mk2, 7 links, 6 joints
Links:
- removed link arm_base_link
- removed link arm_diff_pitch_link
- removed link arm_diff_roll_link
- removed link arm_pitch_forearm_link
- removed link arm_pitch_wrist_link
- removed link arm_roll_forearm_link
- removed link arm_roll_wrist_link
- added link base_link
- added link mod1__base_link, mass 0.11481; collision mesh filename=package://reseq_arm_mk2/meshes/module_joint.STL; visual mesh filename=package://reseq_arm_mk2/meshes/module_joint.STL
- added link mod1__pitch_1_link, mass 0.28931; collision mesh filename=package://reseq_arm_mk2/meshes/pitch_1.STL; visual mesh filename=package://reseq_arm_mk2/meshes/pitch_1.STL
- added link mod1__pitch_3_link, mass 0.10409; collision mesh filename=package://reseq_arm_mk2/meshes/pitch_3.STL; visual mesh filename=package://reseq_arm_mk2/meshes/pitch_3.STL
- added link mod1__pitch_5_link, mass 0.056876; collision mesh filename=package://reseq_arm_mk2/meshes/pitch_5.STL; visual mesh filename=package://reseq_arm_mk2/meshes/pitch_5.STL
- added link mod1__roll_2_link, mass 0.11865; collision mesh filename=package://reseq_arm_mk2/meshes/roll_2.STL; visual mesh filename=package://reseq_arm_mk2/meshes/roll_2.STL
- added link mod1__roll_4_link, mass 0.096867; collision mesh filename=package://reseq_arm_mk2/meshes/roll_4.STL; visual mesh filename=package://reseq_arm_mk2/meshes/roll_4.STL
- added link mod1__roll_6_link, mass 0.54009; collision mesh filename=package://reseq_arm_mk2/meshes/roll_6.STL; visual mesh filename=package://reseq_arm_mk2/meshes/roll_6.STL
Joints:
- added joint base_to_module: type fixed, parent base_link, child mod1__base_link, origin xyz=0 0 0 rpy=0 0 0
- joint mod1__base_pitch_arm_joint: child arm_diff_pitch_link -> mod1__pitch_1_link; limit lower=0 upper=1.309 effort=6 velocity=2 -> lower=-3.14 upper=1.309 effort=6 velocity=2; origin xyz=0 0 0 rpy=1.5708 -1.309 0 -> xyz=0 0 0 rpy=1.5708 1.309 3.1416; parent arm_base_link -> mod1__base_link
- joint mod1__base_roll_arm_joint: child arm_diff_roll_link -> mod1__roll_2_link; limit lower=-3.14 upper=3.14 effort=6 velocity=2 -> lower=-6.28 upper=6.28 effort=6 velocity=2; origin xyz=0 0 0 rpy=1.5708 1.5708 0 -> xyz=0 0.16147 0 rpy=1.5708 1.5708 0; parent arm_diff_pitch_link -> mod1__pitch_1_link
- joint mod1__elbow_pitch_arm_joint: child arm_pitch_forearm_link -> mod1__pitch_3_link; origin xyz=0 0 -0.28857 rpy=3.1416 -1.5708 3.1416 -> xyz=0 0 -0.1271 rpy=3.1416 -1.5708 0; parent arm_diff_roll_link -> mod1__roll_2_link
- joint mod1__forearm_roll_arm_joint: child arm_roll_forearm_link -> mod1__roll_4_link; limit lower=-3.14 upper=3.14 effort=3 velocity=1 -> lower=-6.28 upper=6.28 effort=3 velocity=1; origin xyz=0.15351 0.074002 0 rpy=0.2618 -1.5708 3.1416 -> xyz=0.15351 0.074002 0 rpy=3.4034 -1.5708 0; parent arm_pitch_forearm_link -> mod1__pitch_3_link
- joint mod1__wrist_pitch_arm_joint: child arm_pitch_wrist_link -> mod1__pitch_5_link; limit lower=-0.46 upper=1.57 effort=3 velocity=1 -> lower=-1.57 upper=1.57 effort=3 velocity=1; origin xyz=0 0 0.05447 rpy=3.1416 -1.5708 3.1416 -> xyz=0 0 0.05447 rpy=3.1416 -1.5708 0; parent arm_roll_forearm_link -> mod1__roll_4_link
- joint mod1__wrist_roll_arm_joint: child arm_roll_wrist_link -> mod1__roll_6_link; limit lower=-3.14 upper=3.14 effort=3 velocity=1 -> lower=-6.28 upper=6.28 effort=3 velocity=1; origin xyz=0 0 0 rpy=0 1.5708 0 -> xyz=0.065961 0 0 rpy=0 1.5708 0; parent arm_pitch_wrist_link -> mod1__pitch_5_link

File: reseq_ros2/description/ros2_control.xacro (robot description, xacro)
@@ -64,4 +64,5 @@
             <plugin name="gz_ros2_control::GazeboSimROS2ControlPlugin" filename="libgz_ros2_control-system.so">
                 <parameters>$(arg controllers_config_file)</parameters>
+                <use_sim_time>$(arg sim_mode)</use_sim_time>
             </plugin>
         </gazebo>
