Commit message: feat(sensors-gz): Gazebo rgbd_camera and thermal_camera implementation

File: reseq_description/description/sensors/gazebo/cameras_holder.xacro (robot description, xacro)
@@ -2,10 +2,10 @@
 <robot>
     <!-- THIS FILE DEFINES THE END EFFECTOR CAMERA HOLDER -->
-    <joint name="ef_cameras_holder_joint" type="fixed">
+    <joint name="cameras_holder_joint" type="fixed">
         <origin xyz="0 -0.03 0.15" rpy="1.57 -1.57 0"/>
         <parent link="arm_roll_wrist_link"/>
-        <child link="ef_cameras_holder_link"/>
+        <child link="cameras_holder_link"/>
     </joint>
-    <link name="ef_cameras_holder_link">
+    <link name="cameras_holder_link">
         <visual name="cube">
             <origin xyz="0 0 0"/>
@@ -18,11 +18,11 @@
         </visual>
     </link>
-    <gazebo reference="ef_cameras_holder_link">
+    <gazebo reference="cameras_holder_link">
         <!--http://sdformat.org/spec?ver=1.12&elem=sensor-->
         <material>Gazebo/Red</material>
         <sensor name="rgbd_camera" type="rgbd_camera">
-            <pose> 0 0 0 0 0 0 0 </pose>
+            <pose relative_to="cameras_holder_link"> 0 0 0 0 0 0 </pose>
             <visualize>true</visualize>
-            <update_rate>10</update_rate>
+            <update_rate>30</update_rate>
             <always_on>true</always_on>
             <topic>rgbd_camera</topic>
@@ -45,8 +45,22 @@
                 </depth_camera>
             </camera>
-            <gz_frame_id>ef_cameras_holder_link</gz_frame_id>
-            <!-- <plugin name="depth_camera" filename="">
-                <frame_name>depth_camera_frame</frame_name>
-            </plugin> -->
+            <gz_frame_id>cameras_holder_link</gz_frame_id>
+        </sensor>
+        <!-- modeling themo camera Adafruit MLX90640 IR Thermal Camera Breakout - 55 Degree -->
+        <sensor name="thermal_camera" type="thermal_camera">
+            <always_on>true</always_on>
+            <update_rate>2</update_rate>
+            <visualize>true</visualize>
+            <topic>thermal_camera</topic>
+            <enable_metrics>true</enable_metrics>
+            <frame_id>cameras_holder_link</frame_id>
+            <pose relative_to="cameras_holder_link"></pose>
+            <camera>
+                <horizontal_fov>0.9599</horizontal_fov> <!-- 55 degrees -->
+                <image>
+                    <width>32</width>
+                    <height>24</height>
+                </image>
+            </camera>
         </sensor>
     </gazebo>
