Commit message: can interface parameter added

File: reseq_description/description/control/ros2_control.xacro (robot description, xacro)
@@ -10,5 +10,5 @@
             </xacro:unless>
             <param name="num_modules">${NumModules}</param>
-            <!-- TODO: vcan, and gazebo alternatives -->
+            <param name="can_interface">${CanInterface}</param>
         </hardware>
         <xacro:include filename="$(find reseq_description)/description/control/body_joints.xacro"/>

File: reseq_description/description/macros/reseq_parameters.xacro (robot description, xacro)
@@ -13,4 +13,5 @@
   <!-- chassis related -->
   <xacro:property name="NumModules" value="${config['num_modules']}"/>
+  <xacro:property name="CanInterface" value="${config['canbus']['channel']}"/>
   <xacro:property name="WheelBase" value="${config['xacro']['WheelBase']}"/>
   <xacro:property name="EquivalentWheelDiameter" value="${r_eq*2}"/>
