Commit message: feat(reseq_description): Add IMU sensor integration for chassis modules and update related macros

File: reseq_description/description/control/body_joints.xacro (robot description, xacro)
@@ -13,4 +13,21 @@
                 <xacro:control_joint_factory id="${module}" />
             </xacro:if>
+            <!-- IMU sensor hardware interfaces.
+                 Sim: GazeboSimSystem reads the Gazebo IMU sensor and exposes these state interfaces.
+                 Hardware: ReseqHardware reads CAN messages 0x92 (accel) and 0x93 (gyro)
+                 from the STEVAL-MKI178V2 / ISM330DLC board via PicoLowLevel firmware.
+                 imu_sensor_broadcaster reads these interfaces and publishes sensor_msgs/Imu. -->
+            <sensor name="imu${module}">
+                <state_interface name="orientation.x"/>
+                <state_interface name="orientation.y"/>
+                <state_interface name="orientation.z"/>
+                <state_interface name="orientation.w"/>
+                <state_interface name="angular_velocity.x"/>
+                <state_interface name="angular_velocity.y"/>
+                <state_interface name="angular_velocity.z"/>
+                <state_interface name="linear_acceleration.x"/>
+                <state_interface name="linear_acceleration.y"/>
+                <state_interface name="linear_acceleration.z"/>
+            </sensor>
             <xacro:loop module="${module + 1}" n_modules="${n_modules}" />
         </xacro:if>

File: reseq_description/description/macros/chassis.xacro (robot description, xacro)
@@ -5,5 +5,5 @@
     @param id: the id of the chassis (starting from 1)
   -->
-  <xacro:macro name="chassis" params="id">
+  <xacro:macro name="chassis" params="id physics_link">
     <link name="chassis${id}_link">
       <xacro:replicate_collision>
@@ -34,4 +34,6 @@
     <xacro:wheel_factory id="${id}" pos="back" side="left" />
     <xacro:wheel_factory id="${id}" pos="back" side="right" />
+    <!-- IMU (STEVAL-MKI178V2 / ISM330DLC) on each chassis module -->
+    <xacro:imu_sensor id="${id}" physics_link="${physics_link}" />
   </xacro:macro>
 </robot>

File: reseq_description/description/macros/reseq_body.xacro (robot description, xacro)
@@ -7,4 +7,5 @@
   <xacro:include filename="$(find reseq_description)/description/control/control_macros.xacro" />
   <xacro:include filename="$(find reseq_description)/description/sensors/lidar.xacro" />
+  <xacro:include filename="$(find reseq_description)/description/sensors/imu.xacro" />
   <link name="base_link" />
   <link name="base_footprint" />
@@ -24,5 +25,11 @@
     <xacro:if value="${module &lt; n_modules}">
       <!-- Create module and following joint -->
-      <xacro:chassis id="${module}"/>
+      <!-- Module 1 is fixed to base_link (merged). Modules 2+ live on joint_p_N_link (revolute, not merged). -->
+      <xacro:if value="${module == 1}">
+        <xacro:chassis id="${module}" physics_link="base_link"/>
+      </xacro:if>
+      <xacro:unless value="${module == 1}">
+        <xacro:chassis id="${module}" physics_link="joint_p_${module}_link"/>
+      </xacro:unless>
       <xacro:chassis_joint_factory id="${module + 1}"/>
       <xacro:loop module="${module + 1}" n_modules="${n_modules}"/>
@@ -30,5 +37,10 @@
     <xacro:if value="${module == n_modules}">
       <!-- Create last module -->
-      <xacro:chassis id="${module}"/>
+      <xacro:if value="${module == 1}">
+        <xacro:chassis id="${module}" physics_link="base_link"/>
+      </xacro:if>
+      <xacro:unless value="${module == 1}">
+        <xacro:chassis id="${module}" physics_link="joint_p_${module}_link"/>
+      </xacro:unless>
     </xacro:if>
   </xacro:macro>

File: reseq_description/description/macros/reseq_parameters.xacro (robot description, xacro)
@@ -44,3 +44,6 @@
     <color rgba="0.5 0.5 0.5 1" />
   </material>
+  <material name="IMUColor">
+    <color rgba="0.1 0.1 0.1 1" />
+  </material>
 </robot>
