Commit message: fix: Update reseq controllers and URDF for more realistic traction steering

File: reseq_description/description/control/control_macros.xacro (robot description, xacro)
@@ -27,8 +27,10 @@
             <state_interface name="velocity" />
         </joint>
-        <joint name="mod${id}__yaw_joint">
-            <command_interface name="position" />
-            <state_interface name="position" />
-        </joint>
+        <xacro:unless value="$(arg passive_yaw)">
+            <joint name="mod${id}__yaw_joint">
+                <command_interface name="position" />
+                <state_interface name="position" />
+            </joint>
+        </xacro:unless>
     </xacro:macro>
 </robot>

File: reseq_description/description/macros/chassis.xacro (robot description, xacro)
@@ -23,5 +23,5 @@
         y="${ModuleWidth-2*TrackWidth-2*toll}"
         z="${EquivalentWheelDiameter-2*ChassisTopAndBottomClearance}">
-        <origin xyz="${EquivalentWheelDiameter/12+(toll+JointDiameter/2)/2} 0 0" rpy="0 0 0" />
+        <origin xyz="-${EquivalentWheelDiameter/12+(toll+JointDiameter/2)/2} 0 0" rpy="0 0 0" />
       </xacro:inertial_box>
     </link>
@@ -30,4 +30,11 @@
     </gazebo>
     <!-- Wheels -->
+    <!-- diff_drive_controller integrates the midpoint of its driven axle. -->
+    <link name="rear_axle${id}_link" />
+    <joint name="rear_axle${id}_joint" type="fixed">
+      <parent link="chassis${id}_link" />
+      <child link="rear_axle${id}_link" />
+      <origin xyz="${-WheelBase/2} 0 0" rpy="0 0 0" />
+    </joint>
     <xacro:wheel_factory id="${id}" pos="front" side="left" />
     <xacro:wheel_factory id="${id}" pos="front" side="right" />

File: reseq_description/description/macros/joint.xacro (robot description, xacro)
@@ -46,4 +46,7 @@
       <axis xyz="0 0 1" />
       <dynamics damping="0.5" friction="0.1" />
+      <gazebo>
+        <friction>0.1</friction>
+      </gazebo>
     </joint>
     <link name="joint_y_${id}_link">

File: reseq_description/description/macros/wheel.xacro (robot description, xacro)
@@ -52,6 +52,10 @@
         </xacro:inertial_cylinder_y>
         </link>
+        <!-- Gazebo friction parameters for skid-steer drive. -->
         <gazebo reference="${side}_${pos}_wheel_${id}_link">
             <material>Gazebo/Black</material>
+            <mu1>1.0</mu1>
+            <mu2>0.3</mu2>
+            <fdir1>1 0 0</fdir1>
         </gazebo>
     </xacro:macro>

File: reseq_description/description/mk1/reseq.urdf.xacro (robot description, xacro)
@@ -3,4 +3,5 @@
   <xacro:arg name="use_ros2_control" default="true"/>
   <xacro:arg name="sim_mode" default="false"/>
+  <xacro:arg name="passive_yaw" default="false"/>
   <xacro:include filename="$(find reseq_description)/description/macros/reseq_parameters.xacro" />
   <xacro:include filename="$(find reseq_description)/description/macros/materials.xacro" />

File: reseq_description/description/mk2/reseq.urdf.xacro (robot description, xacro)
@@ -3,4 +3,5 @@
   <xacro:arg name="use_ros2_control" default="true"/>
   <xacro:arg name="sim_mode" default="false"/>
+  <xacro:arg name="passive_yaw" default="false"/>
   <xacro:include filename="$(find reseq_description)/description/macros/reseq_parameters.xacro" />
   <xacro:include filename="$(find reseq_description)/description/macros/materials.xacro" />

Commit message: feat: Introduce passive_yaw argument for yaw joint control in launch files and macros

File: reseq_description/description/control/control_macros.xacro (robot description, xacro)
@@ -27,10 +27,10 @@
             <state_interface name="velocity" />
         </joint>
-        <xacro:unless value="$(arg passive_yaw)">
-            <joint name="mod${id}__yaw_joint">
+        <joint name="mod${id}__yaw_joint">
+            <xacro:unless value="$(arg passive_yaw)">
                 <command_interface name="position" />
-                <state_interface name="position" />
-            </joint>
-        </xacro:unless>
+            </xacro:unless>
+            <state_interface name="position" />
+        </joint>
     </xacro:macro>
 </robot>

File: reseq_description/description/macros/joint.xacro (robot description, xacro)
@@ -45,8 +45,20 @@
       <origin xyz="-${JointB} 0 0" rpy="0 0 0" />
       <axis xyz="0 0 1" />
-      <dynamics damping="0.5" friction="0.1" />
-      <gazebo>
-        <friction>0.1</friction>
-      </gazebo>
+      <xacro:if value="$(arg passive_yaw)">
+        <dynamics damping="0.05" friction="0.01" />
+      </xacro:if>
+      <xacro:unless value="$(arg passive_yaw)">
+        <dynamics damping="0.5" friction="0.1" />
+      </xacro:unless>
+      <xacro:if value="$(arg passive_yaw)">
+        <gazebo>
+          <friction>0.01</friction>
+        </gazebo>
+      </xacro:if>
+      <xacro:unless value="$(arg passive_yaw)">
+        <gazebo>
+          <friction>0.1</friction>
+        </gazebo>
+      </xacro:unless>
     </joint>
     <link name="joint_y_${id}_link">
