Commit message: beak registration in control_joints.xacro

File: reseq_description/description/mk2/arm/control_joints.xacro (robot description, xacro)
@@ -49,3 +49,7 @@
         </xacro:if>
     </joint>
+    <joint name="mod1__beak">
+        <command_interface name="position" />
+        <state_interface name="position" />
+    </joint>
 </robot>
