Commit message: feat(sim): command the beak in simulation, also from BBLACK
- mod1__beak position interface and beak_controller (sim only)
- beak_controller spawned after the arm velocity controller
- scaler publishes the beak angle on /beak_controller/commands when BBLACK is
  pressed; the direct CAN command on the real robot is unchanged

File: reseq_description/description/mk2/arm/control_joints.xacro (robot description, xacro)
@@ -80,3 +80,11 @@
         </xacro:if>
     </joint>
+    <xacro:if value="$(arg sim_mode)">
+        <joint name="mod1__beak">
+            <command_interface name="position" />
+            <state_interface name="position">
+                <param name="initial_value">0.0</param>
+            </state_interface>
+        </joint>
+    </xacro:if>
 </robot>
