Commit message: fix(joint): Update joint limits and dynamics for dynamixel

File: reseq_description/description/macros/joint.xacro (robot description, xacro)
@@ -13,7 +13,8 @@
       <child link="joint_r_${id}_link" />
       <!-- Effort in Nm -->
-      <limit effort="2.0" lower="${-roll}" upper="${roll}" velocity="0.5" />
+      <limit effort="7.0" lower="${-roll}" upper="${roll}" velocity="3.14" />
       <origin xyz="-${WheelBase/2} 0 0" rpy="0 0 0" />
       <axis xyz="1 0 0" />
+      <dynamics damping="0.5" friction="0.1" />
     </joint>
     <link name="joint_r_${id}_link">
@@ -41,7 +42,8 @@
       <child link="joint_y_${id}_link" />
       <!-- Effort in Nm -->
-      <limit effort="20.0" lower="${-yaw}" upper="${yaw}" velocity="0.5" />
+      <limit effort="7.0" lower="${-yaw}" upper="${yaw}" velocity="3.14" />
       <origin xyz="-${JointB} 0 0" rpy="0 0 0" />
       <axis xyz="0 0 1" />
+      <dynamics damping="0.5" friction="0.1" />
     </joint>
     <link name="joint_y_${id}_link">
@@ -78,7 +80,8 @@
       <child link="joint_p_${id}_link" />
       <!-- Effort in Nm -->
-      <limit effort="20.0" lower="${-pitch}" upper="${pitch}" velocity="0.5" />
+      <limit effort="7.0" lower="${-pitch}" upper="${pitch}" velocity="3.14" />
       <origin xyz="${-JointA} 0 0" rpy="0 0 0" />
       <axis xyz="0 1 0" />
+      <dynamics damping="0.5" friction="0.1" />
     </joint>
     <link name="joint_p_${id}_link">
