Commit message: feat: Add TOF obstacle detection and joint lift controller integration

File: reseq_description/description/macros/chassis.xacro (robot description, xacro)
@@ -34,6 +34,67 @@
     <xacro:wheel_factory id="${id}" pos="back" side="left" />
     <xacro:wheel_factory id="${id}" pos="back" side="right" />
+    <!-- Small front caster wheels on chassis1 only (half diameter, floating) -->
+    <xacro:if value="${id == 1}">
+      <!-- Small front-left caster wheel (fixed to chassis) -->
+      <joint name="mod${id}__small_front_left_wheel" type="fixed">
+        <parent link="chassis${id}_link"/>
+        <child link="small_front_left_wheel_${id}_link"/>
+        <origin xyz="${WheelBase/2 + 0.08} ${(ModuleWidth/2-TrackWidth/2)/2 + 0.02} ${EquivalentWheelDiameter/4}" rpy="0 0 0"/>
+      </joint>
+      <link name="small_front_left_wheel_${id}_link">
+        <visual>
+          <origin xyz="0 0 0" rpy="${pi/2} 0 0"/>
+          <geometry>
+            <cylinder radius="${EquivalentWheelDiameter/4}" length="${TrackWidth/2}"/>
+          </geometry>
+          <material name="WheelColor"/>
+        </visual>
+        <collision>
+          <origin xyz="0 0 0" rpy="${pi/2} 0 0"/>
+          <geometry>
+            <cylinder radius="${EquivalentWheelDiameter/4}" length="${TrackWidth/2}"/>
+          </geometry>
+        </collision>
+        <xacro:inertial_cylinder_y mass="${WheelMass/4}" length="${TrackWidth/2}" radius="${EquivalentWheelDiameter/4}">
+          <origin xyz="0 0 0" rpy="-${pi/2} 0 0"/>
+        </xacro:inertial_cylinder_y>
+      </link>
+      <gazebo reference="small_front_left_wheel_${id}_link">
+        <material>Gazebo/Black</material>
+      </gazebo>
+      <!-- Small front-right caster wheel (fixed to chassis) -->
+      <joint name="mod${id}__small_front_right_wheel" type="fixed">
+        <parent link="chassis${id}_link"/>
+        <child link="small_front_right_wheel_${id}_link"/>
+        <origin xyz="${WheelBase/2 + 0.08} ${-(ModuleWidth/2-TrackWidth/2)/2 - 0.02} ${EquivalentWheelDiameter/4}" rpy="0 0 0"/>
+      </joint>
+      <link name="small_front_right_wheel_${id}_link">
+        <visual>
+          <origin xyz="0 0 0" rpy="${pi/2} 0 0"/>
+          <geometry>
+            <cylinder radius="${EquivalentWheelDiameter/4}" length="${TrackWidth/2}"/>
+          </geometry>
+          <material name="WheelColor"/>
+        </visual>
+        <collision>
+          <origin xyz="0 0 0" rpy="${pi/2} 0 0"/>
+          <geometry>
+            <cylinder radius="${EquivalentWheelDiameter/4}" length="${TrackWidth/2}"/>
+          </geometry>
+        </collision>
+        <xacro:inertial_cylinder_y mass="${WheelMass/4}" length="${TrackWidth/2}" radius="${EquivalentWheelDiameter/4}">
+          <origin xyz="0 0 0" rpy="-${pi/2} 0 0"/>
+        </xacro:inertial_cylinder_y>
+      </link>
+      <gazebo reference="small_front_right_wheel_${id}_link">
+        <material>Gazebo/Black</material>
+      </gazebo>
+    </xacro:if>
     <!-- IMU (STEVAL-MKI178V2 / ISM330DLC) on each chassis module -->
     <xacro:imu_sensor id="${id}" physics_link="${physics_link}" />
+    <!-- TOF sensor array on the first module only (front-facing obstacle detection) -->
+    <xacro:if value="${id == 1}">
+      <xacro:tof_sensor_array parent_link="chassis${id}_link" prefix="tof"/>
+    </xacro:if>
   </xacro:macro>
 </robot>

File: reseq_description/description/macros/reseq_body.xacro (robot description, xacro)
@@ -9,4 +9,5 @@
   <xacro:include filename="$(find reseq_description)/description/sensors/imu.xacro" />
   <xacro:include filename="$(find reseq_description)/description/sensors/encoder.xacro" />
+  <xacro:include filename="$(find reseq_description)/description/sensors/tof_sensor.xacro" />
   <link name="base_link" />
   <link name="base_footprint" />
