Commit message: fix(description): correct inertia orientation of wheels, casters and roll joints
inertial_cylinder_y/_x already return the tensor aligned with the cylinder
axis; the extra rpy rotation moved the spin axis inertia to the vertical axis
(wheel spin inertia off by 38%, roll joint by 83%).

File: reseq_description/description/macros/chassis.xacro (robot description, xacro)
@@ -64,5 +64,5 @@
         </collision>
         <xacro:inertial_cylinder_y mass="${WheelMass/4}" length="${TrackWidth/2}" radius="${EquivalentWheelDiameter/4}">
-          <origin xyz="0 0 0" rpy="-${pi/2} 0 0"/>
+          <origin xyz="0 0 0" rpy="0 0 0"/>
         </xacro:inertial_cylinder_y>
       </link>
@@ -91,5 +91,5 @@
         </collision>
         <xacro:inertial_cylinder_y mass="${WheelMass/4}" length="${TrackWidth/2}" radius="${EquivalentWheelDiameter/4}">
-          <origin xyz="0 0 0" rpy="-${pi/2} 0 0"/>
+          <origin xyz="0 0 0" rpy="0 0 0"/>
         </xacro:inertial_cylinder_y>
       </link>

File: reseq_description/description/macros/joint.xacro (robot description, xacro)
@@ -31,5 +31,5 @@
         length = "${JointB}"
         radius = "${JointWidth/2}">
-        <origin xyz="-${JointB/2} 0 0" rpy="0 ${pi/2} 0" />
+        <origin xyz="-${JointB/2} 0 0" rpy="0 0 0" />
       </xacro:inertial_cylinder_x>
     </link>

File: reseq_description/description/macros/wheel.xacro (robot description, xacro)
@@ -49,5 +49,5 @@
         <xacro:inertial_cylinder_y mass="${WheelMass}" length="${TrackWidth}"
             radius="${EquivalentWheelDiameter/2}">
-            <origin xyz="0 0 0" rpy="-${pi/2} 0 0" />
+            <origin xyz="0 0 0" rpy="0 0 0" />
         </xacro:inertial_cylinder_y>
         </link>
