Commit message: fix: Correct side_sign logic in wheel.xacro and remove software compensation of angular_sign in scaler.py

File: reseq_description/description/macros/wheel.xacro (robot description, xacro)
@@ -12,7 +12,7 @@
             <xacro:property name="pos_sign" value="-1" />
         </xacro:if>
-        <xacro:property name="side_sign" value="1" />
+        <xacro:property name="side_sign" value="-1" />
         <xacro:if value="${side == 'right'}">
-            <xacro:property name="side_sign" value="-1" />
+            <xacro:property name="side_sign" value="1" />
         </xacro:if>
         <xacro:if value="${pos == 'back'}">
