Commit message: robot config file path fix

File: reseq_arm_mk2/urdf/arm.urdf.xacro (robot description, xacro)
@@ -10,5 +10,8 @@
     <xacro:arg name="sim_mode" default="false" />
     <xacro:arg name="version" default="mk2" />
+    <xacro:arg name="config_path" default="$(find reseq_description)/config/mk2/reseq_mk2_can.yaml" />
     <xacro:arg name="controllers_config_file" default="$(find reseq_description)/config/reseq_controllers.yaml" />
+    <xacro:property name="config_path_prop" value="${xacro.load_yaml(config_path)}" />
+    <xacro:property name="CanInterface" value="${config_path_prop['canbus']['channel']}" />
     <xacro:property name="NumModules" value="0" />
     <xacro:include filename="$(find reseq_description)/description/control/ros2_control.xacro" />

Commit message: xacro file config path fix

File: reseq_arm_mk2/urdf/arm.urdf.xacro (robot description, xacro)
@@ -12,6 +12,7 @@
     <xacro:arg name="config_path" default="$(find reseq_description)/config/mk2/reseq_mk2_can.yaml" />
     <xacro:arg name="controllers_config_file" default="$(find reseq_description)/config/reseq_controllers.yaml" />
-    <xacro:property name="config_path_prop" value="${xacro.load_yaml(config_path)}" />
-    <xacro:property name="CanInterface" value="${config_path_prop['canbus']['channel']}" />
+    <xacro:property name="config_path_prop" value="$(arg config_path)" />
+    <xacro:property name="config" value="${xacro.load_yaml(config_path_prop)}" />
+    <xacro:property name="CanInterface" value="${config['canbus']['channel']}" />
     <xacro:property name="NumModules" value="0" />
     <xacro:include filename="$(find reseq_description)/description/control/ros2_control.xacro" />

Commit message: Fix arm control and sim bringup

File: reseq_arm_mk2/urdf/arm.urdf.xacro (robot description, xacro)
@@ -2,14 +2,15 @@
 <robot
     name="reseq_arm_mk2" xmlns:xacro="http://www.ros.org/wiki/xacro">
+    <xacro:arg name="sim_mode" default="false" />
+    <xacro:arg name="version" default="mk2" />
+    <xacro:arg name="config_path" default="$(find reseq_description)/config/mk2/reseq_mk2_can.yaml" />
+    <xacro:arg name="controllers_config_file" default="$(find reseq_description)/config/reseq_controllers.yaml" />
+    <xacro:arg name="base_z" default="0.0" />
     <link name="world" />
     <joint name="world_to_base_joint" type="fixed">
         <parent link="world"/>
         <child link="arm_base_link"/>
-        <origin xyz="0 0 0" rpy="0 0 0"/>
+        <origin xyz="0 0 $(arg base_z)" rpy="0 0 0"/>
     </joint>
-    <xacro:arg name="sim_mode" default="false" />
-    <xacro:arg name="version" default="mk2" />
-    <xacro:arg name="config_path" default="$(find reseq_description)/config/mk2/reseq_mk2_can.yaml" />
-    <xacro:arg name="controllers_config_file" default="$(find reseq_description)/config/reseq_controllers.yaml" />
     <xacro:property name="config_path_prop" value="$(arg config_path)" />
     <xacro:property name="config" value="${xacro.load_yaml(config_path_prop)}" />

File: reseq_description/description/control/ros2_control.xacro (robot description, xacro)
@@ -19,4 +19,6 @@
             <plugin name="gz_ros2_control::GazeboSimROS2ControlPlugin" filename="libgz_ros2_control-system.so">
                 <parameters>$(find reseq_description)/config/temp/reseq_controllers.yaml</parameters>
+                <hold_joints>true</hold_joints>
+                <position_proportional_gain>0.1</position_proportional_gain>
             </plugin>
         </gazebo>

File: reseq_description/description/mk2/arm/control_joints.xacro (robot description, xacro)
@@ -2,49 +2,55 @@
 <robot xmlns:xacro="http://www.ros.org/wiki/xacro">
     <joint name="mod1__base_pitch_arm_joint">
-        <xacro:if value="$(arg sim_mode)" >
-            <command_interface name="position" />
-        </xacro:if>
         <command_interface name="velocity" />
-        <state_interface name="position" />
+        <state_interface name="position">
+            <xacro:if value="$(arg sim_mode)">
+                <param name="initial_value">0.0</param>
+            </xacro:if>
+        </state_interface>
         <state_interface name="velocity" />
     </joint>
     <joint name="mod1__base_roll_arm_joint">
-        <xacro:if value="$(arg sim_mode)" >
-            <command_interface name="position" />
-        </xacro:if>
         <command_interface name="velocity" />
-        <state_interface name="position" />
+        <state_interface name="position">
+            <xacro:if value="$(arg sim_mode)">
+                <param name="initial_value">0.0</param>
+            </xacro:if>
+        </state_interface>
         <state_interface name="velocity" />
     </joint>
     <joint name="mod1__elbow_pitch_arm_joint">
-        <xacro:if value="$(arg sim_mode)" >
-            <command_interface name="position" />
-        </xacro:if>
         <command_interface name="velocity" />
-        <state_interface name="position" />
+        <state_interface name="position">
+            <xacro:if value="$(arg sim_mode)">
+                <param name="initial_value">0.0</param>
+            </xacro:if>
+        </state_interface>
         <state_interface name="velocity" />
     </joint>
     <joint name="mod1__forearm_roll_arm_joint">
-        <xacro:if value="$(arg sim_mode)" >
-            <command_interface name="position" />
-        </xacro:if>
         <command_interface name="velocity" />
-        <state_interface name="position" />
+        <state_interface name="position">
+            <xacro:if value="$(arg sim_mode)">
+                <param name="initial_value">0.0</param>
+            </xacro:if>
+        </state_interface>
         <state_interface name="velocity" />
     </joint>
     <joint name="mod1__wrist_pitch_arm_joint">
-        <xacro:if value="$(arg sim_mode)" >
-            <command_interface name="position" />
-        </xacro:if>
         <command_interface name="velocity" />
-        <state_interface name="position" />
+        <state_interface name="position">
+            <xacro:if value="$(arg sim_mode)">
+                <param name="initial_value">0.0</param>
+            </xacro:if>
+        </state_interface>
         <state_interface name="velocity" />
     </joint>
     <joint name="mod1__wrist_roll_arm_joint">
-        <xacro:if value="$(arg sim_mode)" >
-            <command_interface name="position" />
-        </xacro:if>
         <command_interface name="velocity" />
-        <state_interface name="position" />
+        <state_interface name="position">
+            <xacro:if value="$(arg sim_mode)">
+                <param name="initial_value">0.0</param>
+            </xacro:if>
+        </state_interface>
         <state_interface name="velocity" />
     </joint>
