Commit message: feat(mk2-arm): Basic gz ros2-control

File: reseq_arm_mk2/urdf/reseq_arm_mk2.xacro (robot description, xacro)
@@ -1,7 +1,7 @@
 <?xml version="1.0" encoding="utf-8"?>
-<!-- Automatically generated by SOLIDWORKS URDF Export Plugin -->
-<!-- Do not modify manually-->
 <robot
-  name="reseq_arm_mk2">
+  name="reseq_arm_mk2" xmlns:xacro="http://www.ros.org/wiki/xacro">
+  <xacro:property name="NumModules" value="0" />
+  <xacro:include filename="$(find reseq_ros2)/description/ros2_control.xacro" />
   <link
     name="arm_base_link">

File: reseq_ros2/description/ros2_control.xacro (robot description, xacro)
@@ -29,18 +29,33 @@
         <xacro:loop module="1" n_modules="${NumModules}" />
         <!-- ARM CONTROLLER INTERFACES -->
-        <joint name="arm_pitch_1_joint">
+        <joint name="mod1__base_pitch_arm_joint">
             <command_interface name="position" />
             <state_interface name="position" />
             <state_interface name="velocity"/>
         </joint>
-        <joint name="arm_head_pitch_1_joint">
+        <joint name="mod1__base_roll_arm_joint">
             <command_interface name="position" />
             <state_interface name="position" />
             <state_interface name="velocity"/>
         </joint>
-        <joint name="arm_head_roll_1_joint">
+        <joint name="mod1__elbow_pitch_arm_joint">
             <command_interface name="position" />
             <state_interface name="position" />
-            <state_interface name="velocity" />
+            <state_interface name="velocity"/>
+        </joint>
+        <joint name="mod1__forearm_roll_arm_joint">
+            <command_interface name="position" />
+            <state_interface name="position" />
+            <state_interface name="velocity"/>
+        </joint>
+        <joint name="mod1__wrist_pitch_arm_joint">
+            <command_interface name="position" />
+            <state_interface name="position" />
+            <state_interface name="velocity"/>
+        </joint>
+        <joint name="mod1__wrist_roll_arm_joint">
+            <command_interface name="position" />
+            <state_interface name="position" />
+            <state_interface name="velocity"/>
         </joint>
     </ros2_control>
@@ -48,5 +63,5 @@
         <gazebo>
             <plugin name="gz_ros2_control::GazeboSimROS2ControlPlugin" filename="libgz_ros2_control-system.so">
-                <parameters>$(find reseq_ros2)/config/temp/reseq_controllers.yaml</parameters>
+                <parameters>$(find reseq_ros2)/config/reseq_controllers.yaml</parameters>
             </plugin>
         </gazebo>

Commit message: fix: update the parameters in order to fix the remote controller.

File: reseq_arm_mk2/urdf/reseq_arm_mk2.xacro (robot description, xacro)
@@ -1,5 +1,8 @@
 <?xml version="1.0" encoding="utf-8"?>
+<!-- This URDF was automatically created by SolidWorks to URDF Exporter! Originally created by Stephen Brawner (brawner@gmail.com)
+     Commit Version: 1.6.0-4-g7f85cfe  Build Version: 1.6.7995.38578
+     For more information, please see http://wiki.ros.org/sw_urdf_exporter -->
 <robot
-  name="reseq_arm_mk2" xmlns:xacro="http://www.ros.org/wiki/xacro">
+  name="urdf_export_4">
   <link
     name="arm_base_link">
@@ -24,19 +27,19 @@
       <geometry>
         <mesh
-          filename="package://reseq_arm_mk2/meshes/arm_base_link.STL" />
-      </geometry>
-      <material
-        name="">
-        <color
-          rgba="0.75294 0.75294 0.75294 1" />
-      </material>
-    </visual>
-    <collision>
-      <origin
-        xyz="0 0 0"
-        rpy="0 0 0" />
-      <geometry>
-        <mesh
-          filename="package://reseq_arm_mk2/meshes/arm_base_link.STL" />
+          filename="package://urdf_export_4/meshes/arm_base_link.STL" />
+      </geometry>
+      <material
+        name="">
+        <color
+          rgba="0.75294 0.75294 0.75294 1" />
+      </material>
+    </visual>
+    <collision>
+      <origin
+        xyz="0 0 0"
+        rpy="0 0 0" />
+      <geometry>
+        <mesh
+          filename="package://urdf_export_4/meshes/arm_base_link.STL" />
       </geometry>
     </collision>
@@ -46,14 +49,14 @@
     <inertial>
       <origin
-        xyz="-1.3878E-17 0.00059334 1.7347E-18"
+        xyz="-0.00059334 -1.3878E-17 3.4694E-18"
         rpy="0 0 0" />
       <mass
         value="0.28931" />
       <inertia
-        ixx="0.0002425"
-        ixy="-1.6941E-20"
-        ixz="-1.5531E-20"
-        iyy="0.00023577"
-        iyz="8.3058E-21"
+        ixx="0.00023577"
+        ixy="1.6941E-20"
+        ixz="-8.3058E-21"
+        iyy="0.0002425"
+        iyz="-1.5531E-20"
         izz="0.00025759" />
     </inertial>
@@ -64,19 +67,19 @@
       <geometry>
         <mesh
-          filename="package://reseq_arm_mk2/meshes/arm_diff_pitch_link.STL" />
-      </geometry>
-      <material
-        name="">
-        <color
-          rgba="0.75294 0.75294 0.75294 1" />
-      </material>
-    </visual>
-    <collision>
-      <origin
-        xyz="0 0 0"
-        rpy="0 0 0" />
-      <geometry>
-        <mesh
-          filename="package://reseq_arm_mk2/meshes/arm_diff_pitch_link.STL" />
+          filename="package://urdf_export_4/meshes/arm_diff_pitch_link.STL" />
+      </geometry>
+      <material
+        name="">
+        <color
+          rgba="0.75294 0.75294 0.75294 1" />
+      </material>
+    </visual>
+    <collision>
+      <origin
+        xyz="0 0 0"
+        rpy="0 0 0" />
+      <geometry>
+        <mesh
+          filename="package://urdf_export_4/meshes/arm_diff_pitch_link.STL" />
       </geometry>
     </collision>
@@ -87,5 +90,5 @@
     <origin
       xyz="0 0 0"
-      rpy="1.5708 -1.309 0" />
+      rpy="1.5708 0.2 0" />
     <parent
       link="arm_base_link" />
@@ -95,6 +98,6 @@
       xyz="0 0 -1" />
     <limit
-      lower="-1.05"
-      upper="1.309"
+      lower="-0.1"
+      upper="2.8"
       effort="6"
       velocity="2" />
@@ -104,37 +107,37 @@
     <inertial>
       <origin
-        xyz="1.1115E-08 7.62E-08 -0.14664"
+        xyz="-0.14664 7.62E-08 -1.1115E-08"
         rpy="0 0 0" />
       <mass
         value="0.11865" />
       <inertia
-        ixx="0.00051345"
-        ixy="-2.7475E-10"
-        ixz="-9.7641E-11"
+        ixx="1.0228E-05"
+        ixy="2.2625E-10"
+        ixz="9.7641E-11"
         iyy="0.00051383"
-        iyz="2.2625E-10"
-        izz="1.0228E-05" />
-    </inertial>
-    <visual>
-      <origin
-        xyz="0 0 0"
-        rpy="0 0 0" />
-      <geometry>
-        <mesh
-          filename="package://reseq_arm_mk2/meshes/arm_diff_roll_link.STL" />
-      </geometry>
-      <material
-        name="">
-        <color
-          rgba="0.75294 0.75294 0.75294 1" />
-      </material>
-    </visual>
-    <collision>
-      <origin
-        xyz="0 0 0"
-        rpy="0 0 0" />
-      <geometry>
-        <mesh
-          filename="package://reseq_arm_mk2/meshes/arm_diff_roll_link.STL" />
+        iyz="2.7475E-10"
+        izz="0.00051345" />
+    </inertial>
+    <visual>
+      <origin
+        xyz="0 0 0"
+        rpy="0 0 0" />
+      <geometry>
+        <mesh
+          filename="package://urdf_export_4/meshes/arm_diff_roll_link.STL" />
+      </geometry>
+      <material
+        name="">
+        <color
+          rgba="0.75294 0.75294 0.75294 1" />
+      </material>
+    </visual>
+    <collision>
+      <origin
+        xyz="0 0 0"
+        rpy="0 0 0" />
+      <geometry>
+        <mesh
+          filename="package://urdf_export_4/meshes/arm_diff_roll_link.STL" />
       </geometry>
     </collision>
@@ -145,5 +148,5 @@
     <origin
       xyz="0 0 0"
-      rpy="1.5708 1.5708 0" />
+      rpy="0 0 0" />
     <parent
       link="arm_diff_pitch_link" />
@@ -151,5 +154,5 @@
       link="arm_diff_roll_link" />
     <axis
-      xyz="0 0 1" />
+      xyz="1 0 0" />
     <limit
       lower="-3.14"
@@ -169,7 +172,7 @@
         ixx="4.6765E-05"
         ixy="-9.086E-05"
-        ixz="1.3681E-20"
+        ixz="1.3572E-20"
         iyy="0.00027451"
-        iyz="3.2975E-21"
+        iyz="3.2775E-21"
         izz="0.00031255" />
     </inertial>
@@ -180,19 +183,19 @@
       <geometry>
         <mesh
-          filename="package://reseq_arm_mk2/meshes/arm_pitch_forearm_link.STL" />
-      </geometry>
-      <material
-        name="">
-        <color
-          rgba="0.75294 0.75294 0.75294 1" />
-      </material>
-    </visual>
-    <collision>
-      <origin
-        xyz="0 0 0"
-        rpy="0 0 0" />
-      <geometry>
-        <mesh
-          filename="package://reseq_arm_mk2/meshes/arm_pitch_forearm_link.STL" />
+          filename="package://urdf_export_4/meshes/arm_pitch_forearm_link.STL" />
+      </geometry>
+      <material
+        name="">
+        <color
+          rgba="0.75294 0.75294 0.75294 1" />
+      </material>
+    </visual>
+    <collision>
+      <origin
+        xyz="0 0 0"
+        rpy="0 0 0" />
+      <geometry>
+        <mesh
+          filename="package://urdf_export_4/meshes/arm_pitch_forearm_link.STL" />
       </geometry>
     </collision>
@@ -202,6 +205,6 @@
     type="revolute">
     <origin
-      xyz="0 0 -0.28857"
-      rpy="3.1416 -1.5708 3.1416" />
+      xyz="-0.28857 0 0"
+      rpy="0 0 0.2" />
     <parent
       link="arm_diff_roll_link" />
@@ -211,5 +214,5 @@
       xyz="0 0 1" />
     <limit
-      lower="-1.05"
+      lower="-0.1"
       upper="2.88"
       effort="6"
@@ -226,6 +229,6 @@
       <inertia
         ixx="5.2065E-05"
-        ixy="1.6912E-22"
-        ixz="-6.5731E-21"
+        ixy="1.7168E-22"
+        ixz="-6.5851E-21"
         iyy="4.9885E-05"
         iyz="2.3291E-07"
@@ -238,19 +241,19 @@
       <geometry>
         <mesh
-          filename="package://reseq_arm_mk2/meshes/arm_roll_forearm_link.STL" />
-      </geometry>
-      <material
-        name="">
-        <color
-          rgba="0.75294 0.75294 0.75294 1" />
-      </material>
-    </visual>
-    <collision>
-      <origin
-        xyz="0 0 0"
-        rpy="0 0 0" />
-      <geometry>
-        <mesh
-          filename="package://reseq_arm_mk2/meshes/arm_roll_forearm_link.STL" />
+          filename="package://urdf_export_4/meshes/arm_roll_forearm_link.STL" />
+      </geometry>
+      <material
+        name="">
+        <color
+          rgba="0.75294 0.75294 0.75294 1" />
+      </material>
+    </visual>
+    <collision>
+      <origin
+        xyz="0 0 0"
+        rpy="0 0 0" />
+      <geometry>
+        <mesh
+          filename="package://urdf_export_4/meshes/arm_roll_forearm_link.STL" />
       </geometry>
     </collision>
@@ -261,5 +264,5 @@
     <origin
       xyz="0.15351 0.074002 0"
-      rpy="0.2618 -1.5708 3.1416" />
+      rpy="0.2618 -1.5708 3.14" />
     <parent
       link="arm_pitch_forearm_link" />
@@ -278,37 +281,37 @@
     <inertial>
       <origin
-        xyz="0.045311 1.3878E-17 -3.296E-17"
+        xyz="5.3776E-17 2.7756E-17 0.045311"
         rpy="0 0 0" />
       <mass
         value="0.056876" />
       <inertia
-        ixx="1.5222E-05"
-        ixy="2.5626E-21"
-        ixz="3.1474E-21"
+        ixx="1.6114E-05"
+        ixy="3.0569E-22"
+        ixz="-3.5109E-21"
         iyy="2.2881E-05"
-        iyz="-1.4326E-21"
-        izz="1.6114E-05" />
-    </inertial>
-    <visual>
-      <origin
-        xyz="0 0 0"
-        rpy="0 0 0" />
-      <geometry>
-        <mesh
-          filename="package://reseq_arm_mk2/meshes/arm_pitch_wrist_link.STL" />
-      </geometry>
-      <material
-        name="">
-        <color
-          rgba="0.75294 0.75294 0.75294 1" />
-      </material>
-    </visual>
-    <collision>
-      <origin
-        xyz="0 0 0"
-        rpy="0 0 0" />
-      <geometry>
-        <mesh
-          filename="package://reseq_arm_mk2/meshes/arm_pitch_wrist_link.STL" />
+        iyz="1.0674E-21"
+        izz="1.5222E-05" />
+    </inertial>
+    <visual>
+      <origin
+        xyz="0 0 0"
+        rpy="0 0 0" />
+      <geometry>
+        <mesh
+          filename="package://urdf_export_4/meshes/arm_pitch_wrist_link.STL" />
+      </geometry>
+      <material
+        name="">
+        <color
+          rgba="0.75294 0.75294 0.75294 1" />
+      </material>
+    </visual>
+    <collision>
+      <origin
+        xyz="0 0 0"
+        rpy="0 0 0" />
+      <geometry>
+        <mesh
+          filename="package://urdf_export_4/meshes/arm_pitch_wrist_link.STL" />
       </geometry>
     </collision>
@@ -319,5 +322,5 @@
     <origin
       xyz="0 0 0.05447"
-      rpy="3.1416 -1.5708 3.1416" />
+      rpy="-0.25 0 0" />
     <parent
       link="arm_roll_forearm_link" />
@@ -325,5 +328,5 @@
       link="arm_pitch_wrist_link" />
     <axis
-      xyz="0 0 -1" />
+      xyz="-1 0 0" />
     <limit
       lower="-0.46"
@@ -342,6 +345,6 @@
       <inertia
         ixx="0.00046764"
-        ixy="1.372E-19"
-        ixz="1.5587E-19"
+        ixy="1.3696E-19"
+        ixz="1.5471E-19"
         iyy="0.000956"
         iyz="7.6437E-06"
@@ -354,19 +357,19 @@
       <geometry>
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
File: reseq_description/description/control/ros2_control.xacro (robot description, xacro)
@@ -10,4 +10,5 @@
             </xacro:unless>
             <param name="num_modules">${NumModules}</param>
+            <param name="command_cycle_ms">30</param>
             <!-- TODO: vcan, and gazebo alternatives -->
         </hardware>

Commit message: (#99) fix: correct misaligned arm meshes and add gazebo joint dynamics / self-collisions

File: reseq_arm_mk2/urdf/reseq_arm_mk2.xacro (robot description, xacro)
@@ -99,4 +99,5 @@
       effort="6"
       velocity="2" />
+    <dynamics damping="0.5" friction="0.1" />
   </joint>
   <link
@@ -119,5 +120,5 @@
       <origin
         xyz="0 0 0"
-        rpy="0 0 0" />
+        rpy="0 1.5708 0" />
       <geometry>
         <mesh
@@ -133,5 +134,5 @@
       <origin
         xyz="0 0 0"
-        rpy="0 0 0" />
+        rpy="0 1.5708 0" />
       <geometry>
         <mesh
@@ -157,4 +158,5 @@
       effort="6"
       velocity="2" />
+    <dynamics damping="0.5" friction="0.1" />
   </joint>
   <link
@@ -215,4 +217,5 @@
       effort="6"
       velocity="2" />
+    <dynamics damping="0.5" friction="0.1" />
   </joint>
   <link
@@ -273,4 +276,5 @@
       effort="3"
       velocity="1" />
+    <dynamics damping="0.5" friction="0.1" />
   </joint>
   <link
@@ -293,5 +297,5 @@
       <origin
         xyz="0 0 0"
-        rpy="0 0 0" />
+        rpy="0 -1.5708 0" />
       <geometry>
         <mesh
@@ -307,5 +311,5 @@
       <origin
         xyz="0 0 0"
-        rpy="0 0 0" />
+        rpy="0 -1.5708 0" />
       <geometry>
         <mesh
@@ -331,4 +335,5 @@
       effort="3"
       velocity="1" />
+    <dynamics damping="0.5" friction="0.1" />
   </joint>
   <link
@@ -389,4 +394,33 @@
       effort="3"
       velocity="1" />
-  </joint>
+    <dynamics damping="0.5" friction="0.1" />
+  </joint>
+  <gazebo reference="arm_base_link">
+    <material>Gazebo/Grey</material>
+    <selfCollide>false</selfCollide>
+  </gazebo>
+  <gazebo reference="arm_diff_pitch_link">
+    <material>Gazebo/Grey</material>
+    <selfCollide>false</selfCollide>
+  </gazebo>
+  <gazebo reference="arm_diff_roll_link">
+    <material>Gazebo/Grey</material>
+    <selfCollide>false</selfCollide>
+  </gazebo>
+  <gazebo reference="arm_pitch_forearm_link">
+    <material>Gazebo/Grey</material>
+    <selfCollide>false</selfCollide>
+  </gazebo>
+  <gazebo reference="arm_roll_forearm_link">
+    <material>Gazebo/Grey</material>
+    <selfCollide>false</selfCollide>
+  </gazebo>
+  <gazebo reference="arm_pitch_wrist_link">
+    <material>Gazebo/Grey</material>
+    <selfCollide>false</selfCollide>
+  </gazebo>
+  <gazebo reference="arm_roll_wrist_link">
+    <material>Gazebo/Grey</material>
+    <selfCollide>false</selfCollide>
+  </gazebo>
 </robot>

Commit message: (#99) fix: correct misaligned arm meshes and add gazebo joint dynamic

File: reseq_arm_mk2/urdf/reseq_arm_mk2.xacro (robot description, xacro)
@@ -46,14 +46,14 @@
     <inertial>
       <origin
-        xyz="-1.3878E-17 0.00059334 1.7347E-18"
+        xyz="-0.00059334 -1.3878E-17 3.4694E-18"
         rpy="0 0 0" />
       <mass
         value="0.28931" />
       <inertia
-        ixx="0.0002425"
-        ixy="-1.6941E-20"
-        ixz="-1.5531E-20"
-        iyy="0.00023577"
-        iyz="8.3058E-21"
+        ixx="0.00023577"
+        ixy="1.6941E-20"
+        ixz="-8.3058E-21"
+        iyy="0.0002425"
+        iyz="-1.5531E-20"
         izz="0.00025759" />
     </inertial>
@@ -87,5 +87,5 @@
     <origin
       xyz="0 0 0"
-      rpy="1.5708 -1.309 0" />
+      rpy="1.5708 0.2 0" />
     <parent
       link="arm_base_link" />
@@ -95,8 +95,9 @@
       xyz="0 0 -1" />
     <limit
-      lower="-1.05"
-      upper="1.309"
+      lower="-0.1"
+      upper="2.8"
       effort="6"
       velocity="2" />
+    <dynamics damping="0.5" friction="0.1" />
   </joint>
   <link
@@ -104,20 +105,20 @@
     <inertial>
       <origin
-        xyz="1.1115E-08 7.62E-08 -0.14664"
+        xyz="-0.14664 7.62E-08 -1.1115E-08"
         rpy="0 0 0" />
       <mass
         value="0.11865" />
       <inertia
-        ixx="0.00051345"
-        ixy="-2.7475E-10"
-        ixz="-9.7641E-11"
+        ixx="1.0228E-05"
+        ixy="2.2625E-10"
+        ixz="9.7641E-11"
         iyy="0.00051383"
-        iyz="2.2625E-10"
-        izz="1.0228E-05" />
-    </inertial>
-    <visual>
-      <origin
-        xyz="0 0 0"
-        rpy="0 0 0" />
+        iyz="2.7475E-10"
+        izz="0.00051345" />
+    </inertial>
+    <visual>
+      <origin
+        xyz="0 0 0"
+        rpy="0 1.5708 0" />
       <geometry>
         <mesh
@@ -133,5 +134,5 @@
       <origin
         xyz="0 0 0"
-        rpy="0 0 0" />
+        rpy="0 1.5708 0" />
       <geometry>
         <mesh
@@ -145,5 +146,5 @@
     <origin
       xyz="0 0 0"
-      rpy="1.5708 1.5708 0" />
+      rpy="0 0 0" />
     <parent
       link="arm_diff_pitch_link" />
@@ -151,5 +152,5 @@
       link="arm_diff_roll_link" />
     <axis
-      xyz="0 0 1" />
+      xyz="1 0 0" />
     <limit
       lower="-3.14"
@@ -157,4 +158,5 @@
       effort="6"
       velocity="2" />
+    <dynamics damping="0.5" friction="0.1" />
   </joint>
   <link
@@ -169,7 +171,7 @@
         ixx="4.6765E-05"
         ixy="-9.086E-05"
-        ixz="1.3681E-20"
+        ixz="1.3572E-20"
         iyy="0.00027451"
-        iyz="3.2975E-21"
+        iyz="3.2775E-21"
         izz="0.00031255" />
     </inertial>
@@ -202,6 +204,6 @@
     type="revolute">
     <origin
-      xyz="0 0 -0.28857"
-      rpy="3.1416 -1.5708 3.1416" />
+      xyz="-0.28857 0 0"
+      rpy="0 0 0.2" />
     <parent
       link="arm_diff_roll_link" />
@@ -211,8 +213,9 @@
       xyz="0 0 1" />
     <limit
-      lower="-1.05"
+      lower="-0.1"
       upper="2.88"
       effort="6"
       velocity="2" />
+    <dynamics damping="0.5" friction="0.1" />
   </joint>
   <link
@@ -226,6 +229,6 @@
       <inertia
         ixx="5.2065E-05"
-        ixy="1.6912E-22"
-        ixz="-6.5731E-21"
+        ixy="1.7168E-22"
+        ixz="-6.5851E-21"
         iyy="4.9885E-05"
         iyz="2.3291E-07"
@@ -261,5 +264,5 @@
     <origin
       xyz="0.15351 0.074002 0"
-      rpy="0.2618 -1.5708 3.1416" />
+      rpy="0.2618 -1.5708 3.14" />
     <parent
       link="arm_pitch_forearm_link" />
@@ -273,4 +276,5 @@
       effort="3"
       velocity="1" />
+    <dynamics damping="0.5" friction="0.1" />
   </joint>
   <link
@@ -278,20 +282,20 @@
     <inertial>
       <origin
-        xyz="0.045311 1.3878E-17 -3.296E-17"
+        xyz="5.3776E-17 2.7756E-17 0.045311"
         rpy="0 0 0" />
       <mass
         value="0.056876" />
       <inertia
-        ixx="1.5222E-05"
-        ixy="2.5626E-21"
-        ixz="3.1474E-21"
+        ixx="1.6114E-05"
+        ixy="3.0569E-22"
+        ixz="-3.5109E-21"
         iyy="2.2881E-05"
-        iyz="-1.4326E-21"
-        izz="1.6114E-05" />
-    </inertial>
-    <visual>
-      <origin
-        xyz="0 0 0"
-        rpy="0 0 0" />
+        iyz="1.0674E-21"
+        izz="1.5222E-05" />
+    </inertial>
+    <visual>
+      <origin
+        xyz="0 0 0"
+        rpy="0 -1.5708 0" />
       <geometry>
         <mesh
@@ -307,5 +311,5 @@
       <origin
         xyz="0 0 0"
-        rpy="0 0 0" />
+        rpy="0 -1.5708 0" />
       <geometry>
         <mesh
@@ -319,5 +323,5 @@
     <origin
       xyz="0 0 0.05447"
-      rpy="3.1416 -1.5708 3.1416" />
+      rpy="-0.25 0 0" />
     <parent
       link="arm_roll_forearm_link" />
@@ -325,5 +329,5 @@
       link="arm_pitch_wrist_link" />
     <axis
-      xyz="0 0 -1" />
+      xyz="-1 0 0" />
     <limit
       lower="-0.46"
@@ -331,4 +335,5 @@
       effort="3"
       velocity="1" />
+    <dynamics damping="0.5" friction="0.1" />
   </joint>
   <link
@@ -342,6 +347,6 @@
       <inertia
         ixx="0.00046764"
-        ixy="1.372E-19"
-        ixz="1.5587E-19"
+        ixy="1.3696E-19"
+        ixz="1.5471E-19"
         iyy="0.000956"
         iyz="7.6437E-06"
@@ -377,5 +382,5 @@
     <origin
       xyz="0 0 0"
-      rpy="0 1.5708 0" />
+      rpy="0 0 0" />
     <parent
       link="arm_pitch_wrist_link" />
@@ -389,4 +394,33 @@
       effort="3"
       velocity="1" />
-  </joint>
+    <dynamics damping="0.5" friction="0.1" />
+  </joint>
+  <gazebo reference="arm_base_link">
+    <material>Gazebo/Grey</material>
+    <selfCollide>false</selfCollide>
+  </gazebo>
+  <gazebo reference="arm_diff_pitch_link">
+    <material>Gazebo/Grey</material>
+    <selfCollide>false</selfCollide>
+  </gazebo>
+  <gazebo reference="arm_diff_roll_link">
+    <material>Gazebo/Grey</material>
+    <selfCollide>false</selfCollide>
+  </gazebo>
+  <gazebo reference="arm_pitch_forearm_link">
+    <material>Gazebo/Grey</material>
+    <selfCollide>false</selfCollide>
+  </gazebo>
+  <gazebo reference="arm_roll_forearm_link">
+    <material>Gazebo/Grey</material>
+    <selfCollide>false</selfCollide>
+  </gazebo>
+  <gazebo reference="arm_pitch_wrist_link">
+    <material>Gazebo/Grey</material>
+    <selfCollide>false</selfCollide>
+  </gazebo>
+  <gazebo reference="arm_roll_wrist_link">
+    <material>Gazebo/Grey</material>
+    <selfCollide>false</selfCollide>
+  </gazebo>
 </robot>

Commit message: cartesian solver now uses full 6-row jacobian and quick fixes

File: reseq_arm_mk2/urdf/reseq_arm_mk2.xacro (robot description, xacro)
@@ -396,4 +396,16 @@
     <dynamics damping="0.5" friction="0.1" />
   </joint>
+  <link name="tcp" />
+  <joint name="tcp_joint" type="fixed">
+    <parent link="arm_roll_wrist_link" />
+    <child link="tcp" />
+    <origin xyz="0 0 0.12425" rpy="0 0 0" />
+  </joint>
+  <link name="tool0" />
+  <joint name="tool0_joint" type="fixed">
+    <parent link="tcp" />
+    <child link="tool0" />
+    <origin xyz="0 0 0" rpy="0 -1.5708 1.5708" />
+  </joint>
   <gazebo reference="arm_base_link">
     <material>Gazebo/Grey</material>
