Commit message: Refine arm end-effector modes

File: reseq_arm_mk2/urdf/reseq_arm_mk2.xacro (robot description, xacro)
@@ -2,4 +2,10 @@
 <robot
   name="reseq_arm_mk2" xmlns:xacro="http://www.ros.org/wiki/xacro">
+  <xacro:property
+    name="arm_pitch_effort"
+    value="${60 if '$(arg sim_mode)' == 'true' else 6}" />
+  <xacro:property
+    name="arm_wrist_pitch_effort"
+    value="${30 if '$(arg sim_mode)' == 'true' else 3}" />
   <link
     name="arm_base_link">
@@ -97,5 +103,5 @@
       lower="-0.1"
       upper="2.8"
-      effort="6"
+      effort="${arm_pitch_effort}"
       velocity="2" />
     <dynamics damping="0.5" friction="0.1" />
@@ -215,5 +221,5 @@
       lower="-0.1"
       upper="2.88"
-      effort="6"
+      effort="${arm_pitch_effort}"
       velocity="2" />
     <dynamics damping="0.5" friction="0.1" />
@@ -333,5 +339,5 @@
       lower="-0.46"
       upper="1.57"
-      effort="3"
+      effort="${arm_wrist_pitch_effort}"
       velocity="1" />
     <dynamics damping="0.5" friction="0.1" />

File: reseq_description/description/mk2/arm/control_joints.xacro (robot description, xacro)
@@ -2,48 +2,72 @@
 <robot xmlns:xacro="http://www.ros.org/wiki/xacro">
     <joint name="mod1__base_pitch_arm_joint">
-        <command_interface name="position" />
-        <state_interface name="position" />
+        <xacro:unless value="$(arg sim_mode)">
+            <command_interface name="position" />
+        </xacro:unless>
+        <state_interface name="position">
+            <param name="initial_value">0.0</param>
+        </state_interface>
         <state_interface name="velocity" />
-        <xacro:if value="$(arg sim_mode)" >
+        <xacro:if value="$(arg sim_mode)">
             <command_interface name="velocity" />
         </xacro:if>
     </joint>
     <joint name="mod1__base_roll_arm_joint">
-        <command_interface name="position" />
-        <state_interface name="position" />
+        <xacro:unless value="$(arg sim_mode)">
+            <command_interface name="position" />
+        </xacro:unless>
+        <state_interface name="position">
+            <param name="initial_value">0.0</param>
+        </state_interface>
         <state_interface name="velocity" />
-        <xacro:if value="$(arg sim_mode)" >
+        <xacro:if value="$(arg sim_mode)">
             <command_interface name="velocity" />
         </xacro:if>
     </joint>
     <joint name="mod1__elbow_pitch_arm_joint">
-        <command_interface name="position" />
-        <state_interface name="position" />
+        <xacro:unless value="$(arg sim_mode)">
+            <command_interface name="position" />
+        </xacro:unless>
+        <state_interface name="position">
+            <param name="initial_value">0.0</param>
+        </state_interface>
         <state_interface name="velocity" />
-         <xacro:if value="$(arg sim_mode)" >
+        <xacro:if value="$(arg sim_mode)">
             <command_interface name="velocity" />
         </xacro:if>
     </joint>
     <joint name="mod1__forearm_roll_arm_joint">
-        <command_interface name="position" />
-        <state_interface name="position" />
+        <xacro:unless value="$(arg sim_mode)">
+            <command_interface name="position" />
+        </xacro:unless>
+        <state_interface name="position">
+            <param name="initial_value">0.0</param>
+        </state_interface>
         <state_interface name="velocity" />
-         <xacro:if value="$(arg sim_mode)" >
+        <xacro:if value="$(arg sim_mode)">
             <command_interface name="velocity" />
         </xacro:if>
     </joint>
     <joint name="mod1__wrist_pitch_arm_joint">
-        <command_interface name="position" />
-        <state_interface name="position" />
+        <xacro:unless value="$(arg sim_mode)">
+            <command_interface name="position" />
+        </xacro:unless>
+        <state_interface name="position">
+            <param name="initial_value">0.0</param>
+        </state_interface>
         <state_interface name="velocity" />
-        <xacro:if value="$(arg sim_mode)" >
+        <xacro:if value="$(arg sim_mode)">
             <command_interface name="velocity" />
         </xacro:if>
     </joint>
     <joint name="mod1__wrist_roll_arm_joint">
-        <command_interface name="position" />
-        <state_interface name="position" />
+        <xacro:unless value="$(arg sim_mode)">
+            <command_interface name="position" />
+        </xacro:unless>
+        <state_interface name="position">
+            <param name="initial_value">0.0</param>
+        </state_interface>
         <state_interface name="velocity" />
-        <xacro:if value="$(arg sim_mode)" >
+        <xacro:if value="$(arg sim_mode)">
             <command_interface name="velocity" />
         </xacro:if>
