Commit message: feat: Add realsense link

File: reseq_arm_mk2/urdf/reseq_arm_mk2.xacro (robot description, xacro)
@@ -430,3 +430,22 @@
     <selfCollide>false</selfCollide>
   </gazebo>
+  <!-- realsense link for camera mounting - attached to the wrist on the beak -->
+  <xacro:unless value="$(arg sim_mode)">
+    <link name="realsense_link">
+          <visual name="cube">
+              <origin xyz="0 0 0"/>
+              <geometry>
+                  <box size="0.01 0.01 0.01"/>
+              </geometry>
+              <material name="green">
+                  <color rgba="0 1 0 1.0"/>
+              </material>
+          </visual>
+      </link>
+    <joint name="realsense_joint" type="fixed">
+      <origin xyz="0 -0.03 0.15" rpy="1.57 -1.57 0"/>
+      <parent link="arm_roll_wrist_link"/>
+      <child link="realsense_link"/>
+    </joint>
+  </xacro:unless>
 </robot>

Commit message: fix: Update motor parameters and add rear-wheel drive support

File: reseq_arm_mk2/urdf/reseq_arm_mk2.xacro (robot description, xacro)
@@ -2,10 +2,5 @@
 <robot
   name="reseq_arm_mk2" xmlns:xacro="http://www.ros.org/wiki/xacro">
-  <xacro:property
-    name="arm_pitch_effort"
-    value="${60 if '$(arg sim_mode)' == 'true' else 6}" />
-  <xacro:property
-    name="arm_wrist_pitch_effort"
-    value="${30 if '$(arg sim_mode)' == 'true' else 3}" />
+  <xacro:include filename="$(find reseq_description)/description/macros/reseq_parameters.xacro" />
   <link
     name="arm_base_link">
@@ -162,5 +157,5 @@
       lower="-3.14"
       upper="3.14"
-      effort="6"
+      effort="${arm_base_roll_effort}"
       velocity="2" />
     <dynamics damping="0.5" friction="0.1" />
@@ -280,5 +275,5 @@
       lower="-3.14"
       upper="3.14"
-      effort="3"
+      effort="${arm_forearm_roll_effort}"
       velocity="1" />
     <dynamics damping="0.5" friction="0.1" />
@@ -398,5 +393,5 @@
       lower="-3.14"
       upper="3.14"
-      effort="3"
+      effort="${arm_wrist_roll_effort}"
       velocity="1" />
     <dynamics damping="0.5" friction="0.1" />

File: reseq_description/description/control/body_joints.xacro (robot description, xacro)
@@ -5,6 +5,6 @@
         <xacro:if value="${module &lt;= n_modules}">
             <!-- Wheels -->
-            <xacro:control_wheel_factory id="${module}" pos="front" side="left" />
-            <xacro:control_wheel_factory id="${module}" pos="front" side="right" />
+            <!-- Note: The real robot is rear-wheel drive,
+            so we only expose control interfaces for the rear (back) wheels. -->
             <xacro:control_wheel_factory id="${module}" pos="back" side="left" />
             <xacro:control_wheel_factory id="${module}" pos="back" side="right" />

File: reseq_description/description/macros/joint.xacro (robot description, xacro)
@@ -13,5 +13,5 @@
       <child link="joint_r_${id}_link" />
       <!-- Effort in Nm -->
-      <limit effort="7.0" lower="${-roll}" upper="${roll}" velocity="3.14" />
+      <limit effort="${RollTorque}" lower="${-roll}" upper="${roll}" velocity="${RollVelocity}" />
       <origin xyz="-${WheelBase/2} 0 0" rpy="0 0 0" />
       <axis xyz="1 0 0" />
@@ -42,5 +42,5 @@
       <child link="joint_y_${id}_link" />
       <!-- Effort in Nm -->
-      <limit effort="7.0" lower="${-yaw}" upper="${yaw}" velocity="3.14" />
+      <limit effort="${YawTorque}" lower="${-yaw}" upper="${yaw}" velocity="${YawVelocity}" />
       <origin xyz="-${JointB} 0 0" rpy="0 0 0" />
       <axis xyz="0 0 1" />
@@ -80,5 +80,5 @@
       <child link="joint_p_${id}_link" />
       <!-- Effort in Nm -->
-      <limit effort="7.0" lower="${-pitch}" upper="${pitch}" velocity="3.14" />
+      <limit effort="${PitchTorque}" lower="${-pitch}" upper="${pitch}" velocity="${PitchVelocity}" />
       <origin xyz="${-JointA} 0 0" rpy="0 0 0" />
       <axis xyz="0 1 0" />

File: reseq_description/description/macros/reseq_parameters.xacro (robot description, xacro)
@@ -29,21 +29,24 @@
   <xacro:property name="roll" value="${pi/2}"/>
   <xacro:property name="yaw" value="${pi/4}"/>
+  <!-- actuator limits at 12V: angular velocity [rad/s], output torque [Nm]. -->
+  <xacro:property name="XM540Velocity" value="3.14"/>  <!-- XM540-W270-T -->
+  <xacro:property name="XM540Torque" value="10.6"/>
+  <xacro:property name="XL430Velocity" value="6.39"/>  <!-- XL430-W250-T -->
+  <xacro:property name="XL430Torque" value="1.5"/>
+  <!-- Mechanism limits may be derated independently here. -->
+  <xacro:property name="TractionVelocity" value="${XM540Velocity}"/>
+  <xacro:property name="TractionTorque" value="${XM540Torque}"/>
+  <xacro:property name="YawVelocity" value="${XM540Velocity}"/>
+  <xacro:property name="YawTorque" value="${XM540Torque}"/>
+  <xacro:property name="PitchVelocity" value="${XM540Velocity}"/>
+  <xacro:property name="PitchTorque" value="${XM540Torque}"/>
+  <xacro:property name="RollVelocity" value="${XL430Velocity}"/>
+  <xacro:property name="RollTorque" value="${XL430Torque}"/>
+  <xacro:property name="arm_pitch_effort" value="${XM540Torque}" />
+  <xacro:property name="arm_wrist_pitch_effort" value="${XL430Torque}" />
+  <xacro:property name="arm_base_roll_effort" value="${XM540Torque}" />
+  <xacro:property name="arm_forearm_roll_effort" value="${XL430Torque}" />
+  <xacro:property name="arm_wrist_roll_effort" value="${XL430Torque}" />
   <xacro:property name="JointAMass" value="${config['xacro']['JointAMass']}"/>
   <xacro:property name="JointBMass" value="${config['xacro']['JointBMass']}"/>
-  <!-- Rviz colors (for Gazebo ones change in single files) (from 0 to 1) -->
-  <material name="ChassisColor">
-    <color rgba="1 1 1 1" />
-  </material>
-  <material name="WheelColor">
-    <color rgba="0 0 0 1" />
-  </material>
-  <material name="JointColor">
-    <color rgba="0.5 0.5 0.5 1" />
-  </material>
-  <material name="LidarColor">
-    <color rgba="0.5 0.5 0.5 1" />
-  </material>
-  <material name="IMUColor">
-    <color rgba="0.1 0.1 0.1 1" />
-  </material>
 </robot>

File: reseq_description/description/macros/wheel.xacro (robot description, xacro)
@@ -16,10 +16,21 @@
             <xacro:property name="side_sign" value="-1" />
         </xacro:if>
-        <joint name="mod${id}__${side}_${pos}_wheel" type="continuous">
-        <parent link="chassis${id}_link" />
-        <child link="${side}_${pos}_wheel_${id}_link" />
-        <origin xyz="${pos_sign*WheelBase/2} ${side_sign*(ModuleWidth/2-TrackWidth/2)} 0" rpy="0 0 0" />
-        <axis xyz="0 1 0" />
-        </joint>
+        <xacro:if value="${pos == 'back'}">
+            <joint name="mod${id}__${side}_${pos}_wheel" type="revolute">
+                <limit effort="${TractionTorque}" lower="-1e10" upper="1e10" velocity="${TractionVelocity}" />
+                <parent link="chassis${id}_link" />
+                <child link="${side}_${pos}_wheel_${id}_link" />
+                <origin xyz="${pos_sign*WheelBase/2} ${side_sign*(ModuleWidth/2-TrackWidth/2)} 0" rpy="0 0 0" />
+                <axis xyz="0 1 0" />
+            </joint>
+        </xacro:if>
+        <xacro:unless value="${pos == 'back'}">
+            <joint name="mod${id}__${side}_${pos}_wheel" type="continuous">
+                <parent link="chassis${id}_link" />
+                <child link="${side}_${pos}_wheel_${id}_link" />
+                <origin xyz="${pos_sign*WheelBase/2} ${side_sign*(ModuleWidth/2-TrackWidth/2)} 0" rpy="0 0 0" />
+                <axis xyz="0 1 0" />
+            </joint>
+        </xacro:unless>
         <link name="${side}_${pos}_wheel_${id}_link">
         <visual>

File: reseq_description/description/mk1/reseq.urdf.xacro (robot description, xacro)
@@ -4,4 +4,5 @@
   <xacro:arg name="sim_mode" default="false"/>
   <xacro:include filename="$(find reseq_description)/description/macros/reseq_parameters.xacro" />
+  <xacro:include filename="$(find reseq_description)/description/macros/materials.xacro" />
   <xacro:include filename="$(find reseq_description)/description/macros/inertial_macros.xacro" />
   <xacro:include filename="$(find reseq_description)/description/macros/utils.xacro" />

File: reseq_description/description/mk2/reseq.urdf.xacro (robot description, xacro)
@@ -4,4 +4,5 @@
   <xacro:arg name="sim_mode" default="false"/>
   <xacro:include filename="$(find reseq_description)/description/macros/reseq_parameters.xacro" />
+  <xacro:include filename="$(find reseq_description)/description/macros/materials.xacro" />
   <xacro:include filename="$(find reseq_description)/description/macros/inertial_macros.xacro" />
   <xacro:include filename="$(find reseq_description)/description/macros/utils.xacro" />

Commit message: feat(arm): add new beak gripper model
- beak_body.STL (body + fixed lower finger) replaces the old fused gripper mesh
  on arm_roll_wrist_link, with its inertial
- new beak_finger_upper_link and revolute joint mod1__beak (axis X,
  0 = closed, positive = open)
- SRDF collision exclusions for the new link

Placeholders: beak masses (CAD at 1 g/cm3), upper limit (1.0 rad) and servo
effort/velocity. Lower limit is -0.05 because DART locks a joint that starts
exactly on its limit.

File: reseq_arm_mk2/urdf/reseq_arm_mk2.xacro (robot description, xacro)
@@ -342,37 +342,37 @@
     <inertial>
       <origin
-        xyz="2.6021E-17 0.0094155 0.12425"
-        rpy="0 0 0" />
-      <mass
-        value="0.55801" />
-      <inertia
-        ixx="0.00046764"
-        ixy="1.3696E-19"
-        ixz="1.5471E-19"
-        iyy="0.000956"
-        iyz="7.6437E-06"
-        izz="0.00082011" />
-    </inertial>
-    <visual>
-      <origin
-        xyz="0 0 0"
-        rpy="0 0 0" />
-      <geometry>
-        <mesh
-          filename="package://reseq_arm_mk2/meshes/arm_roll_wrist_link.STL" />
-      </geometry>
-      <material
-        name="">
-        <color
-          rgba="0.75294 0.75294 0.75294 1" />
-      </material>
-    </visual>
-    <collision>
-      <origin
-        xyz="0 0 0"
-        rpy="0 0 0" />
-      <geometry>
-        <mesh
-          filename="package://reseq_arm_mk2/meshes/arm_roll_wrist_link.STL" />
+        xyz="0.0001 0.0071 0.1197"
+        rpy="0 0 0" />
+      <mass
+        value="0.1341" />
+      <inertia
+        ixx="1.332159E-04"
+        ixy="0"
+        ixz="-3.0E-10"
+        iyy="1.128104E-04"
+        iyz="-2.35230E-05"
+        izz="4.67873E-05" />
+    </inertial>
+    <visual>
+      <origin
+        xyz="0 0 0"
+        rpy="0 0 0" />
+      <geometry>
+        <mesh
+          filename="package://reseq_arm_mk2/meshes/beak_body.STL" />
+      </geometry>
+      <material
+        name="">
+        <color
+          rgba="0.75294 0.75294 0.75294 1" />
+      </material>
+    </visual>
+    <collision>
+      <origin
+        xyz="0 0 0"
+        rpy="0 0 0" />
+      <geometry>
+        <mesh
+          filename="package://reseq_arm_mk2/meshes/beak_body.STL" />
       </geometry>
     </collision>
@@ -397,4 +397,63 @@
     <dynamics damping="0.5" friction="0.1" />
   </joint>
+  <link
+    name="beak_finger_upper_link">
+    <inertial>
+      <origin
+        xyz="0.0208 0.0127 0.0386"
+        rpy="0 0 0" />
+      <mass
+        value="0.0233" />
+      <inertia
+        ixx="7.8788E-06"
+        ixy="-6.43E-08"
+        ixz="-2.019E-07"
+        iyy="1.04238E-05"
+        iyz="-2.6102E-06"
+        izz="5.3419E-06" />
+    </inertial>
+    <visual>
+      <origin
+        xyz="0 0 0"
+        rpy="0 0 0" />
+      <geometry>
+        <mesh
+          filename="package://reseq_arm_mk2/meshes/beak_finger_upper.STL" />
+      </geometry>
+      <material
+        name="">
+        <color
+          rgba="0.75294 0.75294 0.75294 1" />
+      </material>
+    </visual>
+    <collision>
+      <origin
+        xyz="0 0 0"
+        rpy="0 0 0" />
+      <geometry>
+        <mesh
+          filename="package://reseq_arm_mk2/meshes/beak_finger_upper.STL" />
+      </geometry>
+    </collision>
+  </link>
+  <joint
+    name="mod1__beak"
+    type="revolute">
+    <origin
+      xyz="-0.021 -0.0073 0.1307"
+      rpy="0 0 0" />
+    <parent
+      link="arm_roll_wrist_link" />
+    <child
+      link="beak_finger_upper_link" />
+    <axis
+      xyz="1 0 0" />
+    <limit
+      lower="-0.05"
+      upper="1.0"
+      effort="${XL430Torque}"
+      velocity="${XL430Velocity}" />
+    <dynamics damping="0.5" friction="0.1" />
+  </joint>
   <gazebo reference="arm_base_link">
     <material>Gazebo/Grey</material>
@@ -422,4 +481,8 @@
   </gazebo>
   <gazebo reference="arm_roll_wrist_link">
+    <material>Gazebo/Grey</material>
+    <selfCollide>false</selfCollide>
+  </gazebo>
+  <gazebo reference="beak_finger_upper_link">
     <material>Gazebo/Grey</material>
     <selfCollide>false</selfCollide>
