Commit message: fix(lidar): Adjust dimensions and positions of lidar components in xacro file
Co-authored-by: Copilot <copilot@github.com>

File: reseq_description/description/sensors/lidar.xacro (robot description, xacro)
@@ -4,5 +4,5 @@
     <parent link="chassis2_link"/>
     <child link="laser_frame"/>
-    <origin xyz="-0.07 0 0.1" rpy="0 0 0"/>
+    <origin xyz="-0.07 0 0.2" rpy="0 0 0"/>
   </joint>
   <link name="laser_frame">
@@ -10,5 +10,5 @@
     <visual>
       <geometry>
-        <cylinder radius="0.05" length="0.04"/>
+        <cylinder radius="0.03" length="0.04"/>
       </geometry>
       <material name="LidarColor"/>
@@ -16,7 +16,7 @@
     <!-- pole to lidar -->
     <visual>
-      <origin xyz="0 0 -0.05" rpy="0 0 0"/>
+      <origin xyz="0 0 -0.1" rpy="0 0 0"/>
       <geometry>
-        <cylinder radius="0.01" length="0.1"/>
+        <cylinder radius="0.01" length="0.15"/>
       </geometry>
       <material name="LidarColor"/>
@@ -24,8 +24,8 @@
     <collision>
       <geometry>
-        <cylinder radius="0.05" length="0.04"/>
+        <cylinder radius="0.03" length="0.04"/>
       </geometry>
     </collision>
-    <xacro:inertial_cylinder_z mass="0.1" length="0.04" radius="0.05">
+    <xacro:inertial_cylinder_z mass="0.1" length="0.04" radius="0.03">
       <origin xyz="0 0 0" rpy="0 0 ${pi/2}"/>
     </xacro:inertial_cylinder_z>
