Commit message: fix: Joint body_to_arm

File: reseq_description/description/mk2/reseq.urdf.xacro (robot description, xacro)
@@ -8,4 +8,9 @@
   <xacro:include filename="$(find reseq_description)/description/macros/reseq_body.xacro" />
   <xacro:include filename="$(find reseq_arm_mk2)/urdf/reseq_arm_mk2.xacro" />
+  <joint name="body_to_arm_joint" type="fixed">
+    <parent link="chassis1_link"/>
+    <child link="arm_base_link"/>
+    <origin xyz="${WheelBase/2} 0 0" />
+  </joint>
   <xacro:include filename="$(find reseq_description)/description/control/ros2_control.xacro" />
 </robot>

Commit message: Add real arm TCP frame
Define a real-robot tcp link matching the simulated camera holder frame so the Cartesian arm controller uses the same KDL tool frame on hardware.

File: reseq_description/description/mk2/reseq.urdf.xacro (robot description, xacro)
@@ -13,4 +13,13 @@
     <origin xyz="${WheelBase/2} 0 0" />
   </joint>
+  <!-- Real robot TCP frame matching the simulated camera holder frame. -->
+  <xacro:unless value="$(arg sim_mode)">
+    <joint name="tcp_joint" type="fixed">
+      <origin xyz="0 -0.03 0.15" rpy="1.57 -1.57 0"/>
+      <parent link="arm_roll_wrist_link"/>
+      <child link="tcp"/>
+    </joint>
+    <link name="tcp"/>
+  </xacro:unless>
   <xacro:include filename="$(find reseq_description)/description/control/ros2_control.xacro" />
   <!-- Cameras holder (RGBD + thermal) on the arm end-effector — Gazebo sim only -->
